Commit message: Freddy description in rolling
- Added torso shoulders
- Added kinova gen3 arms
- Added robotiq 2f85 grippers

File: freddy_base_description/urdf/materials.urdf.xacro (robot description, xacro)
@@ -2,29 +2,29 @@
 <robot>
   <material name="Orange">
-    <color rgba="1.0 0.4 0.0 1.0"/>
+    <color rgba="1.0 0.4 0.0 1.0" />
   </material>
   <material name="Grey">
-    <color rgba="0.7 0.7 0.7 1.0"/>
+    <color rgba="0.7 0.7 0.7 1.0" />
   </material>
   <material name="DarkGrey">
-    <color rgba="0.3 0.3 0.3 1.0"/>
+    <color rgba="0.3 0.3 0.3 1.0" />
   </material>
   <material name="White">
-    <color rgba="1.0 1.0 1.0 1.0"/>
+    <color rgba="1.0 1.0 1.0 1.0" />
   </material>
   <material name="Black">
-    <color rgba="0.0 0.0 0.0 1.0"/>
+    <color rgba="0.0 0.0 0.0 1.0" />
   </material>
   <material name="Red">
-    <color rgba="1.0 0.0 0.0 1.0"/>
+    <color rgba="1.0 0.0 0.0 1.0" />
   </material>
   <material name="Green">
-    <color rgba="0.0 1.0 0.0 1.0"/>
+    <color rgba="0.0 1.0 0.0 1.0" />
   </material>
   <material name="Blue">
-    <color rgba="0.0 0.0 0.8 1.0"/>
+    <color rgba="0.0 0.0 0.8 1.0" />
   </material>
   <material name="LightGrey">
-    <color rgba="0.82 0.82 0.82 1.0"/>
+    <color rgba="0.82 0.82 0.82 1.0" />
   </material>
 </robot>

File: freddy_description/robots/freddy.urdf.xacro (robot description, xacro)
@@ -1,14 +1,208 @@
 <?xml version='1.0'?>
-<robot xmlns:xacro="http://www.ros.org/wiki/xacro" name="freddy" >
+<robot xmlns:xacro="http://www.ros.org/wiki/xacro" name="freddy">
     <xacro:arg name="use_gpu_2d_laser" default="false" />
+    <!-- Arguments -->
+    <xacro:arg name="prefix_arm_left" default="kinova_left_" />
+    <xacro:arg name="prefix_arm_right" default="kinova_right_" />
+    <xacro:arg name="arm" default="gen3" />
+    <xacro:arg name="dof" default="7" />
+    <xacro:arg name="vision" default="true" />
+    <xacro:arg name="robot_ip_left" default="192.168.1.10" />
+    <xacro:arg name="robot_ip_right" default="192.168.1.11" />
+    <xacro:arg name="username" default="admin" />
+    <xacro:arg name="password" default="admin" />
+    <xacro:arg name="port" default="10000" />
+    <xacro:arg name="port_realtime" default="10001" />
+    <xacro:arg name="session_inactivity_timeout_ms" default="60000" />
+    <xacro:arg name="connection_inactivity_timeout_ms" default="2000" />
+    <xacro:arg name="gripper" default="robotiq_2f_85" />
+    <xacro:arg name="gripper_joint_name" default="finger_joint" />
+    <xacro:arg name="gripper_max_velocity" default="100.0" />
+    <xacro:arg name="gripper_max_force" default="100.0" />
+    <xacro:arg name="use_internal_bus_gripper_comm" default="false" />
+    <xacro:arg name="use_fake_hardware" default="false" />
+    <xacro:arg name="fake_sensor_commands" default="false" />
+    <xacro:arg name="sim_gazebo" default="false" />
+    <xacro:arg name="sim_ignition" default="false" />
+    <xacro:arg name="sim_isaac" default="false" />
+    <xacro:arg name="gazebo_renderer" default="ogre" />
+    <xacro:arg name="camera_width" default="640" />
+    <xacro:arg name="camera_height" default="480" />
+    <xacro:arg name="camera_fps" default="6" />
+    <xacro:arg name="simulation_controllers"
+        default="$(find kortex_description)/arm/$(arg arm)/$(arg dof)dof/config/ros2_controllers.yaml" />
     <xacro:include filename="$(find freddy_base_description)/urdf/materials.urdf.xacro" />
     <xacro:include filename="$(find freddy_base_description)/urdf/freddy_base.urdf.xacro" />
     <xacro:include filename="$(find freddy_torso_description)/urdf/freddy_torso.urdf.xacro" />
-    <link name="base_link"/>
-    <xacro:freddy_base name="freddy_base" parent="base_link" use_gpu_2d_laser="$(arg use_gpu_2d_laser)">
-        <origin xyz="0.0 0.0 0.0" rpy="0.0 0.0 0.0"/>
+    <xacro:include filename="$(find kortex_description)/robots/kortex_robot.xacro" />
+    <!-- initial position for simulations (Mock Hardware, Gazebo, Ignition) -->
+    <xacro:arg name="initial_positions_file"
+        default="$(find freddy_description)/config/initial_positions.yaml" />
+    <!-- convert to property to use substitution in function -->
+    <xacro:property name="initial_positions_file" default="$(arg initial_positions_file)" />
+    <link name="base_link" />
+    <xacro:freddy_base name="freddy_base" parent="base_link"
+        use_gpu_2d_laser="$(arg use_gpu_2d_laser)">
+        <origin xyz="0.0 0.0 0.0" rpy="0.0 0.0 0.0" />
     </xacro:freddy_base>
     <xacro:freddy_torso name="freddy_torso" parent="base_link">
-        <origin xyz="0.0 0.0 0.0" rpy="0.0 0.0 0.0"/>
+        <origin xyz="0.0 0.0 0.0" rpy="0.0 0.0 0.0" />
     </xacro:freddy_torso>
+    <!-- arms -->
+    <!-- left arm -->
+    <xacro:load_robot
+        parent="freddy_torso_shoulder_left_arm_attach_link"
+        arm="$(arg arm)"
+        gripper="$(arg gripper)"
+        gripper_joint_name="$(arg gripper_joint_name)"
+        gripper_max_velocity="$(arg gripper_max_velocity)"
+        gripper_max_force="$(arg gripper_max_force)"
+        dof="$(arg dof)"
+        vision="$(arg vision)"
+        robot_ip="$(arg robot_ip_left)"
+        username="$(arg username)"
+        password="$(arg password)"
+        port="$(arg port)"
+        port_realtime="$(arg port_realtime)"
+        session_inactivity_timeout_ms="$(arg session_inactivity_timeout_ms)"
+        connection_inactivity_timeout_ms="$(arg connection_inactivity_timeout_ms)"
+        use_internal_bus_gripper_comm="$(arg use_internal_bus_gripper_comm)"
+        prefix="$(arg prefix_arm_left)"
+        use_fake_hardware="$(arg use_fake_hardware)"
+        fake_sensor_commands="$(arg fake_sensor_commands)"
+        sim_gazebo="$(arg sim_gazebo)"
+        sim_ignition="$(arg sim_ignition)"
+        sim_isaac="$(arg sim_isaac)"
+        initial_positions="${xacro.load_yaml(initial_positions_file)}">
+        <origin xyz="0 0 0" rpy="0 0 0" />
+    </xacro:load_robot>
+    <!-- right arm -->
+    <xacro:load_robot
+        parent="freddy_torso_shoulder_right_arm_attach_link"
+        arm="$(arg arm)"
+        gripper="$(arg gripper)"
+        gripper_joint_name="$(arg gripper_joint_name)"
+        gripper_max_velocity="$(arg gripper_max_velocity)"
+        gripper_max_force="$(arg gripper_max_force)"
+        dof="$(arg dof)"
+        vision="$(arg vision)"
+        robot_ip="$(arg robot_ip_right)"
+        username="$(arg username)"
+        password="$(arg password)"
+        port="$(arg port)"
+        port_realtime="$(arg port_realtime)"
+        session_inactivity_timeout_ms="$(arg session_inactivity_timeout_ms)"
+        connection_inactivity_timeout_ms="$(arg connection_inactivity_timeout_ms)"
+        use_internal_bus_gripper_comm="$(arg use_internal_bus_gripper_comm)"
+        prefix="$(arg prefix_arm_right)"
+        use_fake_hardware="$(arg use_fake_hardware)"
+        fake_sensor_commands="$(arg fake_sensor_commands)"
+        sim_gazebo="$(arg sim_gazebo)"
+        sim_ignition="$(arg sim_ignition)"
+        sim_isaac="$(arg sim_isaac)"
+        initial_positions="${xacro.load_yaml(initial_positions_file)}">
+        <origin xyz="0 0 0" rpy="0 0 0" />
+    </xacro:load_robot>
+    <!-- grasp links -->
+    <link name="kinova_left_grasp_link" />
+    <link name="kinova_right_grasp_link" />
+    <!-- grasp link joints -->
+    <joint name="kinova_left_grasp_link_joint" type="fixed">
+        <origin xyz="0 0 0.15" rpy="0 0 0" />
+        <parent link="kinova_left_robotiq_85_base_link" />
+        <child link="kinova_left_grasp_link" />
+    </joint>
+    <joint name="kinova_right_grasp_link_joint" type="fixed">
+        <origin xyz="0 0 0.15" rpy="0 0 0" />
+        <parent link="kinova_right_robotiq_85_base_link" />
+        <child link="kinova_right_grasp_link" />
+    </joint>
+    <xacro:if value="$(arg sim_gazebo)">
+        <!-- Gazebo plugins -->
+        <gazebo reference="world">
+        </gazebo>
+        <gazebo>
+            <plugin filename="libgazebo_ros2_control.so" name="gazebo_ros2_control">
+                <parameters>$(arg simulation_controllers)</parameters>
+            </plugin>
+        </gazebo>
+    </xacro:if>
+    <!-- TODO: Verify if the below snippet works for dual arm setup -->
+    <xacro:if value="$(arg sim_ignition)">
+        <!-- Gazebo plugins -->
+        <gazebo reference="world">
+        </gazebo>
+        <gazebo>
+            <plugin filename="libign_ros2_control-system.so"
+                name="ign_ros2_control::IgnitionROS2ControlPlugin">
+                <parameters>$(arg simulation_controllers)</parameters>
+                <controller_manager_node_name>$(arg prefix)controller_manager</controller_manager_node_name>
+            </plugin>
+            <plugin filename="libignition-gazebo-sensors-system.so"
+                name="ignition::gazebo::systems::Sensors">
+                <render_engine>$(arg gazebo_renderer)</render_engine>
+            </plugin>
+        </gazebo>
+        <gazebo reference="camera_color_frame">
+            <sensor name="camera_sensor" type="rgbd_camera">
+                <camera>
+                    <horizontal_fov>1.047</horizontal_fov>
+                    <image>
+                        <width>$(arg camera_width)</width>
+                        <height>$(arg camera_height)</height>
+                        <format>RGB_INT8</format>
+                    </image>
+                    <clip>
+                        <near>0.1</near>
+                        <far>5</far>
+                    </clip>
+                    <distortion>
+                        <k1>0.0</k1>
+                        <k2>0.0</k2>
+                        <k3>0.0</k3>
+                        <p1>0.0</p1>
+                        <p2>0.0</p2>
+                        <center>0.5 0.5</center>
+                    </distortion>
+                    <lens>
+                        <intrinsics>
+                            <fx>554.25469</fx>
+                            <fy>554.25469</fy>
+                            <cx>320.5</cx>
+                            <cy>240.5</cy>
+                            <s>0</s>
+                        </intrinsics>
+                        <!-- These need to match the intrinsics above or
+            Ignition will default to different default values -->
+                        <projection>
+                            <p_fx>554.25469</p_fx>
+                            <p_fy>554.25469</p_fy>
+                            <p_cx>320.5</p_cx>
+                            <p_cy>240.5</p_cy>
+                            <tx>0</tx>
+                            <ty>0</ty>
+                        </projection>
+                    </lens>
+                    <noise>
+                        <type>gaussian</type>
+                        <mean>0</mean>
+                        <stddev>0.00</stddev>
+                    </noise>
+                    <depth_camera>
+                        <clip>
+                            <near>0.25</near>
+                            <far>5</far>
+                        </clip>
+                    </depth_camera>
+                    <optical_frame_id>color_optical_frame</optical_frame_id>
+                </camera>
+                <ignition_frame_id>camera_color_frame</ignition_frame_id>
+                <always_on>1</always_on>
+                <update_rate>$(arg camera_fps)</update_rate>
+                <visualize>true</visualize>
+                <topic>wrist_mounted_camera</topic>
+                <enable_metrics>false</enable_metrics>
+            </sensor>
+        </gazebo>
+    </xacro:if>
 </robot>

File: freddy_torso_description/urdf/freddy_torso.urdf.xacro (robot description, xacro)
@@ -2,8 +2,12 @@
 <robot xmlns:xacro="http://www.ros.org/wiki/xacro">
     <!-- torso parameters -->
-    <xacro:property name="torso_height" value="0.3"/>
-    <xacro:property name="torso_width" value="0.4"/>
-    <xacro:property name="torso_thickness" value="0.19"/>
-    <xacro:property name="torso_back_offset" value="0.02"/>
+    <xacro:property name="torso_height" value="0.3" />
+    <xacro:property name="torso_width" value="0.4" />
+    <xacro:property name="torso_thickness" value="0.19" />
+    <xacro:property name="torso_back_offset" value="0.02" />
+    <xacro:property name="torso_shoulder_z_offset" value="0.03" />
+    <xacro:property name="torso_shoulder_height" value="0.2" />
+    <xacro:property name="torso_shoulder_width" value="0.2" />
+    <xacro:property name="torso_shoulder_thickness" value="0.02" />
     <xacro:include filename="$(find freddy_base_description)/urdf/common.xacro" />
     <xacro:include filename="$(find freddy_base_description)/urdf/freddy_base.urdf.xacro" />
@@ -11,19 +15,25 @@
         <!-- TORSO -->
         <joint name="${name}_joint" type="fixed">
-            <xacro:insert_block name="origin" />
-            <parent link="${parent}"/>
+            <origin
+                xyz="${-base_size_x/2 + torso_back_offset + torso_thickness/2} 0 ${wheel_slit_height + base_size_z}"
+                rpy="0 0 0" />
+            <parent link="${parent}" />
             <child link="${name}_link" />
         </joint>
         <link name="${name}_link">
             <visual>
-                <origin xyz="${-base_size_x/2 + torso_back_offset + torso_thickness/2} 0 ${wheel_slit_height + base_size_z + torso_height/2}" rpy="0 0 0"/>
+                <origin
+                    xyz="0 0 ${torso_height/2}"
+                    rpy="0 0 0" />
                 <geometry>
                     <box size="${torso_thickness} ${torso_width} ${torso_height}" />
                 </geometry>
-                <material name="DarkGrey"/>
+                <material name="Grey" />
             </visual>
             <!-- torso collision -->
             <collision>
-                <origin xyz="${-base_size_x/2 + torso_back_offset + torso_thickness/2} 0 ${wheel_slit_height + base_size_z + torso_height/2}" rpy="0 0 0"/>
+                <origin
+                    xyz="0 0 ${torso_height/2}"
+                    rpy="0 0 0" />
                 <geometry>
                     <box size="${torso_thickness} ${torso_width} ${torso_height}" />
@@ -31,6 +41,86 @@
             </collision>
             <xacro:cuboid_inertia mass="${base_mass}" length="${base_size_x}"
-                                  breadth="${base_size_y}" height="${base_size_z}"/>
+                breadth="${base_size_y}" height="${base_size_z}" />
         </link>
+        <!-- TORSO SHOULDER LEFT -->
+        <joint name="${name}_shoulder_left_joint" type="fixed">
+            <origin
+                xyz="${torso_thickness/2 - torso_shoulder_thickness/2} 0 ${torso_height - torso_shoulder_z_offset}"
+                rpy="0. 0.1309 0.7853982" />
+            <parent link="${name}_link" />
+            <child link="${name}_shoulder_left_link" />
+        </joint>
+        <link name="${name}_shoulder_left_link">
+            <visual>
+                <origin
+                    xyz="0 ${torso_shoulder_width/2} ${torso_shoulder_height/2}"
+                    rpy="0 0 0" />
+                <geometry>
+                    <box
+                        size="${torso_shoulder_thickness} ${torso_shoulder_width} ${torso_shoulder_height}" />
+                </geometry>
+                <material name="Grey" />
+            </visual>
+            <!-- torso shoulder collision -->
+            <collision>
+                <origin
+                    xyz="0 0 ${-torso_shoulder_thickness/2}"
+                    rpy="0 0 0" />
+                <geometry>
+                    <box
+                        size="${torso_shoulder_thickness} ${torso_shoulder_width} ${torso_shoulder_height}" />
+                </geometry>
+            </collision>
+            <xacro:cuboid_inertia mass="${base_mass}" length="${base_size_x}"
+                breadth="${base_size_y}" height="${base_size_z}" />
+        </link>
+        <joint name="${name}_shoulder_left_arm_joint" type="fixed">
+            <origin
+                xyz="0 ${torso_shoulder_width/2} ${torso_shoulder_height/2}"
+                rpy="3.14159 -1.5708 0" />
+            <parent link="${name}_shoulder_left_link" />
+            <child link="${name}_shoulder_left_arm_attach_link" />
+        </joint>
+        <link name="${name}_shoulder_left_arm_attach_link" />
+        <!-- TORSO SHOULDER RIGHT -->
+        <joint name="${name}_shoulder_right_joint" type="fixed">
+            <origin
+                xyz="${torso_thickness/2 - torso_shoulder_thickness/2} 0 ${torso_height - torso_shoulder_z_offset}"
+                rpy="0 0.1309 -0.7853982" />
+            <parent link="${name}_link" />
+            <child link="${name}_shoulder_right_link" />
+        </joint>
+        <link name="${name}_shoulder_right_link">
+            <visual>
+                <origin
+                    xyz="0 ${-torso_shoulder_width/2} ${torso_shoulder_height/2}"
+                    rpy="0 0 0" />
+                <geometry>
+                    <box
+                        size="${torso_shoulder_thickness} ${torso_shoulder_width} ${torso_shoulder_height}" />
+                </geometry>
+                <material name="Grey" />
+            </visual>
+            <!-- torso shoulder collision -->
+            <collision>
+                <origin
+                    xyz="0 0 ${-torso_shoulder_thickness/2}"
+                    rpy="0 0 0" />
+                <geometry>
+                    <box
+                        size="${torso_shoulder_thickness} ${torso_shoulder_width} ${torso_shoulder_height}" />
+                </geometry>
+            </collision>
+            <xacro:cuboid_inertia mass="${base_mass}" length="${base_size_x}"
+                breadth="${base_size_y}" height="${base_size_z}" />
+        </link>
+        <joint name="${name}_shoulder_right_arm_joint" type="fixed">
+            <origin
+                xyz="0 ${-torso_shoulder_width/2} ${torso_shoulder_height/2}"
+                rpy="3.14159 -1.5708 0" />
+            <parent link="${name}_shoulder_right_link" />
+            <child link="${name}_shoulder_right_arm_attach_link" />
+        </joint>
+        <link name="${name}_shoulder_right_arm_attach_link" />
         <gazebo reference="${name}_link">
             <material>Gazebo/RustySteel</material>
