Commit message: Add joint friction and damping

File: freddy_base_description/urdf/kelo_double_wheel_gz.urdf.xacro (robot description, xacro)
@@ -6,4 +6,6 @@
   <xacro:property name="wheel_mass" value="1.0"/>
   <xacro:property name="wheel_inertia" value="0.001"/>
+  <xacro:property name="joint_friction" value="0.2"/>
+  <xacro:property name="joint_damping" value="0.2"/>
   <xacro:property name="pivot_height" value="0.1"/>
   <xacro:property name="pivot_radius" value="0.02"/>
@@ -70,4 +72,5 @@
       <xacro:insert_block name="origin" />
       <axis xyz="0 0 1"/>
+      <dynamics damping="${joint_damping}" friction="${joint_friction}"/>
     </joint>
     <!-- Joint between left wheel hub and pivot -->
@@ -78,5 +81,5 @@
       <axis xyz="0 0 1"/>
       <!-- <limit effort="1000.0" lower="-15" upper="15" velocity="30"/> -->
-      <dynamics damping="0.0" friction="0.0"/>
+      <dynamics damping="${joint_damping}" friction="${joint_friction}"/>
     </joint>
     <!-- Joint between right wheel hub and pivot -->
@@ -87,5 +90,5 @@
       <axis xyz="0 0 1"/>
       <!-- <limit effort="1000.0" lower="-15" upper="15" velocity="30"/> -->
-      <dynamics damping="0.0" friction="0.0"/>
+      <dynamics damping="${joint_damping}" friction="${joint_friction}"/>
     </joint>
     <!-- ros2 control tags -->
