Commit message: Update and refactor xacros

File: freddy_base_description/urdf/freddy_base_gz.urdf.xacro (robot description, xacro)
@@ -11,23 +11,7 @@
     <xacro:property name="base_size_z" value="${base_size_z_bottom + laser_slit_height + base_size_z_top}"/>
     <xacro:property name="base_mass" value="40.0"/>
-    <!-- <xacro:include filename="$(find freddy_base_description)/urdf/sensors/hokuyo.urdf.xacro" /> -->
     <xacro:include filename="$(find freddy_base_description)/urdf/kelo_wheel_gz.urdf.xacro" />
     <xacro:macro name="freddy_base" params="name parent *origin use_gpu_2d_laser:=true">
-        <!-- HOLONOMIC DRIVE PLUGIN -->
-        <!-- <gazebo>
-            <plugin name="gazebo_ros_planar_move" filename="libgazebo_ros_planar_move.so">
-            <commandTopic>cmd_vel</commandTopic>
-            <odometryTopic>odom</odometryTopic>
-            <odometryFrame>odom</odometryFrame>
-            <odometryRate>20.0</odometryRate>
-            <robotBaseFrame>${parent}</robotBaseFrame>
-            </plugin>
-        </gazebo> -->
         <!-- BASE -->
-        <joint name="${name}_joint" type="fixed">
-            <xacro:insert_block name="origin" />
-            <parent link="${parent}"/>
-            <child link="${name}_link" />
-        </joint>
         <link name="${name}_link">
             <visual>
@@ -36,19 +20,4 @@
                     <box size="${base_size_x} ${base_size_y} ${base_size_z_bottom}" />
                 </geometry>
-                <material name="DarkGrey"/>
-            </visual>
-            <visual>
-                <origin xyz="0 0 ${wheel_slit_height + base_size_z_bottom + laser_slit_height/2}" rpy="0 0 0"/>
-                <geometry>
-                    <box size="${base_size_x*0.7} ${base_size_y*0.7} ${laser_slit_height}" />
-                </geometry>
-                <material name="DarkGrey"/>
-            </visual>
-            <visual>
-                <origin xyz="0 0 ${wheel_slit_height + base_size_z_bottom + laser_slit_height + base_size_z_top/2}" rpy="0 0 0"/>
-                <geometry>
-                    <box size="${base_size_x} ${base_size_y} ${base_size_z_top}" />
-                </geometry>
-                <material name="DarkGrey"/>
             </visual>
             <!-- base bottom collisions -->
@@ -69,9 +38,11 @@
                                   breadth="${base_size_y}" height="${base_size_z}"/>
         </link>
-        <gazebo reference="${name}_link">
-            <material>Gazebo/RustySteel</material>
-        </gazebo>
+        <joint name="${name}_joint" type="fixed">
+            <xacro:insert_block name="origin" />
+            <parent link="${parent}"/>
+            <child link="${name}_link" />
+        </joint>
         <!-- WHEELS -->
-        <xacro:kelo_wheel name="left_front_wheel" parent="${name}_link" material_name="Black">
+        <xacro:kelo_wheel name="left_front_wheel" parent="${name}_link" >
             <origin xyz="${base_size_x*0.5 - wheel_radius}
                          ${base_size_y*0.5 - wheel_radius}
@@ -79,5 +50,5 @@
                     rpy="0 0 0"/>
         </xacro:kelo_wheel>
-        <xacro:kelo_wheel name="right_front_wheel" parent="${name}_link" material_name="Black">
+        <xacro:kelo_wheel name="right_front_wheel" parent="${name}_link" >
             <origin xyz="${base_size_x*0.5 - wheel_radius}
                          ${-(base_size_y*0.5 - wheel_radius)}
@@ -85,5 +56,5 @@
                     rpy="0 0 0"/>
         </xacro:kelo_wheel>
-        <xacro:kelo_wheel name="left_back_wheel" parent="${name}_link" material_name="Black">
+        <xacro:kelo_wheel name="left_back_wheel" parent="${name}_link" >
             <origin xyz="${-(base_size_x*0.5 - wheel_radius)}
                          ${base_size_y*0.5 - wheel_radius}
@@ -91,5 +62,5 @@
                     rpy="0 0 0"/>
         </xacro:kelo_wheel>
-        <xacro:kelo_wheel name="right_back_wheel" parent="${name}_link" material_name="Black">
+        <xacro:kelo_wheel name="right_back_wheel" parent="${name}_link" >
             <origin xyz="${-(base_size_x*0.5 - wheel_radius)}
                          ${-(base_size_y*0.5 - wheel_radius)}
@@ -97,28 +68,4 @@
                     rpy="0 0 0"/>
         </xacro:kelo_wheel>
-        <!-- HOKUYO LASER -->
-        <!-- <xacro:if value="$(arg load_sensors)">
-        <xacro:hokuyo name="base_laser_front" parent="${name}_link"
-                           topic="/${robot_name}/base_scan_front" use_gpu="${use_gpu_2d_laser}">
-            <origin xyz="0.26 -0.24 0.25" rpy="${pi} 0 ${-pi/4}"/>
-        </xacro:hokuyo>
-        <xacro:hokuyo name="base_laser_back" parent="${name}_link"
-                           topic="/${robot_name}/base_scan_back" use_gpu="${use_gpu_2d_laser}">
-            <origin xyz="-0.26 0.24 0.25" rpy="${pi} 0 ${3*pi/4}"/>
-        </xacro:hokuyo>
-        </xacro:if> -->
-        <!-- VELOCITY CONTROL GZ PLUGIN -->
-        <!-- <xacro:if value="$(arg sim_gz)"> -->
-        <!-- <gazebo>
-            <plugin
-                filename="gz-sim-velocity-control-system"
-                name="gz::sim::systems::VelocityControl">
-            modified
-            <topic>cmd_vel</topic>
-            <link_name>base_link</link_name>
-            gz added
-            </plugin>
-        </gazebo> -->
-        <!-- </xacro:if> -->
     </xacro:macro>
 </robot>

File: freddy_base_description/urdf/kelo_wheel_gz.urdf.xacro (robot description, xacro)
@@ -5,14 +5,5 @@
     <xacro:property name="inertia_wheels" value="0.001" />
     <xacro:include filename="$(find freddy_base_description)/urdf/common.xacro" />
-    <xacro:macro name="kelo_wheel" params="name parent *origin material_name">
-        <joint name="${name}_joint" type="revolute">
-            <xacro:insert_block name="origin" />
-            <parent link="${parent}"/>
-            <child link="${name}_link"/>
-            <!-- Joint axis and limits (revolute) -->
-            <axis xyz="0 0 1" />
-            <limits effort="1000" velocity="10" lower="-1.79769e+308" upper="1.79769e+308" />
-            <!-- Joint axis and limits  -->
-        </joint>
+    <xacro:macro name="kelo_wheel" params="name parent *origin">
         <link name="${name}_link">
             <visual>
@@ -20,5 +11,4 @@
                     <sphere radius="${wheel_radius}" />
                 </geometry>
-                <material name="${material_name}"/>
             </visual>
             <collision>
@@ -29,9 +19,14 @@
             <xacro:sphere_inertia mass="${wheel_mass}" radius="${wheel_radius}" />
         </link>
-        <gazebo reference="${name}_link">
-            <mu1>0.0</mu1>
-            <mu2>0.0</mu2>
-            <material>Gazebo/Black</material>
-        </gazebo>
+        <joint name="${name}_joint" type="revolute">
+            <xacro:insert_block name="origin" />
+            <parent link="${parent}"/>
+            <child link="${name}_link"/>
+            <!-- Joint axis and limits (revolute) -->
+            <axis xyz="0 1 0" />
+            <limit effort="1000" velocity="100" lower="-1.79769e+308" upper="1.79769e+308" />
+            <dynamics damping="0.7"/>
+            <!-- Joint axis and limits  -->
+        </joint>
     </xacro:macro>
 </robot>

File: freddy_base_description/urdf/kelo_wheel_old_gz.urdf.xacro (robot description, xacro)
@@ -5,5 +5,14 @@
     <xacro:property name="inertia_wheels" value="0.001" />
     <xacro:include filename="$(find freddy_base_description)/urdf/common.xacro" />
-    <xacro:macro name="kelo_wheel" params="name parent *origin">
+    <xacro:macro name="kelo_wheel" params="name parent *origin material_name">
+        <joint name="${name}_joint" type="revolute">
+            <xacro:insert_block name="origin" />
+            <parent link="${parent}"/>
+            <child link="${name}_link"/>
+            <!-- Joint axis and limits (revolute) -->
+            <axis xyz="0 0 1" />
+            <limits effort="1000" velocity="10" lower="-1.79769e+308" upper="1.79769e+308" />
+            <!-- Joint axis and limits  -->
+        </joint>
         <link name="${name}_link">
             <visual>
@@ -11,4 +20,5 @@
                     <sphere radius="${wheel_radius}" />
                 </geometry>
+                <material name="${material_name}"/>
             </visual>
             <collision>
@@ -19,14 +29,9 @@
             <xacro:sphere_inertia mass="${wheel_mass}" radius="${wheel_radius}" />
         </link>
-        <joint name="${name}_joint" type="revolute">
-            <xacro:insert_block name="origin" />
-            <parent link="${parent}"/>
-            <child link="${name}_link"/>
-            <!-- Joint axis and limits (revolute) -->
-            <axis xyz="0 1 0" />
-            <limit effort="1000" velocity="100" lower="-1.79769e+308" upper="1.79769e+308" />
-            <dynamics damping="0.7"/>
-            <!-- Joint axis and limits  -->
-        </joint>
+        <gazebo reference="${name}_link">
+            <mu1>0.0</mu1>
+            <mu2>0.0</mu2>
+            <material>Gazebo/Black</material>
+        </gazebo>
     </xacro:macro>
 </robot>

File: freddy_description/robots/freddy_gz.urdf.xacro (robot description, xacro)
@@ -2,52 +2,8 @@
 <robot xmlns:xacro="http://www.ros.org/wiki/xacro" name="freddy">
     <xacro:arg name="use_gpu_2d_laser" default="false" />
-    <!-- Arguments -->
-    <xacro:arg name="prefix_arm_left" default="kinova_left_" />
-    <xacro:arg name="prefix_arm_right" default="kinova_right_" />
-    <!-- Robot prefix -->
+    <!-- Robot tf_prefix -->
     <xacro:arg name="tf_prefix" default="" />
-    <!-- Load arms and sensors -->
-    <xacro:arg name="load_arms" default="false" />
-    <xacro:arg name="load_sensors" default="false" />
-    <xacro:arg name="arm" default="gen3" />
-    <xacro:arg name="dof" default="7" />
-    <xacro:arg name="vision" default="true" />
-    <xacro:arg name="robot_ip_left" default="192.168.1.10" />
-    <xacro:arg name="robot_ip_right" default="192.168.1.11" />
-    <xacro:arg name="username" default="admin" />
-    <xacro:arg name="password" default="admin" />
-    <xacro:arg name="port" default="10000" />
-    <xacro:arg name="port_realtime" default="10001" />
-    <xacro:arg name="session_inactivity_timeout_ms" default="60000" />
-    <xacro:arg name="connection_inactivity_timeout_ms" default="2000" />
-    <xacro:arg name="gripper" default="robotiq_2f_85" />
-    <xacro:arg name="gripper_joint_name" default="finger_joint" />
-    <xacro:arg name="gripper_max_velocity" default="100.0" />
-    <xacro:arg name="gripper_max_force" default="100.0" />
-    <xacro:arg name="use_internal_bus_gripper_comm" default="false" />
-    <xacro:arg name="use_fake_hardware" default="false" />
-    <xacro:arg name="fake_sensor_commands" default="false" />
-    <xacro:arg name="sim_gazebo" default="false" />
-    <xacro:arg name="sim_gz" default="false" />
-    <xacro:arg name="sim_ignition" default="false" />
-    <xacro:arg name="sim_isaac" default="false" />
-    <xacro:arg name="gazebo_renderer" default="ogre" />
-    <xacro:arg name="camera_width" default="640" />
-    <xacro:arg name="camera_height" default="480" />
-    <xacro:arg name="camera_fps" default="6" />
-    <!-- <xacro:arg name="simulation_controllers" -->
-        <!-- default="$(find kortex_description)/arm/$(arg arm)/$(arg dof)dof/config/ros2_controllers.yaml" /> -->
-    <!-- <xacro:arg name="base_controller"
-        default="$(find freddy_gazebo)/config/base_controller.yaml" /> -->
-    <xacro:include filename="$(find freddy_base_description)/urdf/materials.urdf.xacro" />
+    <xacro:include filename="$(find freddy_base_description)/urdf/common.xacro" />
     <xacro:include filename="$(find freddy_base_description)/urdf/freddy_base_gz.urdf.xacro" />
-    <xacro:include filename="$(find freddy_torso_description)/urdf/freddy_torso_gz.urdf.xacro" />
-    <!-- <xacro:include filename="$(find kortex_description)/robots/kortex_robot.xacro" /> -->
-    <!-- <xacro:include filename="$(find freddy_description)/ros2_control/freddy_gz.ros2_control.xacro" /> -->
-    <!-- initial position for simulations (Mock Hardware, Gazebo, Ignition) -->
-    <xacro:arg name="initial_positions_file"
-        default="$(find freddy_description)/config/initial_positions.yaml" />
-    <!-- convert to property to use substitution in function -->
-    <xacro:property name="initial_positions_file" default="$(arg initial_positions_file)" />
     <link name="base_link"/>
     <xacro:freddy_base name="freddy_base" parent="base_link"
@@ -55,175 +11,13 @@
         <origin xyz="0.0 0.0 0.0" rpy="0.0 0.0 0.0" />
     </xacro:freddy_base>
-    <xacro:freddy_torso name="freddy_torso" parent="base_link">
-        <origin xyz="0.0 0.0 0.0" rpy="0.0 0.0 0.0" />
-    </xacro:freddy_torso>
-    <!-- arms -->
-    <!-- Load arms if argument true -->
-    <xacro:if value="$(arg load_arms)">
-    <!-- left arm -->
-    <xacro:load_robot
-        parent="freddy_torso_shoulder_left_arm_attach_link"
-        arm="$(arg arm)"
-        gripper="$(arg gripper)"
-        gripper_joint_name="$(arg gripper_joint_name)"
-        gripper_max_velocity="$(arg gripper_max_velocity)"
-        gripper_max_force="$(arg gripper_max_force)"
-        dof="$(arg dof)"
-        vision="$(arg vision)"
-        robot_ip="$(arg robot_ip_left)"
-        username="$(arg username)"
-        password="$(arg password)"
-        port="$(arg port)"
-        port_realtime="$(arg port_realtime)"
-        session_inactivity_timeout_ms="$(arg session_inactivity_timeout_ms)"
-        connection_inactivity_timeout_ms="$(arg connection_inactivity_timeout_ms)"
-        use_internal_bus_gripper_comm="$(arg use_internal_bus_gripper_comm)"
-        prefix="$(arg prefix_arm_left)"
-        use_fake_hardware="$(arg use_fake_hardware)"
-        fake_sensor_commands="$(arg fake_sensor_commands)"
-        sim_gazebo="$(arg sim_gazebo)"
-        sim_ignition="$(arg sim_ignition)"
-        sim_isaac="$(arg sim_isaac)"
-        initial_positions="${xacro.load_yaml(initial_positions_file)}">
-        <origin xyz="0 0 0" rpy="0 0 0" />
-    </xacro:load_robot>
-    <!-- right arm -->
-    <xacro:load_robot
-        parent="freddy_torso_shoulder_right_arm_attach_link"
-        arm="$(arg arm)"
-        gripper="$(arg gripper)"
-        gripper_joint_name="$(arg gripper_joint_name)"
-        gripper_max_velocity="$(arg gripper_max_velocity)"
-        gripper_max_force="$(arg gripper_max_force)"
-        dof="$(arg dof)"
-        vision="$(arg vision)"
-        robot_ip="$(arg robot_ip_right)"
-        username="$(arg username)"
-        password="$(arg password)"
-        port="$(arg port)"
-        port_realtime="$(arg port_realtime)"
-        session_inactivity_timeout_ms="$(arg session_inactivity_timeout_ms)"
-        connection_inactivity_timeout_ms="$(arg connection_inactivity_timeout_ms)"
-        use_internal_bus_gripper_comm="$(arg use_internal_bus_gripper_comm)"
-        prefix="$(arg prefix_arm_right)"
-        use_fake_hardware="$(arg use_fake_hardware)"
-        fake_sensor_commands="$(arg fake_sensor_commands)"
-        sim_gazebo="$(arg sim_gazebo)"
-        sim_ignition="$(arg sim_ignition)"
-        sim_isaac="$(arg sim_isaac)"
-        initial_positions="${xacro.load_yaml(initial_positions_file)}">
-        <origin xyz="0 0 0" rpy="0 0 0" />
-    </xacro:load_robot>
-    <!-- grasp links -->
-    <link name="kinova_left_grasp_link" />
-    <link name="kinova_right_grasp_link" />
-    <!-- grasp link joints -->
-    <joint name="kinova_left_grasp_link_joint" type="fixed">
-        <origin xyz="0 0 0.15" rpy="0 0 0" />
-        <parent link="kinova_left_robotiq_85_base_link" />
-        <child link="kinova_left_grasp_link" />
-    </joint>
-    <joint name="kinova_right_grasp_link_joint" type="fixed">
-        <origin xyz="0 0 0.15" rpy="0 0 0" />
-        <parent link="kinova_right_robotiq_85_base_link" />
-        <child link="kinova_right_grasp_link" />
-    </joint>
-    <!-- Load arms end -->
-    </xacro:if>
-    <!-- <xacro:if value="$(arg sim_gazebo)">
-        <gazebo reference="world">
-        </gazebo>
-        <gazebo>
-            <plugin name="ros_gz_control" filename="libros_gz_control.so">
-                <parameters>$(arg simulation_controllers)</parameters>
-            </plugin>
-        </gazebo>
-    </xacro:if> -->
-    <!-- Modified for Gazebo Harmonic -->
-    <!-- <xacro:if value="$(arg sim_gz)">
-        <gazebo reference="world">
-        </gazebo>
-        <gazebo>
-            <plugin filename="libgz_ros2_control-system" name="gz_ros2_control::GazeboSimROS2ControlPlugin">
-                <parameters>$(arg base_controller)</parameters>
-            </plugin>
-        </gazebo>
-    </xacro:if> -->
-    <!-- TODO: Verify if the below snippet works for dual arm setup -->
-    <!-- <xacro:if value="$(arg sim_ignition)">
-        <gazebo reference="world">
-        </gazebo>
-        <gazebo>
-            <plugin filename="libign_ros2_control-system.so"
-                name="ign_ros2_control::IgnitionROS2ControlPlugin">
-                <parameters>$(arg simulation_controllers)</parameters>
-                <controller_manager_node_name>$(arg prefix)controller_manager</controller_manager_node_name>
-            </plugin>
-            <plugin filename="libignition-gazebo-sensors-system.so"
-                name="ignition::gazebo::systems::Sensors">
-                <render_engine>$(arg gazebo_renderer)</render_engine>
-            </plugin>
-        </gazebo>
-        <gazebo reference="camera_color_frame">
-            <sensor name="camera_sensor" type="rgbd_camera">
-                <camera>
-                    <horizontal_fov>1.047</horizontal_fov>
-                    <image>
-                        <width>$(arg camera_width)</width>
-                        <height>$(arg camera_height)</height>
-                        <format>RGB_INT8</format>
-                    </image>
-                    <clip>
-                        <near>0.1</near>
-                        <far>5</far>
-                    </clip>
-                    <distortion>
-                        <k1>0.0</k1>
-                        <k2>0.0</k2>
-                        <k3>0.0</k3>
-                        <p1>0.0</p1>
-                        <p2>0.0</p2>
-                        <center>0.5 0.5</center>
-                    </distortion>
-                    <lens>
-                        <intrinsics>
-                            <fx>554.25469</fx>
-                            <fy>554.25469</fy>
-                            <cx>320.5</cx>
-                            <cy>240.5</cy>
-                            <s>0</s>
-                        </intrinsics>
-                        <projection>
-                            <p_fx>554.25469</p_fx>
-                            <p_fy>554.25469</p_fy>
-                            <p_cx>320.5</p_cx>
-                            <p_cy>240.5</p_cy>
-                            <tx>0</tx>
-                            <ty>0</ty>
-                        </projection>
-                    </lens>
-                    <noise>
-                        <type>gaussian</type>
-                        <mean>0</mean>
-                        <stddev>0.00</stddev>
-                    </noise>
-                    <depth_camera>
-                        <clip>
-                            <near>0.25</near>
-                            <far>5</far>
-                        </clip>
-                    </depth_camera>
-                    <optical_frame_id>color_optical_frame</optical_frame_id>
-                </camera>
-                <ignition_frame_id>camera_color_frame</ignition_frame_id>
-                <always_on>1</always_on>
-                <update_rate>$(arg camera_fps)</update_rate>
-                <visualize>true</visualize>
-                <topic>wrist_mounted_camera</topic>
-                <enable_metrics>false</enable_metrics>
-            </sensor>
-        </gazebo>
-    </xacro:if> -->
-    <!-- <xacro:freddy_ros2_control
-    name="FreddyROS2Control" tf_prefix="$(arg tf_prefix)" type="actuator" /> -->
+    <gazebo>
+    <plugin
+        filename="gz-sim-velocity-control-system"
+        name="gz::sim::systems::VelocityControl">
+        <initial_linear>0.0 0 0</initial_linear>
+        <initial_angular>0 0 0.0</initial_angular>
+        <!-- <link_name>base_link</link_name> -->
+        <!-- <topic>cmd_vel</topic> -->
+    </plugin>
+    </gazebo>
 </robot>
