Commit message: Add back robot torso

File: freddy_base_description/urdf/freddy_base_gz.urdf.xacro (robot description, xacro)
@@ -13,4 +13,15 @@
     <xacro:include filename="$(find freddy_base_description)/urdf/kelo_wheel_gz.urdf.xacro" />
     <xacro:macro name="freddy_base" params="name parent *origin use_gpu_2d_laser:=true">
+        <!-- VELOCITY CONTROL PLUGIN -->
+        <gazebo>
+            <plugin
+                filename="gz-sim-velocity-control-system"
+                name="gz::sim::systems::VelocityControl">
+                <initial_linear>0.0 0 0</initial_linear>
+                <initial_angular>0 0 0.0</initial_angular>
+                <!-- <link_name>base_link</link_name> -->
+                <!-- <topic>cmd_vel</topic> -->
+            </plugin>
+        </gazebo>
         <!-- BASE -->
         <link name="${name}_link">
@@ -19,4 +30,16 @@
                 <geometry>
                     <box size="${base_size_x} ${base_size_y} ${base_size_z_bottom}" />
+                </geometry>
+            </visual>
+            <visual>
+                <origin xyz="0 0 ${wheel_slit_height + base_size_z_bottom + laser_slit_height/2}" rpy="0 0 0"/>
+                <geometry>
+                    <box size="${base_size_x*0.7} ${base_size_y*0.7} ${laser_slit_height}" />
+                </geometry>
+            </visual>
+            <visual>
+                <origin xyz="0 0 ${wheel_slit_height + base_size_z_bottom + laser_slit_height + base_size_z_top/2}" rpy="0 0 0"/>
+                <geometry>
+                    <box size="${base_size_x} ${base_size_y} ${base_size_z_top}" />
                 </geometry>
             </visual>

File: freddy_description/robots/freddy_gz.urdf.xacro (robot description, xacro)
@@ -6,4 +6,5 @@
     <xacro:include filename="$(find freddy_base_description)/urdf/common.xacro" />
     <xacro:include filename="$(find freddy_base_description)/urdf/freddy_base_gz.urdf.xacro" />
+    <xacro:include filename="$(find freddy_torso_description)/urdf/freddy_torso_gz.urdf.xacro" />
     <link name="base_link"/>
     <xacro:freddy_base name="freddy_base" parent="base_link"
@@ -11,13 +12,6 @@
         <origin xyz="0.0 0.0 0.0" rpy="0.0 0.0 0.0" />
     </xacro:freddy_base>
-    <gazebo>
-    <plugin
-        filename="gz-sim-velocity-control-system"
-        name="gz::sim::systems::VelocityControl">
-        <initial_linear>0.0 0 0</initial_linear>
-        <initial_angular>0 0 0.0</initial_angular>
-        <!-- <link_name>base_link</link_name> -->
-        <!-- <topic>cmd_vel</topic> -->
-    </plugin>
-    </gazebo>
+    <xacro:freddy_torso name="freddy_torso" parent="base_link">
+        <origin xyz="0.0 0.0 0.0" rpy="0.0 0.0 0.0" />
+    </xacro:freddy_torso>
 </robot>

Commit message: Add double wheel kelo drive

File: freddy_base_description/urdf/freddy_base_gz.urdf.xacro (robot description, xacro)
@@ -11,17 +11,6 @@
     <xacro:property name="base_size_z" value="${base_size_z_bottom + laser_slit_height + base_size_z_top}"/>
     <xacro:property name="base_mass" value="40.0"/>
-    <xacro:include filename="$(find freddy_base_description)/urdf/kelo_wheel_gz.urdf.xacro" />
+    <xacro:include filename="$(find freddy_base_description)/urdf/kelo_double_wheel_gz.urdf.xacro" />
     <xacro:macro name="freddy_base" params="name parent *origin use_gpu_2d_laser:=true">
-        <!-- VELOCITY CONTROL PLUGIN -->
-        <gazebo>
-            <plugin
-                filename="gz-sim-velocity-control-system"
-                name="gz::sim::systems::VelocityControl">
-                <initial_linear>0.0 0 0</initial_linear>
-                <initial_angular>0 0 0.0</initial_angular>
-                <!-- <link_name>base_link</link_name> -->
-                <!-- <topic>cmd_vel</topic> -->
-            </plugin>
-        </gazebo>
         <!-- BASE -->
         <link name="${name}_link">
@@ -67,28 +56,28 @@
         </joint>
         <!-- WHEELS -->
-        <xacro:kelo_wheel name="left_front_wheel" parent="${name}_link" >
+        <xacro:kelo_drive name="kelo_drive_front_left" parent="${name}_link" >
             <origin xyz="${base_size_x*0.5 - wheel_radius}
                          ${base_size_y*0.5 - wheel_radius}
                          ${wheel_radius}"
                     rpy="0 0 0"/>
-        </xacro:kelo_wheel>
-        <xacro:kelo_wheel name="right_front_wheel" parent="${name}_link" >
+        </xacro:kelo_drive>
+        <xacro:kelo_drive name="kelo_drive_front_right" parent="${name}_link" >
             <origin xyz="${base_size_x*0.5 - wheel_radius}
                          ${-(base_size_y*0.5 - wheel_radius)}
                          ${wheel_radius}"
                     rpy="0 0 0"/>
-        </xacro:kelo_wheel>
-        <xacro:kelo_wheel name="left_back_wheel" parent="${name}_link" >
+        </xacro:kelo_drive>
+        <xacro:kelo_drive name="kelo_drive_rear_right" parent="${name}_link" >
             <origin xyz="${-(base_size_x*0.5 - wheel_radius)}
                          ${base_size_y*0.5 - wheel_radius}
                          ${wheel_radius}"
                     rpy="0 0 0"/>
-        </xacro:kelo_wheel>
-        <xacro:kelo_wheel name="right_back_wheel" parent="${name}_link" >
+        </xacro:kelo_drive>
+        <xacro:kelo_drive name="kelo_drive_rear_left" parent="${name}_link" >
             <origin xyz="${-(base_size_x*0.5 - wheel_radius)}
                          ${-(base_size_y*0.5 - wheel_radius)}
                          ${wheel_radius}"
                     rpy="0 0 0"/>
-        </xacro:kelo_wheel>
+        </xacro:kelo_drive>
     </xacro:macro>
 </robot>

File: freddy_description/robots/freddy_gz.urdf.xacro (robot description, xacro)
@@ -1,17 +1,32 @@
 <?xml version='1.0'?>
 <robot xmlns:xacro="http://www.ros.org/wiki/xacro" name="freddy">
-    <xacro:arg name="use_gpu_2d_laser" default="false" />
-    <!-- Robot tf_prefix -->
-    <xacro:arg name="tf_prefix" default="" />
-    <xacro:include filename="$(find freddy_base_description)/urdf/common.xacro" />
-    <xacro:include filename="$(find freddy_base_description)/urdf/freddy_base_gz.urdf.xacro" />
-    <xacro:include filename="$(find freddy_torso_description)/urdf/freddy_torso_gz.urdf.xacro" />
-    <link name="base_link"/>
-    <xacro:freddy_base name="freddy_base" parent="base_link"
-        use_gpu_2d_laser="$(arg use_gpu_2d_laser)">
-        <origin xyz="0.0 0.0 0.0" rpy="0.0 0.0 0.0" />
-    </xacro:freddy_base>
-    <xacro:freddy_torso name="freddy_torso" parent="base_link">
-        <origin xyz="0.0 0.0 0.0" rpy="0.0 0.0 0.0" />
-    </xacro:freddy_torso>
+  <xacro:arg name="use_gpu_2d_laser" default="false" />
+  <!-- Robot tf_prefix -->
+  <xacro:arg name="tf_prefix" default="" />
+  <xacro:include filename="$(find freddy_base_description)/urdf/common.xacro" />
+  <xacro:include filename="$(find freddy_base_description)/urdf/freddy_base_gz.urdf.xacro" />
+  <xacro:include filename="$(find freddy_torso_description)/urdf/freddy_torso_gz.urdf.xacro" />
+  <link name="base_link"/>
+  <xacro:freddy_base name="freddy_base" parent="base_link"
+    use_gpu_2d_laser="$(arg use_gpu_2d_laser)">
+    <origin xyz="0.0 0.0 0.0" rpy="0.0 0.0 0.0" />
+  </xacro:freddy_base>
+  <xacro:freddy_torso name="freddy_torso" parent="base_link">
+    <origin xyz="0.0 0.0 0.0" rpy="0.0 0.0 0.0" />
+  </xacro:freddy_torso>
+  <gazebo>
+    <!-- VELOCITY CONTROL PLUGIN -->
+    <plugin
+      filename="gz-sim-velocity-control-system"
+      name="gz::sim::systems::VelocityControl">
+      <initial_linear>0.0 0 0</initial_linear>
+      <initial_angular>0 0 0.0</initial_angular>
+      <!-- <link_name>base_link</link_name> -->
+      <!-- <topic>cmd_vel</topic> -->
+    </plugin>
+    <!-- Joint state publisher -->
+    <plugin filename="gz_ros2_control-system" name="gz_ros2_control::GazeboSimROS2ControlPlugin">
+      <parameters>$(find freddy_description)/config/ros2_controllers_double_wheel.yaml</parameters>
+    </plugin>
+  </gazebo>
 </robot>

Commit message: Add kelo drive; update xacros

File: freddy_base_description/urdf/freddy_base_gz.urdf.xacro (robot description, xacro)
@@ -47,5 +47,5 @@
                 </geometry>
             </collision>
-            <xacro:cuboid_inertia mass="${base_mass}" length="${base_size_x}"
+            <!-- <xacro:cuboid_inertia mass="${base_mass}" length="${base_size_x}" -->
                                   breadth="${base_size_y}" height="${base_size_z}"/>
         </link>

File: freddy_base_description/urdf/kelo_double_wheel_gz.urdf.xacro (robot description, xacro)
@@ -5,4 +5,5 @@
   <xacro:property name="wheel_separation" value="0.05"/>
   <xacro:property name="wheel_mass" value="1.0"/>
+  <xacro:property name="wheel_inertia" value="0.001"/>
   <xacro:property name="pivot_height" value="0.1"/>
   <xacro:property name="pivot_radius" value="0.02"/>
@@ -29,5 +30,5 @@
         <mass value="${wheel_mass}"/>
         <origin xyz="0 0 0" rpy="0 0 0"/>
-        <inertia ixx="0.1" ixy="0" ixz="0" iyy="0.1" iyz="0" izz="0.1"/>
+        <inertia ixx="${wheel_inertia}" ixy="0" ixz="0" iyy="${wheel_inertia}" iyz="0" izz="${wheel_inertia}"/>
       </inertial>
     </link>
@@ -54,5 +55,5 @@
         <mass value="${wheel_mass}"/>
         <origin xyz="0 0 0" rpy="0 0 0"/>
-        <inertia ixx="0.1" ixy="0" ixz="0" iyy="0.1" iyz="0" izz="0.1"/>
+        <inertia ixx="${wheel_inertia}" ixy="0" ixz="0" iyy="${wheel_inertia}" iyz="0" izz="${wheel_inertia}"/>
       </inertial>
     </link>

File: freddy_torso_description/urdf/freddy_torso_gz.urdf.xacro (robot description, xacro)
@@ -39,5 +39,5 @@
                 </geometry>
             </collision>
-            <xacro:cuboid_inertia mass="${base_mass}" length="${base_size_x}"
+            <xacro:cuboid_inertia mass="${base_mass/10000}" length="${base_size_x}"
                 breadth="${base_size_y}" height="${base_size_z}" />
         </link>
@@ -70,6 +70,6 @@
                 </geometry>
             </collision>
-            <xacro:cuboid_inertia mass="${base_mass}" length="${base_size_x}"
-                breadth="${base_size_y}" height="${base_size_z}" />
+            <!-- <xacro:cuboid_inertia mass="${base_mass}" length="${base_size_x}"
+                breadth="${base_size_y}" height="${base_size_z}" /> -->
         </link>
         <joint name="${name}_shoulder_left_arm_joint" type="fixed">
@@ -110,6 +110,6 @@
             </collision>
             <!-- This is causing the base to topple over under combined x y velocity -->
-            <xacro:cuboid_inertia mass="${base_mass}" length="${base_size_x}"
-                breadth="${base_size_y}" height="${base_size_z}" />
+            <!-- <xacro:cuboid_inertia mass="${base_mass}" length="${base_size_x}"
+                breadth="${base_size_y}" height="${base_size_z}" /> -->
         </link>
         <joint name="${name}_shoulder_right_arm_joint" type="fixed">

Commit message: Clean up and refactor

File: freddy_base_description/urdf/freddy_base_gz.urdf.xacro (robot description, xacro)
@@ -11,5 +11,5 @@
     <xacro:property name="base_size_z" value="${base_size_z_bottom + laser_slit_height + base_size_z_top}"/>
     <xacro:property name="base_mass" value="40.0"/>
-    <xacro:include filename="$(find freddy_base_description)/urdf/kelo_double_wheel_gz.urdf.xacro" />
+    <xacro:include filename="$(find freddy_base_description)/urdf/kelo_wheel_gz.urdf.xacro" />
     <xacro:macro name="freddy_base" params="name parent *origin use_gpu_2d_laser:=true">
         <!-- BASE -->

File: freddy_base_description/urdf/kelo_wheel_gz.urdf.xacro (robot description, xacro)
@@ -1,32 +1,147 @@
-<?xml version="1.0"?>
 <robot xmlns:xacro="http://www.ros.org/wiki/xacro">
-    <xacro:property name="wheel_radius" value="0.05" />
-    <xacro:property name="wheel_mass" value="1.0" />
-    <xacro:property name="inertia_wheels" value="0.001" />
-    <xacro:include filename="$(find freddy_base_description)/urdf/common.xacro" />
-    <xacro:macro name="kelo_wheel" params="name parent *origin">
-        <link name="${name}_link">
-            <visual>
-                <geometry>
-                    <sphere radius="${wheel_radius}" />
-                </geometry>
-            </visual>
-            <collision>
-                <geometry>
-                    <sphere radius="${wheel_radius}" />
-                </geometry>
-            </collision>
-            <xacro:sphere_inertia mass="${wheel_mass}" radius="${wheel_radius}" />
-        </link>
-        <joint name="${name}_joint" type="revolute">
-            <xacro:insert_block name="origin" />
-            <parent link="${parent}"/>
-            <child link="${name}_link"/>
-            <!-- Joint axis and limits (revolute) -->
-            <axis xyz="0 1 0" />
-            <limit effort="1000" velocity="100" lower="-1.79769e+308" upper="1.79769e+308" />
-            <dynamics damping="0.7"/>
-            <!-- Joint axis and limits  -->
-        </joint>
-    </xacro:macro>
+  <!-- Property definitions -->
+  <xacro:property name="wheel_radius" value="0.05"/>
+  <xacro:property name="wheel_length" value="0.05"/>
+  <xacro:property name="wheel_separation" value="0.05"/>
+  <xacro:property name="wheel_mass" value="1.0"/>
+  <xacro:property name="wheel_inertia" value="0.001"/>
+  <xacro:property name="joint_friction" value="0.2"/>
+  <xacro:property name="joint_damping" value="0.2"/>
+  <xacro:property name="pivot_height" value="0.1"/>
+  <xacro:property name="pivot_radius" value="0.02"/>
+  <xacro:property name="pivot_offset" value="0.01"/>
+  <!-- Pivot macro -->
+  <xacro:macro name="pivot" params="name">
+    <link name="${name}">
+      <visual>
+      <origin xyz="0 0 0" rpy="0 0 0"/>
+        <geometry>
+          <cylinder length="${pivot_height}" radius="${pivot_radius}"/>
+        </geometry>
+        <material name="grey">
+          <color rgba="0.25 0.25 0.25 1"/>
+        </material>
+      </visual>
+      <collision>
+      <origin xyz="0 0 0" rpy="0 0 0"/>
+        <geometry>
+          <cylinder length="${pivot_height}" radius="${pivot_radius}"/>
+        </geometry>
+      </collision>
+      <inertial>
+        <mass value="${wheel_mass}"/>
+        <origin xyz="0 0 0" rpy="0 0 0"/>
+        <inertia ixx="${wheel_inertia}" ixy="0" ixz="0" iyy="${wheel_inertia}" iyz="0" izz="${wheel_inertia}"/>
+      </inertial>
+    </link>
+  </xacro:macro>
+  <!-- Wheel macro -->
+  <xacro:macro name="wheel" params="name">
+    <link name="${name}">
+      <visual>
+      <origin xyz="0 0 0" rpy="0 0 0"/>
+        <geometry>
+          <cylinder length="${wheel_length}" radius="${wheel_radius}"/>
+        </geometry>
+        <material name="black">
+          <color rgba="0 0 0 1"/>
+        </material>
+      </visual>
+      <collision>
+      <origin xyz="0 0 0" rpy="0 0 0"/>
+        <geometry>
+          <cylinder length="${wheel_length}" radius="${wheel_radius}"/>
+        </geometry>
+      </collision>
+      <inertial>
+        <mass value="${wheel_mass}"/>
+        <origin xyz="0 0 0" rpy="0 0 0"/>
+        <inertia ixx="${wheel_inertia}" ixy="0" ixz="0" iyy="${wheel_inertia}" iyz="0" izz="${wheel_inertia}"/>
+      </inertial>
+    </link>
+  </xacro:macro>
+  <!-- Kelo drive macro -->
+  <xacro:macro name="kelo_drive" params="name parent *origin">
+    <xacro:pivot name="${name}_pivot"/>
+    <xacro:wheel name="${name}_hub_left"/>
+    <xacro:wheel name="${name}_hub_right"/>
+    <!-- Joint between pivot and chassis -->
+    <joint name="${name}_pivot_joint" type="continuous">
+      <parent link="${parent}"/>
+      <child link="${name}_pivot"/>
+      <xacro:insert_block name="origin" />
+      <axis xyz="0 0 1"/>
+      <dynamics damping="${joint_damping}" friction="${joint_friction}"/>
+    </joint>
+    <!-- Joint between left wheel hub and pivot -->
+    <joint name="${name}_hub_left_joint" type="continuous">
+      <parent link="${name}_pivot"/>
+      <child link="${name}_hub_left"/>
+      <origin xyz="-${pivot_offset} ${wheel_separation} -${base_size_z_bottom*0.5 - wheel_radius}" rpy="-1.5708 0 0"/>
+      <axis xyz="0 0 1"/>
+      <!-- <limit effort="1000.0" lower="-15" upper="15" velocity="30"/> -->
+      <dynamics damping="${joint_damping}" friction="${joint_friction}"/>
+    </joint>
+    <!-- Joint between right wheel hub and pivot -->
+    <joint name="${name}_hub_right_joint" type="continuous">
+      <parent link="${name}_pivot"/>
+      <child link="${name}_hub_right"/>
+      <origin xyz="-${pivot_offset} -${wheel_separation} -${base_size_z_bottom*0.5 - wheel_radius}" rpy="-1.5708 0 0"/>
+      <axis xyz="0 0 1"/>
+      <!-- <limit effort="1000.0" lower="-15" upper="15" velocity="30"/> -->
+      <dynamics damping="${joint_damping}" friction="${joint_friction}"/>
+    </joint>
+    <!-- ros2 control tags -->
+    <ros2_control name="${name}" type="system">
+      <hardware>
+        <plugin>gz_ros2_control/GazeboSimSystem</plugin>
+      </hardware>
+      <joint name="${name}_hub_left_joint">
+        <command_interface name="position">
+          <param name="min">-1e+100</param>
+          <param name="max">1e+100</param>
+        </command_interface>
+        <command_interface name="velocity">
+          <param name="min">-1e+100</param>
+          <param name="max">1e+100</param>
+        </command_interface>
+        <command_interface name="effort">
+          <param name="min">-1e+100</param>
+          <param name="max">1e+100</param>
+        </command_interface>
+        <state_interface name="position">
+           <param name="initial_value">0.0</param>
+        </state_interface>
+        <state_interface name="velocity"/>
+        <state_interface name="effort"/>
+      </joint>
+      <transmission name="${name}_hub_left_joint_transmission">
+        <plugin>transmission_interface/SimpleTansmission</plugin>
+        <param name="joint_to_actuator">1</param>
+      </transmission>
+      <joint name="${name}_hub_right_joint">
+        <command_interface name="position">
+          <param name="min">-1e+100</param>
+          <param name="max">1e+100</param>
+        </command_interface>
+        <command_interface name="velocity">
+          <param name="min">-1e+100</param>
+          <param name="max">1e+100</param>
+        </command_interface>
+        <command_interface name="effort">
+          <param name="min">-1e+100</param>
+          <param name="max">1e+100</param>
+        </command_interface>
+        <state_interface name="position">
+           <param name="initial_value">0.0</param>
+        </state_interface>
+        <state_interface name="velocity"/>
+        <state_interface name="effort"/>
+      </joint>
+      <transmission name="${name}_hub_right_joint_transmission">
+        <plugin>transmission_interface/SimpleTansmission</plugin>
+        <param name="joint_to_actuator">1</param>
+      </transmission>
+    </ros2_control>
+  </xacro:macro>
 </robot>
