Commit message: arm position at rest

File: freddy_torso_description/urdf/freddy_torso_gz.urdf.xacro (robot description, xacro)
@@ -13,4 +13,81 @@
     <xacro:include filename="$(find freddy_base_description)/urdf/freddy_base_gz.urdf.xacro" />
     <xacro:macro name="freddy_torso" params="name parent *origin use_gpu_2d_laser:=true">
+   <!--<joint name="kinova_left_joint_1">
+      <command_interface name="position">
+          <param name="min">{-2*pi}</param>
+          <param name="max">{2*pi}</param>
+      </command_interface>
+      <state_interface name="position">
+        <param name="initial_value">1.57</param>
+      </state_interface>
+      <state_interface name="velocity"/>
+      <state_interface name="effort"/>
+    </joint>
+    <joint name="kinova_left_joint_2">
+      <command_interface name="position">
+        <param name="min">-2.41</param>
+          <param name="max">2.41</param>
+      </command_interface>
+      <state_interface name="position">
+        <param name="initial_value">-0.35</param>
+      </state_interface>
+      <state_interface name="velocity"/>
+      <state_interface name="effort"/>
+    </joint>
+     <joint name="kinova_left_joint_3">
+      <command_interface name="position">
+        <param name="min">{-2*pi}</param>
+          <param name="max">{2*pi}</param>
+      </command_interface>
+      <state_interface name="position">
+        <param name="initial_value">3.14</param>
+      </state_interface>
+      <state_interface name="velocity"/>
+      <state_interface name="effort"/>
+    </joint>
+     <joint name="kinova_left_joint_4">
+      <command_interface name="position">
+         <param name="min">-2.66</param>
+          <param name="max">2.66</param>
+      </command_interface>
+      <state_interface name="position">
+        <param name="initial_value"> -2.00</param>
+      </state_interface>
+      <state_interface name="velocity"/>
+      <state_interface name="effort"/>
+    </joint>
+    <joint name="kinova_left_joint_5">
+      <command_interface name="position">
+          <param name="min">{-2*pi}</param>
+          <param name="max">{2*pi}</param>
+      </command_interface>
+      <state_interface name="position">
+        <param name="initial_value">0</param>
+      </state_interface>
+      <state_interface name="velocity"/>
+      <state_interface name="effort"/>
+    </joint>
+     <joint name="kinova_left_joint_6">
+      <command_interface name="position">
+          <param name="min">-2.23</param>
+          <param name="max">2.23</param>
+      </command_interface>
+      <state_interface name="position">
+        <param name="initial_value">-1.00</param>
+      </state_interface>
+      <state_interface name="velocity"/>
+      <state_interface name="effort"/>
+    </joint>
+    <joint name="kinova_left_joint_7">
+      <command_interface name="position">
+          <param name="min">{-2*pi}</param>
+          <param name="max">{2*pi}</param>
+      </command_interface>
+      <state_interface name="position">
+        <param name="initial_value">1.57</param>
+      </state_interface>
+      <state_interface name="velocity"/>
+      <state_interface name="effort"/>
+    </joint> -->
         <!-- TORSO -->
         <joint name="${name}_joint" type="fixed">
