Commit message: Add left arm

File: freddy_description/robots/freddy_arms_gz.urdf.xacro (robot description, xacro)
@@ -4,5 +4,36 @@
     <!-- Robot tf_prefix -->
     <xacro:arg name="tf_prefix" default="" />
+    <xacro:arg name="prefix_arm_left" default="kinova_left_" />
+    <xacro:arg name="arm" default="gen3" />
+    <xacro:arg name="dof" default="7" />
     <xacro:arg name="sim_gz" default="true" />
+    <xacro:arg name="vision" default="true" />
+    <xacro:arg name="robot_ip_left" default="192.168.1.10" />
+    <xacro:arg name="robot_ip_right" default="192.168.1.11" />
+    <xacro:arg name="username" default="admin" />
+    <xacro:arg name="password" default="admin" />
+    <xacro:arg name="port" default="10000" />
+    <xacro:arg name="port_realtime" default="10001" />
+    <xacro:arg name="session_inactivity_timeout_ms" default="60000" />
+    <xacro:arg name="connection_inactivity_timeout_ms" default="2000" />
+    <xacro:arg name="gripper" default="robotiq_2f_85" />
+    <xacro:arg name="gripper_joint_name" default="finger_joint" />
+    <xacro:arg name="gripper_max_velocity" default="100.0" />
+    <xacro:arg name="gripper_max_force" default="100.0" />
+    <xacro:arg name="use_internal_bus_gripper_comm" default="false" />
+    <xacro:arg name="use_fake_hardware" default="false" />
+    <xacro:arg name="fake_sensor_commands" default="false" />
+    <xacro:arg name="sim_gazebo" default="false" />
+    <xacro:arg name="sim_ignition" default="false" />
+    <xacro:arg name="sim_isaac" default="false" />
+    <xacro:arg name="gazebo_renderer" default="ogre" />
+    <xacro:arg name="camera_width" default="640" />
+    <xacro:arg name="camera_height" default="480" />
+    <xacro:arg name="camera_fps" default="6" />
+    <xacro:arg name="simulation_controllers" default="$(find kortex_description)/arm/$(arg arm)/$(arg dof)dof/config/ros2_controllers.yaml" />
+    <!-- Initial position for simulations (Mock Hardware, Gazebo, Ignition) -->
+    <xacro:arg name="initial_positions_file" default="$(find freddy_description)/config/initial_positions.yaml" />
+    <!-- Convert to property to use substitution in function -->
+    <xacro:property name="initial_positions_file" default="$(arg initial_positions_file)" />
     <xacro:include filename="$(find freddy_base_description)/urdf/common.xacro" />
     <xacro:include filename="$(find freddy_base_description)/urdf/freddy_base_gz.urdf.xacro" />
@@ -55,9 +86,9 @@
     <xacro:if value="$(arg sim_gz)">
         <!-- Gazebo plugins -->
-        <gazebo reference="world">
-        </gazebo>
         <gazebo>
-            <plugin filename="libgazebo_ros2_control.so" name="gazebo_ros2_control">
-                <parameters>$(arg simulation_controllers)</parameters>
+            <plugin filename="libgz_ros2_control-system.so" name="gz_ros2_control::GazeboSimROS2ControlPlugin">
+                <robot_param>robot_description</robot_param>
+                <robot_param_node>robot_state_publisher</robot_param_node>
+                <parameters>$(find freddy_gazebo)/config/base_controller.yaml</parameters>
             </plugin>
         </gazebo>

Commit message: Left and right arm controller added

File: freddy_description/robots/freddy_arms_gz.urdf.xacro (robot description, xacro)
@@ -39,5 +39,5 @@
     <xacro:include filename="$(find freddy_base_description)/urdf/freddy_base_gz.urdf.xacro" />
     <xacro:include filename="$(find freddy_torso_description)/urdf/freddy_torso_gz.urdf.xacro" />
-    <xacro:include filename="$(find kortex_description)/robots/kortex_robot_gz.xacro" />
+    <xacro:include filename="$(find kortex_description)/robots/kortex_robot.xacro" />
     <link name="base_link"/>
     <xacro:freddy_base name="freddy_base" parent="base_link"

File: freddy_description/robots/freddy_gz_torso1.urdf.xacro (robot description, xacro)
@@ -23,4 +23,5 @@
     <xacro:arg name="use_fake_hardware" default="true" />
     <xacro:arg name="fake_sensor_commands" default="true" />
+    <xacro:arg name="sim_gz" default="true" />
     <xacro:arg name="sim_gazebo" default="false" />
     <xacro:arg name="sim_ignition" default="false" />
@@ -32,5 +33,4 @@
     <xacro:arg name="simulation_controllers"
         default="$(find freddy_gazebo)/config/torso_controller.yaml" />
-<xacro:property name="sim_gz" value="true"/>
     <xacro:include filename="$(find freddy_base_description)/urdf/materials.urdf.xacro" />
     <xacro:include filename="$(find kortex_description)/robots/kortex_robot.xacro" />
@@ -51,14 +51,10 @@
     <xacro:arg name="initial_positions_file"
         default="$(find freddy_description)/config/initial_positions.yaml" />
+    <xacro:arg name="initial_positions_file_right"
+        default="$(find freddy_description)/config/initial_positions_right.yaml" />
     <!-- convert to property to use substitution in function -->
     <xacro:property name="initial_positions_file" default="$(arg initial_positions_file)" />
+     <xacro:property name="initial_positions_file_right" default="$(arg initial_positions_file_right)" />
 <!-- Commented for testing -->
-    <!-- arms -->
- <!-- Taken out from params below
- gripper="$(arg gripper)"
-        gripper_joint_name="$(arg gripper_joint_name)"
-        gripper_max_velocity="$(arg gripper_max_velocity)"
-        gripper_max_force="$(arg gripper_max_force)" -->
-    <!-- left arm -->
     <xacro:load_robot
         parent="freddy_torso_shoulder_left_arm_attach_link"
@@ -81,4 +77,5 @@
         use_fake_hardware="$(arg use_fake_hardware)"
         fake_sensor_commands="$(arg fake_sensor_commands)"
+        sim_gz="$(arg sim_gz)"
         sim_gazebo="$(arg sim_gazebo)"
         sim_ignition="$(arg sim_ignition)"
@@ -87,5 +84,6 @@
         <origin xyz="0 0 0" rpy="0 0 0" />
     </xacro:load_robot>
-    <!-- <xacro:load_robot
+ <!-- right arm -->
+    <xacro:load_robot
         parent="freddy_torso_shoulder_right_arm_attach_link"
         arm="$(arg arm)"
@@ -107,23 +105,11 @@
         use_fake_hardware="$(arg use_fake_hardware)"
         fake_sensor_commands="$(arg fake_sensor_commands)"
+        sim_gz="$(arg sim_gz)"
         sim_gazebo="$(arg sim_gazebo)"
         sim_ignition="$(arg sim_ignition)"
         sim_isaac="$(arg sim_isaac)"
-        initial_positions="${xacro.load_yaml(initial_positions_file)}">
+        initial_positions="${xacro.load_yaml(initial_positions_file_right)}">
         <origin xyz="0 0 0" rpy="0 0 0" />
-    </xacro:load_robot>  -->
-<ros2_control name="GazeboSimSystem" type="system">
-    <hardware>
-      <plugin>gz_ros2_control/GazeboSimSystem</plugin>
-    </hardware> -->
-    <!-- <joint name="kinova_left_joint_1">
-      <command_interface name="velocity">
-      <param name="min">-1</param>
-      <param name="max">1</param>
-        </command_interface>
-      <state_interface name="velocity"/>
-      <state_interface name="position"/>
-    </joint> -->
-<!-- </ros2_control>
+    </xacro:load_robot>
     <gazebo>
             <plugin filename="gz_ros2_control-system" name="gz_ros2_control::GazeboSimROS2ControlPlugin">
@@ -131,127 +117,6 @@
                 <robot_param_node>robot_state_publisher</robot_param_node>
                 <parameters>$(find freddy_gazebo)/config/torso_controller.yaml</parameters>
+                 <controller_manager_node_name>arms_controller_manager</controller_manager_node_name>
             </plugin>
-     <!-- <plugin
-        filename="gz-sim-joint-controller-system"
-        name="gz::sim::systems::JointController">
-        <joint_name>kinova_left_joint_1</joint_name>
-        <p_gain>0.2</p_gain>
-        <i_gain>0.01</i_gain>
-      </plugin> -->
-<!--
-        <plugin filename="gz-sim-joint-state-publisher-system" name="gz::sim::systems::JointStatePublisher">
-            <topic>joint_states</topic>
-        </plugin>
-   -->
-      <!-- <plugin
-        filename="gz-sim-joint-state-publisher-system"
-        name="gz::sim::systems::JointStatePublisher">
-        <joint_name>kinova_left_joint_1</joint_name>
-        </plugin> -->
-        <!-- <plugin
-            filename="gz-sim-joint-position-controller-system"
-            name="gz::sim::systems::JointPositionController">
-            <joint_name>kinova_left_joint_1</joint_name>
-            <topic>kinova_left_joint_1</topic>
-            <p_gain>1</p_gain>
-            <i_gain>0.1</i_gain>
-            <d_gain>0.01</d_gain>
-            <i_max>1</i_max>
-            <i_min>-1</i_min>
-            <cmd_max>1000</cmd_max>
-            <cmd_min>-1000</cmd_min>
-            </plugin> -->
-            <!-- <plugin
-        filename="gz-sim-joint-controller-system"
-        name="gz::sim::systems::JointController">
-        <joint_name>kinova_right_joint_1</joint_name>
-        <p_gain>0.2</p_gain>
-        <i_gain>0.01</i_gain>
-      </plugin>
-       <plugin
-        filename="gz-sim-joint-controller-system"
-        name="gz::sim::systems::JointController">
-        <joint_name>kinova_left_joint_2</joint_name>
-        <p_gain>0.2</p_gain>
-        <i_gain>0.01</i_gain>
-      </plugin>
-       <plugin
-        filename="gz-sim-joint-controller-system"
-        name="gz::sim::systems::JointController">
-        <joint_name>kinova_left_joint_3</joint_name>
-        <p_gain>0.2</p_gain>
-        <i_gain>0.01</i_gain>
-      </plugin>
-      <plugin
-        filename="gz-sim-joint-controller-system"
-        name="gz::sim::systems::JointController">
-        <joint_name>kinova_left_joint_4</joint_name>
-        <p_gain>0.2</p_gain>
-        <i_gain>0.01</i_gain>
-      </plugin>
-       <plugin
-        filename="gz-sim-joint-controller-system"
-        name="gz::sim::systems::JointController">
-        <joint_name>kinova_left_joint_5</joint_name>
-        <p_gain>0.2</p_gain>
-        <i_gain>0.01</i_gain>
-      </plugin>
-       <plugin
-        filename="gz-sim-joint-controller-system"
-        name="gz::sim::systems::JointController">
-        <joint_name>kinova_left_joint_6</joint_name>
-        <p_gain>0.2</p_gain>
-        <i_gain>0.01</i_gain>
-      </plugin>
-      <plugin
-        filename="gz-sim-joint-controller-system"
-        name="gz::sim::systems::JointController">
-        <joint_name>kinova_left_joint_7</joint_name>
-        <p_gain>0.2</p_gain>
-        <i_gain>0.01</i_gain>
-      </plugin>
-      <plugin
-        filename="gz-sim-joint-controller-system"
-        name="gz::sim::systems::JointController">
-        <joint_name>kinova_right_joint_2</joint_name>
-        <p_gain>0.2</p_gain>
-        <i_gain>0.01</i_gain>
-      </plugin>
-       <plugin
-        filename="gz-sim-joint-controller-system"
-        name="gz::sim::systems::JointController">
-        <joint_name>kinova_right_joint_3</joint_name>
-        <p_gain>0.2</p_gain>
-        <i_gain>0.01</i_gain>
-      </plugin>
-      <plugin
-        filename="gz-sim-joint-controller-system"
-        name="gz::sim::systems::JointController">
-        <joint_name>kinova_right_joint_4</joint_name>
-        <p_gain>0.2</p_gain>
-        <i_gain>0.01</i_gain>
-      </plugin>
-       <plugin
-        filename="gz-sim-joint-controller-system"
-        name="gz::sim::systems::JointController">
-        <joint_name>kinova_right_joint_5</joint_name>
-        <p_gain>0.2</p_gain>
-        <i_gain>0.01</i_gain>
-      </plugin>
-       <plugin
-        filename="gz-sim-joint-controller-system"
-        name="gz::sim::systems::JointController">
-        <joint_name>kinova_right_joint_6</joint_name>
-        <p_gain>0.2</p_gain>
-        <i_gain>0.01</i_gain>
-      </plugin>
-      <plugin
-        filename="gz-sim-joint-controller-system"
-        name="gz::sim::systems::JointController">
-        <joint_name>kinova_right_joint_7</joint_name>
-        <p_gain>0.2</p_gain>
-        <i_gain>0.01</i_gain>
-      </plugin>
-      -->
     </gazebo>
 </robot>

File: freddy_torso_description/urdf/freddy_torso_gz.urdf.xacro (robot description, xacro)
@@ -13,86 +13,4 @@
     <xacro:include filename="$(find freddy_base_description)/urdf/freddy_base_gz.urdf.xacro" />
     <xacro:macro name="freddy_torso" params="name parent *origin use_gpu_2d_laser:=true">
-<ros2_control name="GazeboSimSystem" type="system">
-    <hardware>
-      <plugin>gz_ros2_control/GazeboSimSystem</plugin>
-    </hardware>
-</ros2_control>
-   <!--<joint name="kinova_left_joint_1">
-      <command_interface name="position">
-          <param name="min">{-2*pi}</param>
-          <param name="max">{2*pi}</param>
-      </command_interface>
-      <state_interface name="position">
-        <param name="initial_value">1.57</param>
-      </state_interface>
-      <state_interface name="velocity"/>
-      <state_interface name="effort"/>
-    </joint>
-    <joint name="kinova_left_joint_2">
-      <command_interface name="position">
-        <param name="min">-2.41</param>
-          <param name="max">2.41</param>
-      </command_interface>
-      <state_interface name="position">
-        <param name="initial_value">-0.35</param>
-      </state_interface>
-      <state_interface name="velocity"/>
-      <state_interface name="effort"/>
-    </joint>
-     <joint name="kinova_left_joint_3">
-      <command_interface name="position">
-        <param name="min">{-2*pi}</param>
-          <param name="max">{2*pi}</param>
-      </command_interface>
-      <state_interface name="position">
-        <param name="initial_value">3.14</param>
-      </state_interface>
-      <state_interface name="velocity"/>
-      <state_interface name="effort"/>
-    </joint>
-     <joint name="kinova_left_joint_4">
-      <command_interface name="position">
-         <param name="min">-2.66</param>
-          <param name="max">2.66</param>
-      </command_interface>
-      <state_interface name="position">
-        <param name="initial_value"> -2.00</param>
-      </state_interface>
-      <state_interface name="velocity"/>
-      <state_interface name="effort"/>
-    </joint>
-    <joint name="kinova_left_joint_5">
-      <command_interface name="position">
-          <param name="min">{-2*pi}</param>
-          <param name="max">{2*pi}</param>
-      </command_interface>
-      <state_interface name="position">
-        <param name="initial_value">0</param>
-      </state_interface>
-      <state_interface name="velocity"/>
-      <state_interface name="effort"/>
-    </joint>
-     <joint name="kinova_left_joint_6">
-      <command_interface name="position">
-          <param name="min">-2.23</param>
-          <param name="max">2.23</param>
-      </command_interface>
-      <state_interface name="position">
-        <param name="initial_value">-1.00</param>
-      </state_interface>
-      <state_interface name="velocity"/>
-      <state_interface name="effort"/>
-    </joint>
-    <joint name="kinova_left_joint_7">
-      <command_interface name="position">
-          <param name="min">{-2*pi}</param>
-          <param name="max">{2*pi}</param>
-      </command_interface>
-      <state_interface name="position">
-        <param name="initial_value">1.57</param>
-      </state_interface>
-      <state_interface name="velocity"/>
-      <state_interface name="effort"/>
-    </joint> -->
         <!-- TORSO -->
         <joint name="${name}_joint" type="fixed">
@@ -202,5 +120,8 @@
             <child link="${name}_shoulder_right_arm_attach_link" />
         </joint>
-        <link name="${name}_shoulder_right_arm_attach_link" />
+         <link name="${name}_shoulder_right_arm_attach_link" />
+        <gazebo reference="${name}_link">
+            <material>Gazebo/RustySteel</material>
+        </gazebo>
     </xacro:macro>
 </robot>
