Commit message: clean-up of the repo

File: freddy_description/robots/freddy_gz.urdf.xacro (robot description, xacro)
@@ -1,32 +1,120 @@
 <?xml version='1.0'?>
 <robot xmlns:xacro="http://www.ros.org/wiki/xacro" name="freddy">
-  <xacro:arg name="use_gpu_2d_laser" default="false" />
-  <!-- Robot tf_prefix -->
-  <xacro:arg name="tf_prefix" default="" />
+    <xacro:arg name="use_gpu_2d_laser" default="false" />
+    <!-- Arguments -->
+    <xacro:arg name="prefix_arm_left" default="kinova_left_" />
+    <xacro:arg name="prefix_arm_right" default="kinova_right_" />
+    <xacro:arg name="arm" default="gen3" />
+    <xacro:arg name="dof" default="7" />
+    <xacro:arg name="vision" default="false" />
+    <xacro:arg name="robot_ip_left" default="192.168.1.10" />
+    <xacro:arg name="robot_ip_right" default="192.168.1.11" />
+    <xacro:arg name="username" default="admin" />
+    <xacro:arg name="password" default="admin" />
+    <xacro:arg name="port" default="10000" />
+    <xacro:arg name="port_realtime" default="10001" />
+    <xacro:arg name="session_inactivity_timeout_ms" default="60000" />
+    <xacro:arg name="connection_inactivity_timeout_ms" default="2000" />
+     <xacro:arg name="gripper" default="robotiq_2f_85" />
+    <xacro:arg name="gripper_joint_name" default="finger_joint" />
+    <xacro:arg name="gripper_max_velocity" default="100.0" />
+    <xacro:arg name="gripper_max_force" default="100.0" />
+    <xacro:arg name="use_internal_bus_gripper_comm" default="false" />
+    <xacro:arg name="use_fake_hardware" default="true" />
+    <xacro:arg name="fake_sensor_commands" default="true" />
+    <xacro:arg name="sim_gz" default="true" />
+    <xacro:arg name="sim_gazebo" default="false" />
+    <xacro:arg name="sim_ignition" default="false" />
+     <xacro:arg name="sim_isaac" default="false" />
+    <xacro:arg name="gazebo_renderer" default="ogre" />
+    <xacro:arg name="camera_width" default="640" />
+    <xacro:arg name="camera_height" default="480" />
+    <xacro:arg name="camera_fps" default="6" />
+    <xacro:arg name="simulation_controllers"
+        default="$(find freddy_gazebo)/config/torso_controller.yaml" />
+    <!-- <xacro:include filename="$(find freddy_base_description)/urdf/materials.urdf.xacro" /> -->
+    <xacro:include filename="$(find kortex_description)/robots/kortex_robot.xacro" />
+ <!-- Added it for testing -->
   <xacro:include filename="$(find freddy_base_description)/urdf/common.xacro" />
-  <xacro:include filename="$(find freddy_base_description)/urdf/freddy_base_gz.urdf.xacro" />
-  <xacro:include filename="$(find freddy_torso_description)/urdf/freddy_torso_gz.urdf.xacro" />
-  <link name="base_link"/>
-  <xacro:freddy_base name="freddy_base" parent="base_link"
-    use_gpu_2d_laser="$(arg use_gpu_2d_laser)">
-    <origin xyz="0.0 0.0 0.0" rpy="0.0 0.0 0.0" />
-  </xacro:freddy_base>
-  <xacro:freddy_torso name="freddy_torso" parent="base_link">
-    <origin xyz="0.0 0.0 0.0" rpy="0.0 0.0 0.0" />
-  </xacro:freddy_torso>
-  <gazebo>
-    <!-- VELOCITY CONTROL PLUGIN -->
-    <plugin
-      filename="gz-sim-velocity-control-system"
-      name="gz::sim::systems::VelocityControl">
-      <initial_linear>0.0 0 0</initial_linear>
-      <initial_angular>0 0 0.0</initial_angular>
-      <!-- <link_name>base_link</link_name> -->
-      <!-- <topic>cmd_vel</topic> -->
-    </plugin>
-    <!-- Joint state publisher -->
-    <plugin filename="gz_ros2_control-system" name="gz_ros2_control::GazeboSimROS2ControlPlugin">
-      <parameters>$(find freddy_description)/config/ros2_controllers_double_wheel.yaml</parameters>
-    </plugin>
-  </gazebo>
+    <xacro:include filename="$(find freddy_base_description)/urdf/freddy_base_gz.urdf.xacro" />
+    <xacro:include filename="$(find freddy_torso_description)/urdf/freddy_torso_gz.urdf.xacro" />
+    <link name="base_link"/>
+    <xacro:freddy_base name="freddy_base" parent="base_link"
+        use_gpu_2d_laser="$(arg use_gpu_2d_laser)">
+        <origin xyz="0.0 0.0 0.0" rpy="0.0 0.0 0.0" />
+    </xacro:freddy_base>
+    <xacro:freddy_torso name="freddy_torso" parent="base_link">
+        <origin xyz="0.0 0.0 0.0" rpy="0.0 0.0 0.0" />
+    </xacro:freddy_torso>
+    <!-- initial position for simulations (Mock Hardware, Gazebo, Ignition) -->
+    <xacro:arg name="initial_positions_file"
+        default="$(find freddy_description)/config/initial_positions.yaml" />
+    <xacro:arg name="initial_positions_file_right"
+        default="$(find freddy_description)/config/initial_positions_right.yaml" />
+    <!-- convert to property to use substitution in function -->
+    <xacro:property name="initial_positions_file" default="$(arg initial_positions_file)" />
+     <xacro:property name="initial_positions_file_right" default="$(arg initial_positions_file_right)" />
+<!-- Commented for testing -->
+    <xacro:load_robot
+        parent="freddy_torso_shoulder_left_arm_attach_link"
+        arm="$(arg arm)"
+        gripper=""
+        gripper_joint_name="$(arg gripper_joint_name)"
+        gripper_max_velocity="$(arg gripper_max_velocity)"
+        gripper_max_force="$(arg gripper_max_force)"
+        dof="$(arg dof)"
+        vision="$(arg vision)"
+        robot_ip="$(arg robot_ip_left)"
+        username="$(arg username)"
+        password="$(arg password)"
+        port="$(arg port)"
+        port_realtime="$(arg port_realtime)"
+        session_inactivity_timeout_ms="$(arg session_inactivity_timeout_ms)"
+        connection_inactivity_timeout_ms="$(arg connection_inactivity_timeout_ms)"
+        use_internal_bus_gripper_comm="$(arg use_internal_bus_gripper_comm)"
+        prefix="$(arg prefix_arm_left)"
+        use_fake_hardware="$(arg use_fake_hardware)"
+        fake_sensor_commands="$(arg fake_sensor_commands)"
+        sim_gz="$(arg sim_gz)"
+        sim_gazebo="$(arg sim_gazebo)"
+        sim_ignition="$(arg sim_ignition)"
+        sim_isaac="$(arg sim_isaac)"
+        initial_positions="${xacro.load_yaml(initial_positions_file)}">
+        <origin xyz="0 0 0" rpy="0 0 0" />
+    </xacro:load_robot>
+ <!-- right arm -->
+    <xacro:load_robot
+        parent="freddy_torso_shoulder_right_arm_attach_link"
+        arm="$(arg arm)"
+        gripper=""
+        gripper_joint_name="$(arg gripper_joint_name)"
+        gripper_max_velocity="$(arg gripper_max_velocity)"
+        gripper_max_force="$(arg gripper_max_force)"
+        dof="$(arg dof)"
+        vision="$(arg vision)"
+        robot_ip="$(arg robot_ip_right)"
+        username="$(arg username)"
+        password="$(arg password)"
+        port="$(arg port)"
+        port_realtime="$(arg port_realtime)"
+        session_inactivity_timeout_ms="$(arg session_inactivity_timeout_ms)"
+        connection_inactivity_timeout_ms="$(arg connection_inactivity_timeout_ms)"
+        use_internal_bus_gripper_comm="$(arg use_internal_bus_gripper_comm)"
+        prefix="$(arg prefix_arm_right)"
+        use_fake_hardware="$(arg use_fake_hardware)"
+        fake_sensor_commands="$(arg fake_sensor_commands)"
+        sim_gz="$(arg sim_gz)"
+        sim_gazebo="$(arg sim_gazebo)"
+        sim_ignition="$(arg sim_ignition)"
+        sim_isaac="$(arg sim_isaac)"
+        initial_positions="${xacro.load_yaml(initial_positions_file_right)}">
+        <origin xyz="0 0 0" rpy="0 0 0" />
+    </xacro:load_robot>
+    <gazebo>
+            <plugin filename="gz_ros2_control-system" name="gz_ros2_control::GazeboSimROS2ControlPlugin">
+                <robot_param>robot_description</robot_param>
+                <robot_param_node>robot_state_publisher</robot_param_node>
+                <parameters>$(find freddy_gazebo)/config/torso_controller.yaml</parameters>
+            </plugin>
+    </gazebo>
 </robot>

Commit message: Cleanup

File: freddy_description/robots/freddy_gz.urdf.xacro (robot description, xacro)
@@ -16,5 +16,5 @@
     <xacro:arg name="session_inactivity_timeout_ms" default="60000" />
     <xacro:arg name="connection_inactivity_timeout_ms" default="2000" />
-     <xacro:arg name="gripper" default="robotiq_2f_85" />
+    <xacro:arg name="gripper" default="robotiq_2f_85" />
     <xacro:arg name="gripper_joint_name" default="finger_joint" />
     <xacro:arg name="gripper_max_velocity" default="100.0" />
@@ -26,5 +26,5 @@
     <xacro:arg name="sim_gazebo" default="false" />
     <xacro:arg name="sim_ignition" default="false" />
-     <xacro:arg name="sim_isaac" default="false" />
+    <xacro:arg name="sim_isaac" default="false" />
     <xacro:arg name="gazebo_renderer" default="ogre" />
     <xacro:arg name="camera_width" default="640" />
@@ -35,6 +35,6 @@
     <!-- <xacro:include filename="$(find freddy_base_description)/urdf/materials.urdf.xacro" /> -->
     <xacro:include filename="$(find kortex_description)/robots/kortex_robot.xacro" />
- <!-- Added it for testing -->
-  <xacro:include filename="$(find freddy_base_description)/urdf/common.xacro" />
+    <!-- Added it for testing -->
+    <xacro:include filename="$(find freddy_base_description)/urdf/common.xacro" />
     <xacro:include filename="$(find freddy_base_description)/urdf/freddy_base_gz.urdf.xacro" />
     <xacro:include filename="$(find freddy_torso_description)/urdf/freddy_torso_gz.urdf.xacro" />
@@ -54,6 +54,6 @@
     <!-- convert to property to use substitution in function -->
     <xacro:property name="initial_positions_file" default="$(arg initial_positions_file)" />
-     <xacro:property name="initial_positions_file_right" default="$(arg initial_positions_file_right)" />
-<!-- Commented for testing -->
+    <xacro:property name="initial_positions_file_right" default="$(arg initial_positions_file_right)" />
+    <!-- Commented for testing -->
     <xacro:load_robot
         parent="freddy_torso_shoulder_left_arm_attach_link"
@@ -83,5 +83,5 @@
         <origin xyz="0 0 0" rpy="0 0 0" />
     </xacro:load_robot>
- <!-- right arm -->
+    <!-- right arm -->
     <xacro:load_robot
         parent="freddy_torso_shoulder_right_arm_attach_link"
@@ -112,10 +112,9 @@
     </xacro:load_robot>
     <gazebo>
-            <plugin filename="gz_ros2_control-system" name="gz_ros2_control::GazeboSimROS2ControlPlugin">
-                <robot_param>robot_description</robot_param>
-                <robot_param_node>robot_state_publisher</robot_param_node>
-                <parameters>$(arg simulation_controllers)</parameters>
-                <!-- <parameters>$(find freddy_gazebo)/config/arms_controller.yaml</parameters>          -->
-            </plugin>
+        <plugin filename="gz_ros2_control-system" name="gz_ros2_control::GazeboSimROS2ControlPlugin">
+            <robot_param>robot_description</robot_param>
+            <robot_param_node>robot_state_publisher</robot_param_node>
+            <parameters>$(arg simulation_controllers)</parameters>
+        </plugin>
     </gazebo>
 </robot>

Commit message: Rename initial position files

File: freddy_description/robots/freddy_gz.urdf.xacro (robot description, xacro)
@@ -48,10 +48,10 @@
     </xacro:freddy_torso>
     <!-- initial position for simulations (Mock Hardware, Gazebo, Ignition) -->
-    <xacro:arg name="initial_positions_file"
-        default="$(find freddy_description)/config/initial_positions.yaml" />
+    <xacro:arg name="initial_positions_file_left"
+        default="$(find freddy_description)/config/initial_positions_arm_left.yaml" />
     <xacro:arg name="initial_positions_file_right"
-        default="$(find freddy_description)/config/initial_positions_right.yaml" />
+        default="$(find freddy_description)/config/initial_positions_arm_right.yaml" />
     <!-- convert to property to use substitution in function -->
-    <xacro:property name="initial_positions_file" default="$(arg initial_positions_file)" />
+    <xacro:property name="initial_positions_file_left" default="$(arg initial_positions_file_left)" />
     <xacro:property name="initial_positions_file_right" default="$(arg initial_positions_file_right)" />
     <!-- Commented for testing -->
@@ -80,5 +80,5 @@
         sim_ignition="$(arg sim_ignition)"
         sim_isaac="$(arg sim_isaac)"
-        initial_positions="${xacro.load_yaml(initial_positions_file)}">
+        initial_positions="${xacro.load_yaml(initial_positions_file_left)}">
         <origin xyz="0 0 0" rpy="0 0 0" />
     </xacro:load_robot>
@@ -117,4 +117,5 @@
             <parameters>$(arg simulation_controllers)</parameters>
         </plugin>
+        <self_collide>1</self_collide>
     </gazebo>
 </robot>

File: freddy_torso_description/urdf/freddy_torso_gz.urdf.xacro (robot description, xacro)
@@ -63,5 +63,5 @@
             <collision>
                 <origin
-                    xyz="0 0 ${-torso_shoulder_thickness/2}"
+                    xyz="0 ${torso_shoulder_width/2} ${torso_shoulder_height/2}"
                     rpy="0 0 0" />
                 <geometry>
@@ -70,6 +70,6 @@
                 </geometry>
             </collision>
-            <!-- <xacro:cuboid_inertia mass="${base_mass}" length="${base_size_x}"
-                breadth="${base_size_y}" height="${base_size_z}" /> -->
+            <xacro:cuboid_inertia mass="${base_mass}" length="${base_size_x}"
+                breadth="${base_size_y}" height="${base_size_z}" />
         </link>
         <joint name="${name}_shoulder_left_arm_joint" type="fixed">
@@ -102,5 +102,5 @@
             <collision>
                 <origin
-                    xyz="0 0 ${-torso_shoulder_thickness/2}"
+                    xyz="0 ${-torso_shoulder_width/2} ${torso_shoulder_height/2}"
                     rpy="0 0 0" />
                 <geometry>
@@ -110,6 +110,6 @@
             </collision>
             <!-- This is causing the base to topple over under combined x y velocity -->
-            <!-- <xacro:cuboid_inertia mass="${base_mass}" length="${base_size_x}"
-                breadth="${base_size_y}" height="${base_size_z}" /> -->
+            <xacro:cuboid_inertia mass="${base_mass}" length="${base_size_x}"
+                breadth="${base_size_y}" height="${base_size_z}" />
         </link>
         <joint name="${name}_shoulder_right_arm_joint" type="fixed">
@@ -121,7 +121,4 @@
         </joint>
          <link name="${name}_shoulder_right_arm_attach_link" />
-        <gazebo reference="${name}_link">
-            <material>Gazebo/RustySteel</material>
-        </gazebo>
     </xacro:macro>
 </robot>
