Commit message: renaming to eddie

File: eddie_base_description/urdf/eddie_base_gz.urdf.xacro (robot description, xacro)
@@ -2,5 +2,5 @@
 <robot xmlns:xacro="http://www.ros.org/wiki/xacro">
     <!-- simplified box collision geometry for base -->
-    <xacro:property name="robot_name" value="freddy"/>
+    <xacro:property name="robot_name" value="eddie"/>
     <xacro:property name="base_size_x" value="0.635"/>
     <xacro:property name="base_size_y" value="0.582"/>
@@ -11,6 +11,6 @@
     <xacro:property name="base_size_z" value="${base_size_z_bottom + laser_slit_height + base_size_z_top}"/>
     <xacro:property name="base_mass" value="40.0"/>
-    <xacro:include filename="$(find freddy_base_description)/urdf/kelo_wheel_gz.urdf.xacro" />
-    <xacro:macro name="freddy_base" params="name parent *origin use_gpu_2d_laser:=true">
+    <xacro:include filename="$(find eddie_base_description)/urdf/kelo_wheel_gz.urdf.xacro" />
+    <xacro:macro name="eddie_base" params="name parent *origin use_gpu_2d_laser:=true">
         <!-- BASE -->
         <link name="${name}_link">

File: eddie_base_description/urdf/sensors/hokuyo.urdf.xacro (robot description, xacro)
@@ -26,5 +26,5 @@
 -->
 <robot xmlns:xacro="http://www.ros.org/wiki/xacro">
-    <xacro:include filename="$(find freddy_base_description)/urdf/sensors/common.xacro" />
+    <xacro:include filename="$(find eddie_base_description)/urdf/sensors/common.xacro" />
     <xacro:macro name="hokuyo" params="*origin name:=base_laser_front topic:=base_scan parent:=base_link sample_size:=1080 update_rate:=40
     min_angle:=-2.35619 max_angle:=2.35619 min_range:=0.06 max_range:=10.0 robot_namespace:=/ use_gpu:=true visualize:=false" >
@@ -44,5 +44,5 @@
                 <origin xyz="0 0 0" rpy="0 0 0" />
                 <geometry>
-                    <mesh filename="package://freddy_base_description/meshes/sensors/hokuyo.dae" />
+                    <mesh filename="package://eddie_base_description/meshes/sensors/hokuyo.dae" />
                 </geometry>
             </visual>
@@ -50,5 +50,5 @@
                 <origin xyz="0 0 0" rpy="0 0 0" />
                 <geometry>
-                    <mesh filename="package://freddy_base_description/meshes/sensors/hokuyo_convex.dae" />
+                    <mesh filename="package://eddie_base_description/meshes/sensors/hokuyo_convex.dae" />
                 </geometry>
             </collision>

File: eddie_description/robots/eddie_gz.urdf.xacro (robot description, xacro)
@@ -1,4 +1,4 @@
 <?xml version='1.0'?>
-<robot xmlns:xacro="http://www.ros.org/wiki/xacro" name="freddy">
+<robot xmlns:xacro="http://www.ros.org/wiki/xacro" name="eddie">
     <xacro:arg name="use_gpu_2d_laser" default="false" />
     <!-- Arguments -->
@@ -32,22 +32,22 @@
     <xacro:arg name="camera_fps" default="6" />
     <xacro:arg name="simulation_controllers"
-        default="$(find freddy_gazebo)/config/freddy_controller.yaml" />
+        default="$(find eddie_gazebo)/config/eddie_controller.yaml" />
  <xacro:include filename="$(find kortex_description)/robots/kortex_robot.xacro" />
-  <xacro:include filename="$(find freddy_base_description)/urdf/common.xacro" />
-    <xacro:include filename="$(find freddy_base_description)/urdf/freddy_base_gz.urdf.xacro" />
-    <xacro:include filename="$(find freddy_torso_description)/urdf/freddy_torso_gz.urdf.xacro" />
+  <xacro:include filename="$(find eddie_base_description)/urdf/common.xacro" />
+    <xacro:include filename="$(find eddie_base_description)/urdf/eddie_base_gz.urdf.xacro" />
+    <xacro:include filename="$(find eddie_torso_description)/urdf/eddie_torso_gz.urdf.xacro" />
     <link name="base_link"/>
-    <xacro:freddy_base name="freddy_base" parent="base_link"
+    <xacro:eddie_base name="eddie_base" parent="base_link"
         use_gpu_2d_laser="$(arg use_gpu_2d_laser)">
         <origin xyz="0.0 0.0 0.0" rpy="0.0 0.0 0.0" />
-    </xacro:freddy_base>
-    <xacro:freddy_torso name="freddy_torso" parent="base_link">
+    </xacro:eddie_base>
+    <xacro:eddie_torso name="eddie_torso" parent="base_link">
         <origin xyz="0.0 0.0 0.0" rpy="0.0 0.0 0.0" />
-    </xacro:freddy_torso>
+    </xacro:eddie_torso>
     <!-- initial position for simulations (Mock Hardware, Gazebo, Ignition) -->
     <xacro:arg name="initial_positions_file_left"
-        default="$(find freddy_description)/config/initial_positions_arm_left.yaml" />
+        default="$(find eddie_description)/config/initial_positions_arm_left.yaml" />
     <xacro:arg name="initial_positions_file_right"
-        default="$(find freddy_description)/config/initial_positions_arm_right.yaml" />
+        default="$(find eddie_description)/config/initial_positions_arm_right.yaml" />
     <!-- convert to property to use substitution in function -->
     <xacro:property name="initial_positions_file_left" default="$(arg initial_positions_file_left)" />
@@ -55,5 +55,5 @@
    <!-- left arm  -->
     <xacro:load_robot
-        parent="freddy_torso_shoulder_left_arm_attach_link"
+        parent="eddie_torso_shoulder_left_arm_attach_link"
         arm="$(arg arm)"
         gripper=""
@@ -83,5 +83,5 @@
     <!-- right arm -->
     <xacro:load_robot
-        parent="freddy_torso_shoulder_right_arm_attach_link"
+        parent="eddie_torso_shoulder_right_arm_attach_link"
         arm="$(arg arm)"
         gripper=""

File: eddie_torso_description/urdf/eddie_torso_gz.urdf.xacro (robot description, xacro)
@@ -10,7 +10,7 @@
     <xacro:property name="torso_shoulder_width" value="0.2" />
     <xacro:property name="torso_shoulder_thickness" value="0.02" />
-    <xacro:include filename="$(find freddy_base_description)/urdf/common.xacro" />
-    <xacro:include filename="$(find freddy_base_description)/urdf/freddy_base_gz.urdf.xacro" />
-    <xacro:macro name="freddy_torso" params="name parent *origin use_gpu_2d_laser:=true">
+    <xacro:include filename="$(find eddie_base_description)/urdf/common.xacro" />
+    <xacro:include filename="$(find eddie_base_description)/urdf/eddie_base_gz.urdf.xacro" />
+    <xacro:macro name="eddie_torso" params="name parent *origin use_gpu_2d_laser:=true">
         <!-- TORSO -->
         <joint name="${name}_joint" type="fixed">

File: eddie_torso_description/urdf/sensors/hokuyo.urdf.xacro (robot description, xacro)
@@ -26,5 +26,5 @@
 -->
 <robot xmlns:xacro="http://www.ros.org/wiki/xacro">
-    <xacro:include filename="$(find freddy_description)/urdf/sensors/common.xacro" />
+    <xacro:include filename="$(find eddie_description)/urdf/sensors/common.xacro" />
     <xacro:macro name="hokuyo" params="*origin name:=base_laser_front topic:=base_scan parent:=base_link sample_size:=1080 update_rate:=40
     min_angle:=-2.35619 max_angle:=2.35619 min_range:=0.06 max_range:=10.0 robot_namespace:=/ use_gpu:=true visualize:=false" >
@@ -44,5 +44,5 @@
                 <origin xyz="0 0 0" rpy="0 0 0" />
                 <geometry>
-                    <mesh filename="package://freddy_description/meshes/sensors/hokuyo.dae" />
+                    <mesh filename="package://eddie_description/meshes/sensors/hokuyo.dae" />
                 </geometry>
             </visual>
@@ -50,5 +50,5 @@
                 <origin xyz="0 0 0" rpy="0 0 0" />
                 <geometry>
-                    <mesh filename="package://freddy_description/meshes/sensors/hokuyo_convex.dae" />
+                    <mesh filename="package://eddie_description/meshes/sensors/hokuyo_convex.dae" />
                 </geometry>
             </collision>

Commit message: updates to support gz harmonic

File: eddie_base_description/urdf/eddie_base_gz.urdf.xacro (robot description, xacro)
@@ -20,4 +20,5 @@
                     <box size="${base_size_x} ${base_size_y} ${base_size_z_bottom}" />
                 </geometry>
+                <material name="DarkGrey"/>
             </visual>
             <visual>
@@ -26,4 +27,5 @@
                     <box size="${base_size_x*0.7} ${base_size_y*0.7} ${laser_slit_height}" />
                 </geometry>
+                <material name="LightGrey"/>
             </visual>
             <visual>
@@ -32,4 +34,5 @@
                     <box size="${base_size_x} ${base_size_y} ${base_size_z_top}" />
                 </geometry>
+                <material name="DarkGrey"/>
             </visual>
             <!-- base bottom collisions -->

File: eddie_description/robots/eddie.urdf.xacro (robot description, xacro)
@@ -1,5 +1,4 @@
 <?xml version='1.0'?>
 <robot xmlns:xacro="http://www.ros.org/wiki/xacro" name="eddie">
-    <xacro:arg name="use_gpu_2d_laser" default="false" />
     <!-- Arguments -->
     <xacro:arg name="prefix_arm_left" default="kinova_left_" />
@@ -16,26 +15,25 @@
     <xacro:arg name="session_inactivity_timeout_ms" default="60000" />
     <xacro:arg name="connection_inactivity_timeout_ms" default="2000" />
-    <xacro:arg name="gripper" default="robotiq_2f_85" />
-    <xacro:arg name="gripper_joint_name" default="finger_joint" />
-    <xacro:arg name="gripper_max_velocity" default="100.0" />
-    <xacro:arg name="gripper_max_force" default="100.0" />
-    <xacro:arg name="use_internal_bus_gripper_comm" default="false" />
+    <!-- <xacro:arg name="gripper" default="robotiq_2f_85" /> -->
+    <xacro:arg name="gripper" default="" />
+    <xacro:arg name="gripper_joint_name" default="grasp_joint" />
     <xacro:arg name="use_fake_hardware" default="true" />
     <xacro:arg name="fake_sensor_commands" default="true" />
     <xacro:arg name="sim_gz" default="true" />
-    <xacro:arg name="sim_gazebo" default="false" />
-    <xacro:arg name="sim_ignition" default="false" />
     <xacro:arg name="sim_isaac" default="false" />
-    <xacro:arg name="gazebo_renderer" default="ogre" />
+    <xacro:arg name="use_internal_bus_gripper_comm" default="false" />
     <xacro:arg name="camera_width" default="640" />
     <xacro:arg name="camera_height" default="480" />
-    <xacro:arg name="camera_fps" default="6" />
+    <xacro:arg name="camera_fps" default="30" />
     <xacro:arg name="simulation_controllers"
         default="$(find eddie_gazebo)/config/eddie_controller.yaml" />
- <xacro:include filename="$(find kortex_description)/robots/kortex_robot.xacro" />
-  <xacro:include filename="$(find eddie_base_description)/urdf/common.xacro" />
+    <xacro:arg name="use_gpu_2d_laser" default="false" />
+    <xacro:include filename="$(find eddie_base_description)/urdf/common.xacro" />
     <xacro:include filename="$(find eddie_base_description)/urdf/eddie_base_gz.urdf.xacro" />
     <xacro:include filename="$(find eddie_torso_description)/urdf/eddie_torso_gz.urdf.xacro" />
-    <link name="base_link"/>
+    <xacro:include filename="$(find eddie_description)/robots/kortex_robot.xacro" />
+    <xacro:include filename="$(find eddie_description)/robots/kortex.ros2_gz_control.xacro" />
+    <xacro:include filename="$(find eddie_base_description)/urdf/materials.urdf.xacro" />
+    <link name="base_link" />
     <xacro:eddie_base name="eddie_base" parent="base_link"
         use_gpu_2d_laser="$(arg use_gpu_2d_laser)">
@@ -52,13 +50,13 @@
     <!-- convert to property to use substitution in function -->
     <xacro:property name="initial_positions_file_left" default="$(arg initial_positions_file_left)" />
-    <xacro:property name="initial_positions_file_right" default="$(arg initial_positions_file_right)" />
-   <!-- left arm  -->
-    <xacro:load_robot
+    <xacro:property name="initial_positions_file_right"
+        default="$(arg initial_positions_file_right)" />
+    <!-- left arm  -->
+    <xacro:kinova_arm
         parent="eddie_torso_shoulder_left_arm_attach_link"
+        prefix="$(arg prefix_arm_left)"
         arm="$(arg arm)"
-        gripper=""
+        gripper="$(arg gripper)"
         gripper_joint_name="$(arg gripper_joint_name)"
-        gripper_max_velocity="$(arg gripper_max_velocity)"
-        gripper_max_force="$(arg gripper_max_force)"
         dof="$(arg dof)"
         vision="$(arg vision)"
@@ -70,23 +68,33 @@
         session_inactivity_timeout_ms="$(arg session_inactivity_timeout_ms)"
         connection_inactivity_timeout_ms="$(arg connection_inactivity_timeout_ms)"
-        use_internal_bus_gripper_comm="$(arg use_internal_bus_gripper_comm)"
+        use_fake_hardware="$(arg use_fake_hardware)"
+        fake_sensor_commands="$(arg fake_sensor_commands)"
+        initial_positions="${xacro.load_yaml(initial_positions_file_left)}">
+        <origin xyz="0 0 0" rpy="0 0 0" />
+    </xacro:kinova_arm>
+    <xacro:kortex_ros2_control
+        name="$(arg prefix_arm_left)KortexMultiInterfaceHardware"
         prefix="$(arg prefix_arm_left)"
         use_fake_hardware="$(arg use_fake_hardware)"
         fake_sensor_commands="$(arg fake_sensor_commands)"
         sim_gz="$(arg sim_gz)"
-        sim_gazebo="$(arg sim_gazebo)"
-        sim_ignition="$(arg sim_ignition)"
-        sim_isaac="$(arg sim_isaac)"
-        initial_positions="${xacro.load_yaml(initial_positions_file_left)}">
-        <origin xyz="0 0 0" rpy="0 0 0" />
-    </xacro:load_robot>
+        tf_prefix=""
+        initial_positions="${xacro.load_yaml(initial_positions_file_left)}"
+        robot_ip="$(arg robot_ip_left)"
+        username="$(arg username)"
+        password="$(arg password)"
+        port="$(arg port)"
+        port_realtime="$(arg port_realtime)"
+        session_inactivity_timeout_ms="$(arg session_inactivity_timeout_ms)"
+        connection_inactivity_timeout_ms="$(arg connection_inactivity_timeout_ms)"
+        use_internal_bus_gripper_comm="$(arg use_internal_bus_gripper_comm)"
+        gripper_joint_name="$(arg gripper_joint_name)"/>
     <!-- right arm -->
-    <xacro:load_robot
+    <xacro:kinova_arm
         parent="eddie_torso_shoulder_right_arm_attach_link"
+        prefix="$(arg prefix_arm_right)"
         arm="$(arg arm)"
-        gripper=""
+        gripper="$(arg gripper)"
         gripper_joint_name="$(arg gripper_joint_name)"
-        gripper_max_velocity="$(arg gripper_max_velocity)"
-        gripper_max_force="$(arg gripper_max_force)"
         dof="$(arg dof)"
         vision="$(arg vision)"
@@ -98,18 +106,30 @@
         session_inactivity_timeout_ms="$(arg session_inactivity_timeout_ms)"
         connection_inactivity_timeout_ms="$(arg connection_inactivity_timeout_ms)"
-        use_internal_bus_gripper_comm="$(arg use_internal_bus_gripper_comm)"
+        use_fake_hardware="$(arg use_fake_hardware)"
+        fake_sensor_commands="$(arg fake_sensor_commands)"
+        initial_positions="${xacro.load_yaml(initial_positions_file_right)}">
+        <origin xyz="0 0 0" rpy="0 0 0" />
+    </xacro:kinova_arm>
+    <xacro:kortex_ros2_control
+        name="$(arg prefix_arm_right)KortexMultiInterfaceHardware"
         prefix="$(arg prefix_arm_right)"
         use_fake_hardware="$(arg use_fake_hardware)"
         fake_sensor_commands="$(arg fake_sensor_commands)"
         sim_gz="$(arg sim_gz)"
-        sim_gazebo="$(arg sim_gazebo)"
-        sim_ignition="$(arg sim_ignition)"
-        sim_isaac="$(arg sim_isaac)"
-        initial_positions="${xacro.load_yaml(initial_positions_file_right)}">
-        <origin xyz="0 0 0" rpy="0 0 0" />
-    </xacro:load_robot>
+        tf_prefix=""
+        initial_positions="${xacro.load_yaml(initial_positions_file_right)}"
+        robot_ip="$(arg robot_ip_right)"
+        username="$(arg username)"
+        password="$(arg password)"
+        port="$(arg port)"
+        port_realtime="$(arg port_realtime)"
+        session_inactivity_timeout_ms="$(arg session_inactivity_timeout_ms)"
+        connection_inactivity_timeout_ms="$(arg connection_inactivity_timeout_ms)"
+        use_internal_bus_gripper_comm="$(arg use_internal_bus_gripper_comm)"
+        gripper_joint_name="$(arg gripper_joint_name)"/>
     <!-- gazebo tag for ros2 control -->
     <gazebo>
-        <plugin filename="gz_ros2_control-system" name="gz_ros2_control::GazeboSimROS2ControlPlugin">
+        <plugin filename="libgz_ros2_control-system.so"
+            name="gz_ros2_control::GazeboSimROS2ControlPlugin">
             <robot_param>robot_description</robot_param>
             <robot_param_node>robot_state_publisher</robot_param_node>
@@ -118,3 +138,19 @@
         <self_collide>1</self_collide>
     </gazebo>
+    <gazebo reference="base_link">
+        <gravity>true</gravity>
+        <self_collide>false</self_collide>
+    </gazebo>
+    <gazebo>
+        <plugin
+            filename="gz-sim-odometry-publisher-system"
+            name="gz::sim::systems::OdometryPublisher">
+            <odom_frame>odom</odom_frame>
+            <robot_base_frame>eddie_base_link</robot_base_frame>
+        </plugin>
+        <plugin
+            filename="gz-sim-velocity-control-system"
+            name="gz::sim::systems::VelocityControl">
+        </plugin>
+    </gazebo>
 </robot>

File: eddie_torso_description/urdf/eddie_torso_gz.urdf.xacro (robot description, xacro)
@@ -29,4 +29,5 @@
                     <box size="${torso_thickness} ${torso_width} ${torso_height}" />
                 </geometry>
+                <material name="Grey"/>
             </visual>
             <!-- torso collision -->
@@ -59,4 +60,5 @@
                         size="${torso_shoulder_thickness} ${torso_shoulder_width} ${torso_shoulder_height}" />
                 </geometry>
+                <material name="DarkGrey"/>
             </visual>
             <!-- torso shoulder collision -->
@@ -98,4 +100,5 @@
                         size="${torso_shoulder_thickness} ${torso_shoulder_width} ${torso_shoulder_height}" />
                 </geometry>
+                <material name="DarkGrey"/>
             </visual>
             <!-- torso shoulder collision -->
