Commit message: updated material colors

File: urdf/materials.xacro (robot description, xacro)
@@ -2,14 +2,11 @@
 <robot xmlns:xacro="http://www.ros.org/wiki/xacro" name="eddie_materials">
     <material name="metallic_silver">
-        <color rgba="0.7 0.7 0.7 1.0" />
+        <color rgba="0.5 0.5 0.5 1.0" />
     </material>
     <material name="light_gray">
-        <color rgba="0.35 0.35 0.35 1.0" />
-    </material>
-    <material name="dark_gray">
-        <color rgba="0.15 0.15 0.15 1.0" />
+        <color rgba="0.25 0.25 0.25 1.0" />
     </material>
     <material name="almost_black">
-        <color rgba="0.05 0.05 0.05 0.8" />
+        <color rgba="0.075 0.075 0.075 1.0" />
     </material>
 </robot>
