Commit message: update folder structure

File: urdf/eddie_base.macro.xacro (robot description, xacro)
@@ -2,8 +2,8 @@
 <robot xmlns:xacro="http://www.ros.org/wiki/xacro" name="eddie_base_with_wheels">
     <!-- Include the Wheel and Structure Configuration -->
-    <xacro:include filename="$(find eddie_base_description)/urdf/wheels_with_kelo_drive.macro.xacro"/>
+    <xacro:include filename="$(find eddie_description)/urdf/wheels_with_kelo_drive.macro.xacro"/>
     <xacro:macro name="eddie_with_no_arm" params="">
         <!-- Properties -->
-        <xacro:property name="mesh_package" value="eddie_base_description"/>
+        <xacro:property name="mesh_package" value="eddie_description"/>
         <xacro:property name="eddie_base_file" value="kelo_base.stl"/>
         <xacro:property name="eddie_torso_file" value="kelo_torso.stl"/>
@@ -85,6 +85,4 @@
             <child link="${corner2_prefix}struct_attachment_plate_link"/>
             <origin xyz="${corner2_origin_xyz}" rpy="${corner2_orientation_rpy}"/>
-            <axis xyz="0 0 1"/> <!-- Rotate about the z-axis -->
-            <limit effort="10" velocity="1.0" lower="-3.14" upper="3.14"/>
         </joint>
         <joint name="corner3_joint" type="fixed">

File: urdf/eddie_robot.urdf.xacro (robot description, xacro)
@@ -2,5 +2,5 @@
 <robot xmlns:xacro="http://www.ros.org/wiki/xacro" name="eddie_base_with_wheels">
     <!-- Include the Eddie Base -->
-    <xacro:include filename="$(find eddie_base_description)/urdf/eddie_base.macro.xacro"/>
+    <xacro:include filename="$(find eddie_description)/urdf/eddie_base.macro.xacro"/>
     <xacro:eddie_with_no_arm/>
 </robot>

File: urdf/wheel.macro.xacro (robot description, xacro)
@@ -5,5 +5,5 @@
     <xacro:macro name="wheel" params="wheel_prefix">
         <!-- Properties -->
-        <xacro:property name="mesh_package" value="eddie_base_description"/>
+        <xacro:property name="mesh_package" value="eddie_description"/>
         <xacro:property name="wheel_mesh_file" value="hub_wheel.stl"/>
         <!-- Wheel Link with the specified prefix -->

File: urdf/wheels_with_kelo_drive.macro.xacro (robot description, xacro)
@@ -2,8 +2,8 @@
 <robot xmlns:xacro="http://www.ros.org/wiki/xacro" name="wheels_with_kelo_drive">
     <!-- Include the Wheel -->
-    <xacro:include filename="$(find eddie_base_description)/urdf/wheel.macro.xacro"/>
+    <xacro:include filename="$(find eddie_description)/urdf/wheel.macro.xacro"/>
     <xacro:macro name="wheels_with_kelo_drive" params="struct_prefix">
         <!-- Properties -->
-        <xacro:property name="mesh_package" value="eddie_base_description"/>
+        <xacro:property name="mesh_package" value="eddie_description"/>
         <xacro:property name="struct_mesh_file" value="kelo_drive.stl"/>
         <xacro:property name="struct_attachment_plate_mesh_file" value="kelo_drive_attachment_plates.stl"/>

Commit message: rename and add world frame

File: urdf/eddie_base.macro.xacro (robot description, xacro)
@@ -8,4 +8,5 @@
         <xacro:property name="eddie_base_file" value="kelo_base.stl"/>
         <xacro:property name="eddie_torso_file" value="kelo_torso.stl"/>
+        <link name="world_link"/>
         <!-- Additional Component at Center -->
         <link name="base_link">
@@ -24,8 +25,8 @@
                 </geometry>
             </collision>
-            <!-- <inertial>
+            <inertial>
                 <mass value="1.0"/>
                 <inertia ixx="0" ixy="0" ixz="0" iyy="0" iyz="0" izz="0"/>
-            </inertial> -->
+            </inertial>
         </link>
         <link name="torso_link">
@@ -51,8 +52,8 @@
         <link name="left_arm_link" />
         <link name="right_arm_link" />
-        <xacro:property name="corner1_prefix" value="front_left_cnr_"/>
-        <xacro:property name="corner2_prefix" value="rear_left_cnr_"/>
-        <xacro:property name="corner3_prefix" value="rear_right_cnr_"/>
-        <xacro:property name="corner4_prefix" value="front_right_cnr_"/>
+        <xacro:property name="corner1_prefix" value="front_left_"/>
+        <xacro:property name="corner2_prefix" value="rear_left_"/>
+        <xacro:property name="corner3_prefix" value="rear_right_"/>
+        <xacro:property name="corner4_prefix" value="front_right_"/>
         <xacro:property name="corner1_origin_xyz" value="0.2078 0.1880 -0.0632"/>
         <xacro:property name="corner2_origin_xyz" value="-0.2078 0.1880 -0.0632"/>
@@ -65,4 +66,6 @@
         <xacro:property name="torso_origin_xyz" value="-0.1738 0.0003 0.4184"/>
         <xacro:property name="torso_orientation_rpy" value="0 0 1.5708"/>
+        <xacro:property name="base_link_origin_xyz" value="0 0 0.2164"/>
+        <xacro:property name="base_link_orientation_rpy" value="0 0 0"/>
         <!-- Four instances of the wheel units -->
         <xacro:wheels_with_kelo_drive struct_prefix="${corner1_prefix}"/>
@@ -71,4 +74,9 @@
         <xacro:wheels_with_kelo_drive struct_prefix="${corner4_prefix}"/>
         <!-- Joints -->
+        <joint name="world_frame" type="fixed">
+            <parent link="world_link"/>
+            <child link="base_link"/>
+            <origin xyz="${base_link_origin_xyz}" rpy="${base_link_orientation_rpy}"/>
+        </joint>
         <joint name="base_torso_joint" type="fixed">
             <parent link="base_link"/>
@@ -78,20 +86,20 @@
         <joint name="corner1_joint" type="fixed">
             <parent link="base_link"/>
-            <child link="${corner1_prefix}struct_attachment_plate_link"/>
+            <child link="${corner1_prefix}struct_attachment_link"/>
             <origin xyz="${corner1_origin_xyz}" rpy="${corner1_orientation_rpy}"/>
         </joint>
         <joint name="corner2_joint" type="fixed">
             <parent link="base_link"/>
-            <child link="${corner2_prefix}struct_attachment_plate_link"/>
+            <child link="${corner2_prefix}struct_attachment_link"/>
             <origin xyz="${corner2_origin_xyz}" rpy="${corner2_orientation_rpy}"/>
         </joint>
         <joint name="corner3_joint" type="fixed">
             <parent link="base_link"/>
-            <child link="${corner3_prefix}struct_attachment_plate_link"/>
+            <child link="${corner3_prefix}struct_attachment_link"/>
             <origin xyz="${corner3_origin_xyz}" rpy="${corner3_orientation_rpy}"/>
         </joint>
         <joint name="corner4_joint" type="fixed">
             <parent link="base_link"/>
-            <child link="${corner4_prefix}struct_attachment_plate_link"/>
+            <child link="${corner4_prefix}struct_attachment_link"/>
             <origin xyz="${corner4_origin_xyz}" rpy="${corner4_orientation_rpy}"/>
         </joint>

File: urdf/wheels_with_kelo_drive.macro.xacro (robot description, xacro)
@@ -7,11 +7,11 @@
         <xacro:property name="mesh_package" value="eddie_description"/>
         <xacro:property name="struct_mesh_file" value="kelo_drive.stl"/>
-        <xacro:property name="struct_attachment_plate_mesh_file" value="kelo_drive_attachment_plates.stl"/>
+        <xacro:property name="struct_attachment_mesh_file" value="kelo_drive_attachments.stl"/>
         <!-- Attachment plate link -->
-        <link name="${struct_prefix}struct_attachment_plate_link">
+        <link name="${struct_prefix}struct_attachment_link">
             <visual>
                 <origin rpy="0 0 0" xyz="0 0 0"/>
                 <geometry>
-                    <mesh filename="package://${mesh_package}/meshes/${struct_attachment_plate_mesh_file}" />
+                    <mesh filename="package://${mesh_package}/meshes/${struct_attachment_mesh_file}" />
                 </geometry>
                 <material name="metallic_silver">
@@ -21,5 +21,5 @@
             <collision>
                 <geometry>
-                    <mesh filename="package://${mesh_package}/meshes/${struct_attachment_plate_mesh_file}"/>
+                    <mesh filename="package://${mesh_package}/meshes/${struct_attachment_mesh_file}"/>
                 </geometry>
             </collision>
@@ -51,6 +51,6 @@
         </link>
         <!-- Attachment plate location -->
-        <xacro:property name="attachment_plate_origin_xyz" value="-0.0100 -0.0006 -0.0641"/>
-        <xacro:property name="attachment_plate_orientation_rpy" value="0 0 1.5708"/>
+        <xacro:property name="attachment_origin_xyz" value="-0.0100 -0.0006 -0.0641"/>
+        <xacro:property name="attachment_orientation_rpy" value="0 0 1.5708"/>
         <!-- Right Wheel Instance -->
         <xacro:property name="wheel_prefix_right" value="${struct_prefix}right_"/>
@@ -64,8 +64,8 @@
         <xacro:wheel wheel_prefix="${wheel_prefix_left}"/>
         <!-- Joints -->
-        <joint name="${struct_prefix}struct_to_attachment_plate_joint" type="continuous">
-            <parent link="${struct_prefix}struct_attachment_plate_link"/>
+        <joint name="${struct_prefix}struct_to_attachment_joint" type="continuous">
+            <parent link="${struct_prefix}struct_attachment_link"/>
             <child link="${struct_prefix}struct_link"/>
-            <origin xyz="${attachment_plate_origin_xyz}" rpy="${attachment_plate_orientation_rpy}"/>
+            <origin xyz="${attachment_origin_xyz}" rpy="${attachment_orientation_rpy}"/>
             <axis xyz="0 0 1"/>
         </joint>

Commit message: renaming files and macros

File: urdf/eddie_base.macro.xacro (robot description, xacro)
@@ -1,14 +1,15 @@
 <?xml version="1.0"?>
-<robot xmlns:xacro="http://www.ros.org/wiki/xacro" name="eddie_base_with_wheels">
+<robot xmlns:xacro="http://www.ros.org/wiki/xacro" name="eddie_base">
     <!-- Include the Wheel and Structure Configuration -->
-    <xacro:include filename="$(find eddie_description)/urdf/wheels_with_kelo_drive.macro.xacro"/>
-    <xacro:macro name="eddie_with_no_arm" params="">
+    <xacro:include filename="$(find eddie_description)/urdf/kelo_drive_unit.macro.xacro"/>
+    <xacro:macro name="eddie_base" params="prefix">
         <!-- Properties -->
         <xacro:property name="mesh_package" value="eddie_description"/>
         <xacro:property name="eddie_base_file" value="kelo_base.stl"/>
         <xacro:property name="eddie_torso_file" value="kelo_torso.stl"/>
-        <link name="world_link"/>
+        <!-- Base Footprint -->
+        <link name="${prefix}base_footprint"/>
         <!-- Additional Component at Center -->
-        <link name="base_link">
+        <link name="${prefix}base_link">
             <visual>
                 <origin rpy="0 0 0" xyz="0 0 0"/>
@@ -22,5 +23,6 @@
             <collision>
                 <geometry>
-                    <box size="0.622 0.659 0.308" />
+                    <!-- <box size="0.622 0.659 0.308" /> -->
+                    <mesh filename="package://${mesh_package}/meshes/${eddie_base_file}"/>
                 </geometry>
             </collision>
@@ -30,5 +32,5 @@
             </inertial>
         </link>
-        <link name="torso_link">
+        <link name="${prefix}torso_link">
             <visual>
                 <origin rpy="0 0 0" xyz="0 0 0"/>
@@ -50,18 +52,14 @@
             </inertial>
         </link>
-        <link name="left_arm_link" />
-        <link name="right_arm_link" />
-        <xacro:property name="corner1_prefix" value="front_left_"/>
-        <xacro:property name="corner2_prefix" value="rear_left_"/>
-        <xacro:property name="corner3_prefix" value="rear_right_"/>
-        <xacro:property name="corner4_prefix" value="front_right_"/>
-        <xacro:property name="corner1_origin_xyz" value="0.2078 0.1880 -0.0632"/>
-        <xacro:property name="corner2_origin_xyz" value="-0.2078 0.1880 -0.0632"/>
-        <xacro:property name="corner3_origin_xyz" value="-0.2078 -0.1880 -0.0632"/>
-        <xacro:property name="corner4_origin_xyz" value="0.2078 -0.1880 -0.0632"/>
-        <xacro:property name="corner1_orientation_rpy" value="0 0 1.5708"/>
-        <xacro:property name="corner2_orientation_rpy" value="0 0 1.5708"/>
-        <xacro:property name="corner3_orientation_rpy" value="0 0 -1.5708"/>
-        <xacro:property name="corner4_orientation_rpy" value="0 0 -1.5708"/>
+        <link name="${prefix}left_arm_attachment_link" />
+        <link name="${prefix}right_arm_attachment_link" />
+        <xacro:property name="front_left_origin_xyz" value="0.2078 0.1880 -0.0632"/>
+        <xacro:property name="rear_left_origin_xyz" value="-0.2078 0.1880 -0.0632"/>
+        <xacro:property name="rear_right_origin_xyz" value="-0.2078 -0.1880 -0.0632"/>
+        <xacro:property name="front_right_origin_xyz" value="0.2078 -0.1880 -0.0632"/>
+        <xacro:property name="front_left_orientation_rpy" value="0 0 1.5708"/>
+        <xacro:property name="rear_left_orientation_rpy" value="0 0 1.5708"/>
+        <xacro:property name="rear_right_orientation_rpy" value="0 0 -1.5708"/>
+        <xacro:property name="front_right_orientation_rpy" value="0 0 -1.5708"/>
         <xacro:property name="torso_origin_xyz" value="-0.1738 0.0003 0.4184"/>
         <xacro:property name="torso_orientation_rpy" value="0 0 1.5708"/>
@@ -69,50 +67,49 @@
         <xacro:property name="base_link_orientation_rpy" value="0 0 0"/>
         <!-- Four instances of the wheel units -->
-        <xacro:wheels_with_kelo_drive struct_prefix="${corner1_prefix}"/>
-        <xacro:wheels_with_kelo_drive struct_prefix="${corner2_prefix}"/>
-        <xacro:wheels_with_kelo_drive struct_prefix="${corner3_prefix}"/>
-        <xacro:wheels_with_kelo_drive struct_prefix="${corner4_prefix}"/>
+        <xacro:kelo_drive_unit struct_prefix="${prefix}front_left_"/>
+        <xacro:kelo_drive_unit struct_prefix="${prefix}rear_left_"/>
+        <xacro:kelo_drive_unit struct_prefix="${prefix}rear_right_"/>
+        <xacro:kelo_drive_unit struct_prefix="${prefix}front_right_"/>
         <!-- Joints -->
-        <joint name="world_frame" type="fixed">
-            <parent link="world_link"/>
-            <child link="base_link"/>
+        <joint name="${prefix}base_footprint_joint" type="fixed">
+            <parent link="${prefix}base_footprint"/>
+            <child link="${prefix}base_link"/>
             <origin xyz="${base_link_origin_xyz}" rpy="${base_link_orientation_rpy}"/>
         </joint>
-        <joint name="base_torso_joint" type="fixed">
-            <parent link="base_link"/>
-            <child link="torso_link"/>
+        <joint name="${prefix}base_torso_joint" type="fixed">
+            <parent link="${prefix}base_link"/>
+            <child link="${prefix}torso_link"/>
             <origin xyz="${torso_origin_xyz}" rpy="${torso_orientation_rpy}"/>
         </joint>
-        <joint name="corner1_joint" type="fixed">
-            <parent link="base_link"/>
-            <child link="${corner1_prefix}struct_attachment_link"/>
-            <origin xyz="${corner1_origin_xyz}" rpy="${corner1_orientation_rpy}"/>
+        <joint name="${prefix}front_left_joint" type="fixed">
+            <parent link="${prefix}base_link"/>
+            <child link="${prefix}${front_left_prefix}struct_attachment_link"/>
+            <origin xyz="${front_left_origin_xyz}" rpy="${front_left_orientation_rpy}"/>
         </joint>
-        <joint name="corner2_joint" type="fixed">
-            <parent link="base_link"/>
-            <child link="${corner2_prefix}struct_attachment_link"/>
-            <origin xyz="${corner2_origin_xyz}" rpy="${corner2_orientation_rpy}"/>
+        <joint name="${prefix}rear_left_joint" type="fixed">
+            <parent link="${prefix}base_link"/>
+            <child link="${prefix}${rear_left_prefix}struct_attachment_link"/>
+            <origin xyz="${rear_left_origin_xyz}" rpy="${rear_left_orientation_rpy}"/>
         </joint>
-        <joint name="corner3_joint" type="fixed">
-            <parent link="base_link"/>
-            <child link="${corner3_prefix}struct_attachment_link"/>
-            <origin xyz="${corner3_origin_xyz}" rpy="${corner3_orientation_rpy}"/>
+        <joint name="${prefix}rear_right_joint" type="fixed">
+            <parent link="${prefix}base_link"/>
+            <child link="${prefix}${rear_right_prefix}struct_attachment_link"/>
+            <origin xyz="${rear_right_origin_xyz}" rpy="${rear_right_orientation_rpy}"/>
         </joint>
-        <joint name="corner4_joint" type="fixed">
-            <parent link="base_link"/>
-            <child link="${corner4_prefix}struct_attachment_link"/>
-            <origin xyz="${corner4_origin_xyz}" rpy="${corner4_orientation_rpy}"/>
+        <joint name="${prefix}front_right_joint" type="fixed">
+            <parent link="${prefix}base_link"/>
+            <child link="${prefix}${front_right_prefix}struct_attachment_link"/>
+            <origin xyz="${front_right_origin_xyz}" rpy="${front_right_orientation_rpy}"/>
         </joint>
-        <joint name="left_arm_joint" type="fixed">
-            <parent link="torso_link"/>
-            <child link="left_arm_link"/>
+        <joint name="${prefix}left_arm_attachment_joint" type="fixed">
+            <parent link="${prefix}torso_link"/>
+            <child link="${prefix}left_arm_attachment_link"/>
             <origin xyz="0.0676 -0.0236 0.1160" rpy="0 0.09 -0.7783"/>
         </joint>
-        <joint name="right_arm_joint" type="fixed">
-            <parent link="torso_link"/>
-            <child link="right_arm_link"/>
+        <joint name="${prefix}right_arm_attachment_joint" type="fixed">
+            <parent link="${prefix}torso_link"/>
+            <child link="${prefix}right_arm_attachment_link"/>
             <origin xyz="-0.0676 -0.0236 0.1160" rpy="0 0.09 -2.3632"/>
         </joint>
     </xacro:macro>
-    <!-- <xacro:eddie_with_no_arm/> -->
 </robot>

File: urdf/eddie_robot.urdf.xacro (robot description, xacro)
@@ -3,4 +3,4 @@
     <!-- Include the Eddie Base -->
     <xacro:include filename="$(find eddie_description)/urdf/eddie_base.macro.xacro"/>
-    <xacro:eddie_with_no_arm/>
+    <xacro:eddie_base prefix="eddie_"/>
 </robot>

File: urdf/kelo_drive_unit.macro.xacro (robot description, xacro)
@@ -1,7 +1,7 @@
 <?xml version="1.0"?>
-<robot xmlns:xacro="http://www.ros.org/wiki/xacro" name="wheels_with_kelo_drive">
+<robot xmlns:xacro="http://www.ros.org/wiki/xacro" name="kelo_drive_unit">
     <!-- Include the Wheel -->
-    <xacro:include filename="$(find eddie_description)/urdf/wheel.macro.xacro"/>
-    <xacro:macro name="wheels_with_kelo_drive" params="struct_prefix">
+    <xacro:include filename="$(find eddie_description)/urdf/kelo_hub_wheel.macro.xacro"/>
+    <xacro:macro name="kelo_drive_unit" params="struct_prefix">
         <!-- Properties -->
         <xacro:property name="mesh_package" value="eddie_description"/>
@@ -57,10 +57,10 @@
         <xacro:property name="wheel_orientation_rpy_right" value="-1.5708 0 0"/>
         <xacro:property name="wheel_origin_xyz_right" value="0.0008 -0.0403 -0.0366"/>
-        <xacro:wheel wheel_prefix="${wheel_prefix_right}"/>
+        <xacro:kelo_hub_wheel wheel_prefix="${wheel_prefix_right}"/>
         <!-- Left Wheel Instance -->
         <xacro:property name="wheel_prefix_left" value="${struct_prefix}left_"/>
         <xacro:property name="wheel_orientation_rpy_left" value="1.5708 0 0"/>
         <xacro:property name="wheel_origin_xyz_left" value="0.0008 0.0407 -0.0366"/>
-        <xacro:wheel wheel_prefix="${wheel_prefix_left}"/>
+        <xacro:kelo_hub_wheel wheel_prefix="${wheel_prefix_left}"/>
         <!-- Joints -->
         <joint name="${struct_prefix}struct_to_attachment_joint" type="continuous">
@@ -83,4 +83,3 @@
         </joint>
     </xacro:macro>
-    <!-- <xacro:wheels_with_kelo_drive struct_prefix=""/> -->
 </robot>

File: urdf/kelo_hub_wheel.macro.xacro (robot description, xacro)
@@ -1,7 +1,7 @@
 <?xml version="1.0"?>
-<robot xmlns:xacro="http://www.ros.org/wiki/xacro" name="wheel">
+<robot xmlns:xacro="http://www.ros.org/wiki/xacro" name="kelo_hub_wheel">
     <xacro:arg name="wheel_prefix" default=""/>
     <!-- Define a macro for creating a wheel link with a prefix parameter -->
-    <xacro:macro name="wheel" params="wheel_prefix">
+    <xacro:macro name="kelo_hub_wheel" params="wheel_prefix">
         <!-- Properties -->
         <xacro:property name="mesh_package" value="eddie_description"/>
@@ -29,5 +29,3 @@
         </link>
     </xacro:macro>
-    <!-- Instantiate the wheel macro with a specified prefix -->
-    <!-- <xacro:wheel wheel_prefix=""/> -->
 </robot>
