Commit message: configure arms

File: urdf/eddie_base.macro.xacro (robot description, xacro)
@@ -84,20 +84,20 @@
         <joint name="${prefix}front_left_joint" type="fixed">
             <parent link="${prefix}base_link"/>
-            <child link="${prefix}${front_left_prefix}struct_attachment_link"/>
+            <child link="${prefix}front_left_struct_attachment_link"/>
             <origin xyz="${front_left_origin_xyz}" rpy="${front_left_orientation_rpy}"/>
         </joint>
         <joint name="${prefix}rear_left_joint" type="fixed">
             <parent link="${prefix}base_link"/>
-            <child link="${prefix}${rear_left_prefix}struct_attachment_link"/>
+            <child link="${prefix}rear_left_struct_attachment_link"/>
             <origin xyz="${rear_left_origin_xyz}" rpy="${rear_left_orientation_rpy}"/>
         </joint>
         <joint name="${prefix}rear_right_joint" type="fixed">
             <parent link="${prefix}base_link"/>
-            <child link="${prefix}${rear_right_prefix}struct_attachment_link"/>
+            <child link="${prefix}rear_right_struct_attachment_link"/>
             <origin xyz="${rear_right_origin_xyz}" rpy="${rear_right_orientation_rpy}"/>
         </joint>
         <joint name="${prefix}front_right_joint" type="fixed">
             <parent link="${prefix}base_link"/>
-            <child link="${prefix}${front_right_prefix}struct_attachment_link"/>
+            <child link="${prefix}front_right_struct_attachment_link"/>
             <origin xyz="${front_right_origin_xyz}" rpy="${front_right_orientation_rpy}"/>
         </joint>

File: urdf/eddie_robot.urdf.xacro (robot description, xacro)
@@ -23,12 +23,16 @@
     <xacro:arg name="initial_positions_file_right"
         default="$(find eddie_description)/config/initial_positions_arm_right.yaml" />
+    <!-- convert to property to use substitution in function -->
+    <xacro:property name="initial_positions_file_left" default="$(arg initial_positions_file_left)" />
+    <xacro:property name="initial_positions_file_right"
+        default="$(arg initial_positions_file_right)" />
     <!-- Include the Eddie Base -->
     <xacro:include filename="$(find eddie_description)/urdf/eddie_base.macro.xacro"/>
     <!-- Include Gen3 Arm -->
-    <xacro:include filename="$(find kortex_description)/urdf/kinova_gen3.macro.xacro"/>
-    <xacro:eddie_base prefix="${xacro:arg robot_name}" />
+    <xacro:include filename="$(find eddie_description)/urdf/kinova_gen3.macro.xacro"/>
+    <xacro:eddie_base prefix="$(arg robot_name)" />
     <xacro:kinova_gen3
-        parent="${xacro:arg robot_name}left_arm_attachment_link"
-        prefix="${xacro:arg robot_name}left_arm_"
+        parent="$(arg robot_name)left_arm_attachment_link"
+        prefix="$(arg robot_name)left_arm_"
         gripper="robotiq_2f_85"
         robot_ip="$(arg robot_ip_left)"
@@ -41,12 +45,10 @@
         use_fake_hardware="$(arg use_fake_hardware)"
         fake_sensor_commands="$(arg fake_sensor_commands)"
-        initial_positions="${xacro.load_yaml(initial_positions_file_left)}"
-        >
-        <!-- TODO: Update origin -->
-        <origin xyz="0 0 0" rpy="0 0 0" />
+        initial_positions="${xacro.load_yaml(initial_positions_file_left)}">
+        <origin xyz="0.01549 0 0" rpy="1.5708 -1.5708 1.5708" />
     </xacro:kinova_gen3>
     <xacro:kinova_gen3
-        parent="${xacro:arg robot_name}right_arm_attachment_link"
-        prefix="${xacro:arg robot_name}right_arm_"
+        parent="$(arg robot_name)right_arm_attachment_link"
+        prefix="$(arg robot_name)right_arm_"
         gripper="robotiq_2f_85"
         robot_ip="$(arg robot_ip_right)"
@@ -59,8 +61,6 @@
         use_fake_hardware="$(arg use_fake_hardware)"
         fake_sensor_commands="$(arg fake_sensor_commands)"
-        initial_positions="${xacro.load_yaml(initial_positions_file_right)}"
-        >
-        <!-- TODO: Update origin -->
-        <origin xyz="0 0 0" rpy="0 0 0" />
+        initial_positions="${xacro.load_yaml(initial_positions_file_right)}">
+        <origin xyz="0.01549 0 0" rpy="1.5708 -1.5708 1.5708" />
     </xacro:kinova_gen3>
 </robot>

File: urdf/kelo_drive_unit.macro.xacro (robot description, xacro)
@@ -8,5 +8,13 @@
         <xacro:property name="struct_mesh_file" value="kelo_drive.stl"/>
         <xacro:property name="struct_attachment_mesh_file" value="kelo_drive_attachments.stl"/>
-        <!-- Attachment plate link -->
+        <xacro:property name="attachment_origin_xyz" value="-0.0100 -0.0006 -0.0641"/>
+        <xacro:property name="attachment_orientation_rpy" value="0 0 1.5708"/>
+        <xacro:property name="wheel_prefix_left" value="${struct_prefix}left_"/>
+        <xacro:property name="wheel_prefix_right" value="${struct_prefix}right_"/>
+        <xacro:property name="wheel_orientation_rpy_right" value="-1.5708 0 0"/>
+        <xacro:property name="wheel_origin_xyz_right" value="0.0008 -0.0403 -0.0366"/>
+        <xacro:property name="wheel_orientation_rpy_left" value="1.5708 0 0"/>
+        <xacro:property name="wheel_origin_xyz_left" value="0.0008 0.0407 -0.0366"/>
+        <!-- Links -->
         <link name="${struct_prefix}struct_attachment_link">
             <visual>
@@ -29,5 +37,4 @@
             </inertial>
         </link>
-        <!-- Structure Link -->
         <link name="${struct_prefix}struct_link">
             <visual>
@@ -50,16 +57,6 @@
             </inertial>
         </link>
-        <!-- Attachment plate location -->
-        <xacro:property name="attachment_origin_xyz" value="-0.0100 -0.0006 -0.0641"/>
-        <xacro:property name="attachment_orientation_rpy" value="0 0 1.5708"/>
-        <!-- Right Wheel Instance -->
-        <xacro:property name="wheel_prefix_right" value="${struct_prefix}right_"/>
-        <xacro:property name="wheel_orientation_rpy_right" value="-1.5708 0 0"/>
-        <xacro:property name="wheel_origin_xyz_right" value="0.0008 -0.0403 -0.0366"/>
+        <!-- Instantiate wheels -->
         <xacro:kelo_hub_wheel wheel_prefix="${wheel_prefix_right}"/>
-        <!-- Left Wheel Instance -->
-        <xacro:property name="wheel_prefix_left" value="${struct_prefix}left_"/>
-        <xacro:property name="wheel_orientation_rpy_left" value="1.5708 0 0"/>
-        <xacro:property name="wheel_origin_xyz_left" value="0.0008 0.0407 -0.0366"/>
         <xacro:kelo_hub_wheel wheel_prefix="${wheel_prefix_left}"/>
         <!-- Joints -->

File: urdf/kelo_hub_wheel.macro.xacro (robot description, xacro)
@@ -2,10 +2,9 @@
 <robot xmlns:xacro="http://www.ros.org/wiki/xacro" name="kelo_hub_wheel">
     <xacro:arg name="wheel_prefix" default=""/>
-    <!-- Define a macro for creating a wheel link with a prefix parameter -->
     <xacro:macro name="kelo_hub_wheel" params="wheel_prefix">
         <!-- Properties -->
         <xacro:property name="mesh_package" value="eddie_description"/>
         <xacro:property name="wheel_mesh_file" value="hub_wheel.stl"/>
-        <!-- Wheel Link with the specified prefix -->
+        <!-- Links -->
         <link name="${wheel_prefix}wheel_link">
             <visual>
