Commit message: refactor, add approx mass-inertia, todo: ctrl-gazebo

File: urdf/eddie_base.macro.xacro (robot description, xacro)
@@ -1,15 +1,38 @@
 <?xml version="1.0"?>
 <robot xmlns:xacro="http://www.ros.org/wiki/xacro" name="eddie_base">
-    <!-- Include the Wheel and Structure Configuration -->
+    <!-- Include macro files -->
     <xacro:include filename="$(find eddie_description)/urdf/kelo_drive_unit.macro.xacro"/>
-    <xacro:macro name="eddie_base" params="prefix">
+    <xacro:macro name="eddie_base" params="robot_prefix">
         <!-- Properties -->
         <xacro:property name="mesh_package" value="eddie_description"/>
         <xacro:property name="eddie_base_file" value="kelo_base.stl"/>
         <xacro:property name="eddie_torso_file" value="kelo_torso.stl"/>
-        <!-- Base Footprint -->
-        <link name="${prefix}base_footprint"/>
-        <!-- Additional Component at Center -->
-        <link name="${prefix}base_link">
+        <xacro:property name="front_left_origin_xyz" value="0.2078 0.1880 -0.0632"/>
+        <xacro:property name="rear_left_origin_xyz" value="-0.2078 0.1880 -0.0632"/>
+        <xacro:property name="rear_right_origin_xyz" value="-0.2078 -0.1880 -0.0632"/>
+        <xacro:property name="front_right_origin_xyz" value="0.2078 -0.1880 -0.0632"/>
+        <xacro:property name="front_left_orientation_rpy" value="0 0 1.5708"/>
+        <xacro:property name="rear_left_orientation_rpy" value="0 0 1.5708"/>
+        <xacro:property name="rear_right_orientation_rpy" value="0 0 -1.5708"/>
+        <xacro:property name="front_right_orientation_rpy" value="0 0 -1.5708"/>
+        <xacro:property name="front_right_attachment_cts_jnt_orientation_rpy" value="0 0 -1.5708"/>
+        <xacro:property name="front_left_attachment_cts_jnt_orientation_rpy" value="0 0 1.5708"/>
+        <xacro:property name="rear_right_attachment_cts_jnt_orientation_rpy" value="0 0 -1.5708"/>
+        <xacro:property name="rear_left_attachment_cts_jnt_orientation_rpy" value="0 0 1.5708"/>
+        <xacro:property name="torso_origin_xyz" value="-0.1738 0.0003 0.4184"/>
+        <xacro:property name="torso_orientation_rpy" value="0 0 1.5708"/>
+        <xacro:property name="base_link_origin_xyz" value="0 0 0.2164"/>
+        <xacro:property name="base_link_orientation_rpy" value="0 0 0"/>
+        <!-- Instantiate wheel units -->
+        <xacro:kelo_drive_unit robot_prefix="${robot_prefix}" struct_prefix="front_left_drive_" struct_origin_xyz="${front_left_origin_xyz}" struct_orientation_rpy="${front_left_orientation_rpy}" attachment_cts_jnt_orientation_rpy="${front_left_attachment_cts_jnt_orientation_rpy}"/>
+        <xacro:kelo_drive_unit robot_prefix="${robot_prefix}" struct_prefix="rear_left_drive_" struct_origin_xyz="${rear_left_origin_xyz}" struct_orientation_rpy="${rear_left_orientation_rpy}"  attachment_cts_jnt_orientation_rpy="${rear_left_attachment_cts_jnt_orientation_rpy}"/>
+        <xacro:kelo_drive_unit robot_prefix="${robot_prefix}" struct_prefix="rear_right_drive_" struct_origin_xyz="${rear_right_origin_xyz}" struct_orientation_rpy="${rear_right_orientation_rpy}"  attachment_cts_jnt_orientation_rpy="${front_right_attachment_cts_jnt_orientation_rpy}"/>
+        <xacro:kelo_drive_unit robot_prefix="${robot_prefix}" struct_prefix="front_right_drive_" struct_origin_xyz="${front_right_origin_xyz}" struct_orientation_rpy="${front_right_orientation_rpy}"  attachment_cts_jnt_orientation_rpy="${rear_right_attachment_cts_jnt_orientation_rpy}"/>
+        <!-- Links -->
+        <link name="${robot_prefix}base_footprint"/>
+        <link name="${robot_prefix}left_arm_attachment_link" />
+        <link name="${robot_prefix}right_arm_attachment_link" />
+        <link name="${robot_prefix}torso_link" />
+        <link name="${robot_prefix}base_link">
             <visual>
                 <origin rpy="0 0 0" xyz="0 0 0"/>
@@ -23,16 +46,9 @@
             <collision>
                 <geometry>
-                    <!-- <box size="0.622 0.659 0.308" /> -->
                     <mesh filename="package://${mesh_package}/meshes/${eddie_base_file}"/>
                 </geometry>
             </collision>
-            <inertial>
-                <mass value="1.0"/>
-                <inertia ixx="0" ixy="0" ixz="0" iyy="0" iyz="0" izz="0"/>
-            </inertial>
-        </link>
-        <link name="${prefix}torso_link">
             <visual>
-                <origin rpy="0 0 0" xyz="0 0 0"/>
+                <origin rpy="${torso_orientation_rpy}" xyz="${torso_origin_xyz}"/>
                 <geometry>
                     <mesh filename="package://${mesh_package}/meshes/${eddie_torso_file}" />
@@ -46,68 +62,31 @@
                     <mesh filename="package://${mesh_package}/meshes/${eddie_torso_file}"/>
                 </geometry>
+                <origin rpy="${torso_orientation_rpy}" xyz="${torso_origin_xyz}"/>
             </collision>
             <inertial>
-                <mass value="1.0"/>
-                <inertia ixx="0" ixy="0" ixz="0" iyy="0" iyz="0" izz="0"/>
+                <mass value="76.4377"/>
+                <origin xyz="-0.05172 0.0045 0.2378" rpy="0 0 0"/>
+                <inertia ixx="4.128795216" ixy="0" ixz="0" iyy="4.117596854" iyz="0" izz="3.364397364"/>
             </inertial>
         </link>
-        <link name="${prefix}left_arm_attachment_link" />
-        <link name="${prefix}right_arm_attachment_link" />
-        <xacro:property name="front_left_origin_xyz" value="0.2078 0.1880 -0.0632"/>
-        <xacro:property name="rear_left_origin_xyz" value="-0.2078 0.1880 -0.0632"/>
-        <xacro:property name="rear_right_origin_xyz" value="-0.2078 -0.1880 -0.0632"/>
-        <xacro:property name="front_right_origin_xyz" value="0.2078 -0.1880 -0.0632"/>
-        <xacro:property name="front_left_orientation_rpy" value="0 0 1.5708"/>
-        <xacro:property name="rear_left_orientation_rpy" value="0 0 1.5708"/>
-        <xacro:property name="rear_right_orientation_rpy" value="0 0 -1.5708"/>
-        <xacro:property name="front_right_orientation_rpy" value="0 0 -1.5708"/>
-        <xacro:property name="torso_origin_xyz" value="-0.1738 0.0003 0.4184"/>
-        <xacro:property name="torso_orientation_rpy" value="0 0 1.5708"/>
-        <xacro:property name="base_link_origin_xyz" value="0 0 0.2164"/>
-        <xacro:property name="base_link_orientation_rpy" value="0 0 0"/>
-        <!-- Four instances of the wheel units -->
-        <xacro:kelo_drive_unit struct_prefix="${prefix}front_left_"/>
-        <xacro:kelo_drive_unit struct_prefix="${prefix}rear_left_"/>
-        <xacro:kelo_drive_unit struct_prefix="${prefix}rear_right_"/>
-        <xacro:kelo_drive_unit struct_prefix="${prefix}front_right_"/>
         <!-- Joints -->
-        <joint name="${prefix}base_footprint_joint" type="fixed">
-            <parent link="${prefix}base_footprint"/>
-            <child link="${prefix}base_link"/>
+        <joint name="${robot_prefix}base_footprint_joint" type="fixed">
+            <parent link="${robot_prefix}base_footprint"/>
+            <child link="${robot_prefix}base_link"/>
             <origin xyz="${base_link_origin_xyz}" rpy="${base_link_orientation_rpy}"/>
         </joint>
-        <joint name="${prefix}base_torso_joint" type="fixed">
-            <parent link="${prefix}base_link"/>
-            <child link="${prefix}torso_link"/>
+        <joint name="${robot_prefix}base_torso_joint" type="fixed">
+            <parent link="${robot_prefix}base_link"/>
+            <child link="${robot_prefix}torso_link"/>
             <origin xyz="${torso_origin_xyz}" rpy="${torso_orientation_rpy}"/>
         </joint>
-        <joint name="${prefix}front_left_joint" type="fixed">
-            <parent link="${prefix}base_link"/>
-            <child link="${prefix}front_left_struct_attachment_link"/>
-            <origin xyz="${front_left_origin_xyz}" rpy="${front_left_orientation_rpy}"/>
-        </joint>
-        <joint name="${prefix}rear_left_joint" type="fixed">
-            <parent link="${prefix}base_link"/>
-            <child link="${prefix}rear_left_struct_attachment_link"/>
-            <origin xyz="${rear_left_origin_xyz}" rpy="${rear_left_orientation_rpy}"/>
-        </joint>
-        <joint name="${prefix}rear_right_joint" type="fixed">
-            <parent link="${prefix}base_link"/>
-            <child link="${prefix}rear_right_struct_attachment_link"/>
-            <origin xyz="${rear_right_origin_xyz}" rpy="${rear_right_orientation_rpy}"/>
-        </joint>
-        <joint name="${prefix}front_right_joint" type="fixed">
-            <parent link="${prefix}base_link"/>
-            <child link="${prefix}front_right_struct_attachment_link"/>
-            <origin xyz="${front_right_origin_xyz}" rpy="${front_right_orientation_rpy}"/>
-        </joint>
-        <joint name="${prefix}left_arm_attachment_joint" type="fixed">
-            <parent link="${prefix}torso_link"/>
-            <child link="${prefix}left_arm_attachment_link"/>
+        <joint name="${robot_prefix}left_arm_attachment_joint" type="fixed">
+            <parent link="${robot_prefix}torso_link"/>
+            <child link="${robot_prefix}left_arm_attachment_link"/>
             <origin xyz="0.0676 -0.0236 0.1160" rpy="0 0.09 -0.7783"/>
         </joint>
-        <joint name="${prefix}right_arm_attachment_joint" type="fixed">
-            <parent link="${prefix}torso_link"/>
-            <child link="${prefix}right_arm_attachment_link"/>
+        <joint name="${robot_prefix}right_arm_attachment_joint" type="fixed">
+            <parent link="${robot_prefix}torso_link"/>
+            <child link="${robot_prefix}right_arm_attachment_link"/>
             <origin xyz="-0.0676 -0.0236 0.1160" rpy="0 0.09 -2.3632"/>
         </joint>

File: urdf/eddie_robot.urdf.xacro (robot description, xacro)
@@ -31,5 +31,5 @@
     <!-- Include Gen3 Arm -->
     <xacro:include filename="$(find eddie_description)/urdf/kinova_gen3.macro.xacro"/>
-    <xacro:eddie_base prefix="$(arg robot_name)" />
+    <xacro:eddie_base robot_prefix="$(arg robot_name)" />
     <xacro:kinova_gen3
         parent="$(arg robot_name)left_arm_attachment_link"

File: urdf/kelo_drive_unit.macro.xacro (robot description, xacro)
@@ -1,7 +1,7 @@
 <?xml version="1.0"?>
 <robot xmlns:xacro="http://www.ros.org/wiki/xacro" name="kelo_drive_unit">
-    <!-- Include the Wheel -->
+    <!-- Include macro files -->
     <xacro:include filename="$(find eddie_description)/urdf/kelo_hub_wheel.macro.xacro"/>
-    <xacro:macro name="kelo_drive_unit" params="struct_prefix">
+    <xacro:macro name="kelo_drive_unit" params="robot_prefix struct_prefix struct_origin_xyz struct_orientation_rpy attachment_cts_jnt_orientation_rpy">
         <!-- Properties -->
         <xacro:property name="mesh_package" value="eddie_description"/>
@@ -9,13 +9,15 @@
         <xacro:property name="struct_attachment_mesh_file" value="kelo_drive_attachments.stl"/>
         <xacro:property name="attachment_origin_xyz" value="-0.0100 -0.0006 -0.0641"/>
-        <xacro:property name="attachment_orientation_rpy" value="0 0 1.5708"/>
-        <xacro:property name="wheel_prefix_left" value="${struct_prefix}left_"/>
-        <xacro:property name="wheel_prefix_right" value="${struct_prefix}right_"/>
-        <xacro:property name="wheel_orientation_rpy_right" value="-1.5708 0 0"/>
-        <xacro:property name="wheel_origin_xyz_right" value="0.0008 -0.0403 -0.0366"/>
-        <xacro:property name="wheel_orientation_rpy_left" value="1.5708 0 0"/>
-        <xacro:property name="wheel_origin_xyz_left" value="0.0008 0.0407 -0.0366"/>
+        <xacro:property name="wheel_prefix_left" value="left_wheel_"/>
+        <xacro:property name="wheel_prefix_right" value="right_wheel_"/>
+        <xacro:property name="wheel_orientation_rpy_left" value="-1.5708 0 0"/>
+        <xacro:property name="wheel_origin_xyz_left" value="0.0008 -0.0403 -0.0366"/>
+        <xacro:property name="wheel_orientation_rpy_right" value="1.5708 0 0"/>
+        <xacro:property name="wheel_origin_xyz_right" value="0.0008 0.0407 -0.0366"/>
+        <!-- Instantiate wheels -->
+        <xacro:kelo_hub_wheel wheel_prefix="${wheel_prefix_right}" struct_prefix="${robot_prefix}${struct_prefix}" wheel_origin_xyz="${wheel_origin_xyz_right}" wheel_orientation_rpy="${wheel_orientation_rpy_right}"/>
+        <xacro:kelo_hub_wheel wheel_prefix="${wheel_prefix_left}" struct_prefix="${robot_prefix}${struct_prefix}" wheel_origin_xyz="${wheel_origin_xyz_left}" wheel_orientation_rpy="${wheel_orientation_rpy_left}"/>
         <!-- Links -->
-        <link name="${struct_prefix}struct_attachment_link">
+        <link name="${robot_prefix}${struct_prefix}attachment_link">
             <visual>
                 <origin rpy="0 0 0" xyz="0 0 0"/>
@@ -37,5 +39,5 @@
             </inertial>
         </link>
-        <link name="${struct_prefix}struct_link">
+        <link name="${robot_prefix}${struct_prefix}struct_link">
             <visual>
                 <origin rpy="0 0 0" xyz="0 0 0"/>
@@ -53,28 +55,19 @@
             </collision>
             <inertial>
-                <mass value="1.0"/>
-                <inertia ixx="0" ixy="0" ixz="0" iyy="0" iyz="0" izz="0"/>
+                <mass value="1.892"/>
+                <origin xyz="0 0 0.006" rpy="0 0 0"/>
+                <inertia ixx="0.004574163" ixy="0" ixz="0" iyy="0.004344228" iyz="0" izz="0.004640438"/>
             </inertial>
         </link>
-        <!-- Instantiate wheels -->
-        <xacro:kelo_hub_wheel wheel_prefix="${wheel_prefix_right}"/>
-        <xacro:kelo_hub_wheel wheel_prefix="${wheel_prefix_left}"/>
         <!-- Joints -->
-        <joint name="${struct_prefix}struct_to_attachment_joint" type="continuous">
-            <parent link="${struct_prefix}struct_attachment_link"/>
-            <child link="${struct_prefix}struct_link"/>
-            <origin xyz="${attachment_origin_xyz}" rpy="${attachment_orientation_rpy}"/>
-            <axis xyz="0 0 1"/>
+        <joint name="${robot_prefix}${struct_prefix}attachment_joint" type="fixed">
+            <parent link="${robot_prefix}base_link"/>
+            <child link="${robot_prefix}${struct_prefix}attachment_link"/>
+            <origin xyz="${struct_origin_xyz}" rpy="${struct_orientation_rpy}"/>
         </joint>
-        <joint name="${struct_prefix}${wheel_prefix_left}wheel_joint" type="continuous">
-            <parent link="${struct_prefix}struct_link"/>
-            <child link="${wheel_prefix_left}wheel_link"/>
-            <origin xyz="${wheel_origin_xyz_left}" rpy="${wheel_orientation_rpy_left}"/>
-            <axis xyz="0 0 1"/>
-        </joint>
-        <joint name="${struct_prefix}${wheel_prefix_right}wheel_joint" type="continuous">
-            <parent link="${struct_prefix}struct_link"/>
-            <child link="${wheel_prefix_right}wheel_link"/>
-            <origin xyz="${wheel_origin_xyz_right}" rpy="${wheel_orientation_rpy_right}"/>
+        <joint name="${robot_prefix}${struct_prefix}struct_joint" type="continuous">
+            <parent link="${robot_prefix}${struct_prefix}attachment_link"/>
+            <child link="${robot_prefix}${struct_prefix}struct_link"/>
+            <origin xyz="${attachment_origin_xyz}" rpy="${attachment_cts_jnt_orientation_rpy}"/>
             <axis xyz="0 0 1"/>
         </joint>

File: urdf/kelo_hub_wheel.macro.xacro (robot description, xacro)
@@ -1,11 +1,10 @@
 <?xml version="1.0"?>
 <robot xmlns:xacro="http://www.ros.org/wiki/xacro" name="kelo_hub_wheel">
-    <xacro:arg name="wheel_prefix" default=""/>
-    <xacro:macro name="kelo_hub_wheel" params="wheel_prefix">
+    <xacro:macro name="kelo_hub_wheel" params="wheel_prefix struct_prefix wheel_origin_xyz wheel_orientation_rpy">
         <!-- Properties -->
         <xacro:property name="mesh_package" value="eddie_description"/>
-        <xacro:property name="wheel_mesh_file" value="hub_wheel.stl"/>
+        <xacro:property name="wheel_mesh_file" value="hub_wheel12.stl"/>
         <!-- Links -->
-        <link name="${wheel_prefix}wheel_link">
+        <link name="${struct_prefix}${wheel_prefix}link">
             <visual>
                 <origin rpy="0 0 0" xyz="0 0 0"/>
@@ -23,8 +22,15 @@
             </collision>
             <inertial>
-                <mass value="1.0"/>
-                <inertia ixx="0" ixy="0" ixz="0" iyy="0" iyz="0" izz="0"/>
+                <mass value="1.563"/>
+                <inertia ixx="0.0010" ixy="0" ixz="0" iyy="0.0010" iyz="0" izz="0.0005"/>
             </inertial>
         </link>
+        <!-- Joints -->
+        <joint name="${struct_prefix}${wheel_prefix}joint" type="continuous">
+            <parent link="${struct_prefix}struct_link"/>
+            <child link="${struct_prefix}${wheel_prefix}link"/>
+            <origin xyz="${wheel_origin_xyz}" rpy="${wheel_orientation_rpy}"/>
+            <axis xyz="0 0 1"/>
+        </joint>
     </xacro:macro>
 </robot>
