Commit message: update inertias, refactor

File: urdf/eddie_base.macro.xacro (robot description, xacro)
@@ -16,17 +16,17 @@
         <xacro:property name="rear_right_orientation_rpy" value="0 0 -1.5708"/>
         <xacro:property name="front_right_orientation_rpy" value="0 0 -1.5708"/>
-        <xacro:property name="front_right_attachment_cts_jnt_orientation_rpy" value="0 0 -1.5708"/>
-        <xacro:property name="front_left_attachment_cts_jnt_orientation_rpy" value="0 0 1.5708"/>
-        <xacro:property name="rear_right_attachment_cts_jnt_orientation_rpy" value="0 0 -1.5708"/>
-        <xacro:property name="rear_left_attachment_cts_jnt_orientation_rpy" value="0 0 1.5708"/>
-        <xacro:property name="torso_origin_xyz" value="-0.1738 0.0003 0.4184"/>
-        <xacro:property name="torso_orientation_rpy" value="0 0 1.5708"/>
+        <xacro:property name="front_right_struct_wrt_attachment_orientation_rpy" value="0 0 -1.5708"/>
+        <xacro:property name="front_left_struct_wrt_attachment_orientation_rpy" value="0 0 1.5708"/>
+        <xacro:property name="rear_right_struct_wrt_attachment_orientation_rpy" value="0 0 -1.5708"/>
+        <xacro:property name="rear_left_struct_wrt_attachment_orientation_rpy" value="0 0 1.5708"/>
+        <xacro:property name="torso_origin_wrt_base_link_xyz" value="-0.1738 0.0003 0.4184"/>
+        <xacro:property name="torso_orientation_wrt_base_link_rpy" value="0 0 1.5708"/>
         <xacro:property name="base_link_origin_xyz" value="0 0 0.2164"/>
         <xacro:property name="base_link_orientation_rpy" value="0 0 0"/>
         <!-- Instantiate wheel units -->
-        <xacro:kelo_drive_unit robot_prefix="${robot_prefix}" struct_prefix="front_left_drive_" struct_origin_xyz="${front_left_origin_xyz}" struct_orientation_rpy="${front_left_orientation_rpy}" attachment_cts_jnt_orientation_rpy="${front_left_attachment_cts_jnt_orientation_rpy}"/>
-        <xacro:kelo_drive_unit robot_prefix="${robot_prefix}" struct_prefix="rear_left_drive_" struct_origin_xyz="${rear_left_origin_xyz}" struct_orientation_rpy="${rear_left_orientation_rpy}"  attachment_cts_jnt_orientation_rpy="${rear_left_attachment_cts_jnt_orientation_rpy}"/>
-        <xacro:kelo_drive_unit robot_prefix="${robot_prefix}" struct_prefix="rear_right_drive_" struct_origin_xyz="${rear_right_origin_xyz}" struct_orientation_rpy="${rear_right_orientation_rpy}"  attachment_cts_jnt_orientation_rpy="${front_right_attachment_cts_jnt_orientation_rpy}"/>
-        <xacro:kelo_drive_unit robot_prefix="${robot_prefix}" struct_prefix="front_right_drive_" struct_origin_xyz="${front_right_origin_xyz}" struct_orientation_rpy="${front_right_orientation_rpy}"  attachment_cts_jnt_orientation_rpy="${rear_right_attachment_cts_jnt_orientation_rpy}"/>
+        <xacro:kelo_drive_unit robot_prefix="${robot_prefix}" struct_prefix="front_left_drive_" struct_origin_xyz="${front_left_origin_xyz}" struct_orientation_rpy="${front_left_orientation_rpy}" struct_wrt_attachment_orientation_rpy="${front_left_struct_wrt_attachment_orientation_rpy}"/>
+        <xacro:kelo_drive_unit robot_prefix="${robot_prefix}" struct_prefix="rear_left_drive_" struct_origin_xyz="${rear_left_origin_xyz}" struct_orientation_rpy="${rear_left_orientation_rpy}"  struct_wrt_attachment_orientation_rpy="${rear_left_struct_wrt_attachment_orientation_rpy}"/>
+        <xacro:kelo_drive_unit robot_prefix="${robot_prefix}" struct_prefix="rear_right_drive_" struct_origin_xyz="${rear_right_origin_xyz}" struct_orientation_rpy="${rear_right_orientation_rpy}"  struct_wrt_attachment_orientation_rpy="${front_right_struct_wrt_attachment_orientation_rpy}"/>
+        <xacro:kelo_drive_unit robot_prefix="${robot_prefix}" struct_prefix="front_right_drive_" struct_origin_xyz="${front_right_origin_xyz}" struct_orientation_rpy="${front_right_orientation_rpy}"  struct_wrt_attachment_orientation_rpy="${rear_right_struct_wrt_attachment_orientation_rpy}"/>
         <!-- Links -->
         <link name="${robot_prefix}base_footprint"/>
@@ -50,5 +50,5 @@
             </collision>
             <visual>
-                <origin rpy="${torso_orientation_rpy}" xyz="${torso_origin_xyz}"/>
+                <origin rpy="${torso_orientation_wrt_base_link_rpy}" xyz="${torso_origin_wrt_base_link_xyz}"/>
                 <geometry>
                     <mesh filename="package://${mesh_package}/meshes/${eddie_torso_file}" />
@@ -62,10 +62,10 @@
                     <mesh filename="package://${mesh_package}/meshes/${eddie_torso_file}"/>
                 </geometry>
-                <origin rpy="${torso_orientation_rpy}" xyz="${torso_origin_xyz}"/>
+                <origin rpy="${torso_orientation_wrt_base_link_rpy}" xyz="${torso_origin_wrt_base_link_xyz}"/>
             </collision>
             <inertial>
                 <mass value="76.4377"/>
-                <origin xyz="-0.05172 0.0045 0.2378" rpy="0 0 0"/>
-                <inertia ixx="4.128795216" ixy="0" ixz="0" iyy="4.117596854" iyz="0" izz="3.364397364"/>
+                <origin xyz="-0.05172 -0.0045 0.2378" rpy="0 0 0"/>
+                <inertia ixx="4.128795216" ixy="0.126348211" ixz="0.746707686" iyy="4.117596854" iyz="0.038071359" izz="3.364397364"/>
             </inertial>
         </link>
@@ -79,5 +79,5 @@
             <parent link="${robot_prefix}base_link"/>
             <child link="${robot_prefix}torso_link"/>
-            <origin xyz="${torso_origin_xyz}" rpy="${torso_orientation_rpy}"/>
+            <origin xyz="${torso_origin_wrt_base_link_xyz}" rpy="${torso_orientation_wrt_base_link_rpy}"/>
         </joint>
         <joint name="${robot_prefix}left_arm_attachment_joint" type="fixed">

File: urdf/kelo_drive_unit.macro.xacro (robot description, xacro)
@@ -3,15 +3,15 @@
     <!-- Include macro files -->
     <xacro:include filename="$(find eddie_description)/urdf/kelo_hub_wheel.macro.xacro"/>
-    <xacro:macro name="kelo_drive_unit" params="robot_prefix struct_prefix struct_origin_xyz struct_orientation_rpy attachment_cts_jnt_orientation_rpy">
+    <xacro:macro name="kelo_drive_unit" params="robot_prefix struct_prefix struct_origin_xyz struct_orientation_rpy struct_wrt_attachment_orientation_rpy">
         <!-- Properties -->
         <xacro:property name="mesh_package" value="eddie_description"/>
         <xacro:property name="struct_mesh_file" value="kelo_drive.stl"/>
         <xacro:property name="struct_attachment_mesh_file" value="kelo_drive_attachments.stl"/>
-        <xacro:property name="attachment_origin_xyz" value="-0.0100 -0.0006 -0.0641"/>
+        <xacro:property name="struct_wrt_attachment_origin_xyz" value="-0.0100 -0.0006 -0.0641"/>
         <xacro:property name="wheel_prefix_left" value="left_wheel_"/>
         <xacro:property name="wheel_prefix_right" value="right_wheel_"/>
-        <xacro:property name="wheel_orientation_rpy_left" value="-1.5708 0 0"/>
+        <xacro:property name="wheel_orientation_rpy_left" value="1.5708 3.1416 0"/>
         <xacro:property name="wheel_origin_xyz_left" value="0.0008 -0.0403 -0.0366"/>
-        <xacro:property name="wheel_orientation_rpy_right" value="1.5708 0 0"/>
+        <xacro:property name="wheel_orientation_rpy_right" value="-1.5708 0 0"/>
         <xacro:property name="wheel_origin_xyz_right" value="0.0008 0.0407 -0.0366"/>
         <!-- Instantiate wheels -->
@@ -35,6 +35,6 @@
             </collision>
             <inertial>
-                <mass value="1.0"/>
-                <inertia ixx="0" ixy="0" ixz="0" iyy="0" iyz="0" izz="0"/>
+                <mass value="0.5"/>
+                <inertia ixx="0.00042" ixy="0" ixz="0" iyy="0.00042" iyz="0" izz="0.0008"/>
             </inertial>
         </link>
@@ -55,5 +55,5 @@
             </collision>
             <inertial>
-                <mass value="1.892"/>
+                <mass value="1.392"/>
                 <origin xyz="0 0 0.006" rpy="0 0 0"/>
                 <inertia ixx="0.004574163" ixy="0" ixz="0" iyy="0.004344228" iyz="0" izz="0.004640438"/>
@@ -69,5 +69,5 @@
             <parent link="${robot_prefix}${struct_prefix}attachment_link"/>
             <child link="${robot_prefix}${struct_prefix}struct_link"/>
-            <origin xyz="${attachment_origin_xyz}" rpy="${attachment_cts_jnt_orientation_rpy}"/>
+            <origin xyz="${struct_wrt_attachment_origin_xyz}" rpy="${struct_wrt_attachment_orientation_rpy}"/>
             <axis xyz="0 0 1"/>
         </joint>

File: urdf/kelo_hub_wheel.macro.xacro (robot description, xacro)
@@ -4,5 +4,5 @@
         <!-- Properties -->
         <xacro:property name="mesh_package" value="eddie_description"/>
-        <xacro:property name="wheel_mesh_file" value="hub_wheel12.stl"/>
+        <xacro:property name="wheel_mesh_file" value="hub_wheel.stl"/>
         <!-- Links -->
         <link name="${struct_prefix}${wheel_prefix}link">
@@ -23,5 +23,6 @@
             <inertial>
                 <mass value="1.563"/>
-                <inertia ixx="0.0010" ixy="0" ixz="0" iyy="0.0010" iyz="0" izz="0.0005"/>
+                <origin rpy="0 0 0" xyz="0 0.00003 -0.00044" />
+                <inertia ixx="0.001012837" ixy="0" ixz="0" iyy="0.001013130" iyz="0" izz="0.001579986"/>
             </inertial>
         </link>

Commit message: add control tags

File: urdf/eddie_base.macro.xacro (robot description, xacro)
@@ -3,5 +3,5 @@
     <!-- Include macro files -->
     <xacro:include filename="$(find eddie_description)/urdf/kelo_drive_unit.macro.xacro"/>
-    <xacro:macro name="eddie_base" params="robot_prefix">
+    <xacro:macro name="eddie_base" params="robot_prefix joint_state_gui">
         <!-- Properties -->
         <xacro:property name="mesh_package" value="eddie_description"/>
@@ -25,8 +25,29 @@
         <xacro:property name="base_link_orientation_rpy" value="0 0 0"/>
         <!-- Instantiate wheel units -->
-        <xacro:kelo_drive_unit robot_prefix="${robot_prefix}" struct_prefix="front_left_drive_" struct_origin_xyz="${front_left_origin_xyz}" struct_orientation_rpy="${front_left_orientation_rpy}" struct_wrt_attachment_orientation_rpy="${front_left_struct_wrt_attachment_orientation_rpy}"/>
-        <xacro:kelo_drive_unit robot_prefix="${robot_prefix}" struct_prefix="rear_left_drive_" struct_origin_xyz="${rear_left_origin_xyz}" struct_orientation_rpy="${rear_left_orientation_rpy}"  struct_wrt_attachment_orientation_rpy="${rear_left_struct_wrt_attachment_orientation_rpy}"/>
-        <xacro:kelo_drive_unit robot_prefix="${robot_prefix}" struct_prefix="rear_right_drive_" struct_origin_xyz="${rear_right_origin_xyz}" struct_orientation_rpy="${rear_right_orientation_rpy}"  struct_wrt_attachment_orientation_rpy="${front_right_struct_wrt_attachment_orientation_rpy}"/>
-        <xacro:kelo_drive_unit robot_prefix="${robot_prefix}" struct_prefix="front_right_drive_" struct_origin_xyz="${front_right_origin_xyz}" struct_orientation_rpy="${front_right_orientation_rpy}"  struct_wrt_attachment_orientation_rpy="${rear_right_struct_wrt_attachment_orientation_rpy}"/>
+        <xacro:kelo_drive_unit
+        robot_prefix="${robot_prefix}"
+        joint_state_gui="${joint_state_gui}"
+        struct_prefix="front_left_drive_"
+        struct_origin_xyz="${front_left_origin_xyz}"
+        struct_orientation_rpy="${front_left_orientation_rpy}"
+        struct_wrt_attachment_orientation_rpy="${front_left_struct_wrt_attachment_orientation_rpy}"/>
+        <xacro:kelo_drive_unit robot_prefix="${robot_prefix}"
+        joint_state_gui="${joint_state_gui}"
+        struct_prefix="rear_left_drive_"
+        struct_origin_xyz="${rear_left_origin_xyz}"
+        struct_orientation_rpy="${rear_left_orientation_rpy}"
+        struct_wrt_attachment_orientation_rpy="${rear_left_struct_wrt_attachment_orientation_rpy}"/>
+        <xacro:kelo_drive_unit robot_prefix="${robot_prefix}"
+        joint_state_gui="${joint_state_gui}"
+        struct_prefix="rear_right_drive_"
+        struct_origin_xyz="${rear_right_origin_xyz}"
+        struct_orientation_rpy="${rear_right_orientation_rpy}"
+        struct_wrt_attachment_orientation_rpy="${front_right_struct_wrt_attachment_orientation_rpy}"/>
+        <xacro:kelo_drive_unit robot_prefix="${robot_prefix}"
+        joint_state_gui="${joint_state_gui}"
+        struct_prefix="front_right_drive_"
+        struct_origin_xyz="${front_right_origin_xyz}"
+        struct_orientation_rpy="${front_right_orientation_rpy}"
+        struct_wrt_attachment_orientation_rpy="${rear_right_struct_wrt_attachment_orientation_rpy}"/>
         <!-- Links -->
         <link name="${robot_prefix}base_footprint"/>

File: urdf/eddie_robot.urdf.xacro (robot description, xacro)
@@ -2,4 +2,5 @@
 <robot xmlns:xacro="http://www.ros.org/wiki/xacro" name="eddie_base_with_wheels">
     <xacro:arg name="robot_name" default="eddie_" />
+    <xacro:arg name="joint_state_gui" default="true" />
     <xacro:arg name="robot_ip_left" default="192.168.1.10" />
     <xacro:arg name="robot_ip_right" default="192.168.1.11" />
@@ -31,5 +32,5 @@
     <!-- Include Gen3 Arm -->
     <xacro:include filename="$(find eddie_description)/urdf/kinova_gen3.macro.xacro"/>
-    <xacro:eddie_base robot_prefix="$(arg robot_name)" />
+    <xacro:eddie_base robot_prefix="$(arg robot_name)" joint_state_gui="$(arg joint_state_gui)"/>
     <xacro:kinova_gen3
         parent="$(arg robot_name)left_arm_attachment_link"

File: urdf/kelo_drive_unit.macro.xacro (robot description, xacro)
@@ -3,5 +3,5 @@
     <!-- Include macro files -->
     <xacro:include filename="$(find eddie_description)/urdf/kelo_hub_wheel.macro.xacro"/>
-    <xacro:macro name="kelo_drive_unit" params="robot_prefix struct_prefix struct_origin_xyz struct_orientation_rpy struct_wrt_attachment_orientation_rpy">
+    <xacro:macro name="kelo_drive_unit" params="robot_prefix joint_state_gui struct_prefix struct_origin_xyz struct_orientation_rpy struct_wrt_attachment_orientation_rpy">
         <!-- Properties -->
         <xacro:property name="mesh_package" value="eddie_description"/>
@@ -16,6 +16,14 @@
         <xacro:property name="wheel_origin_xyz_right" value="0.0008 0.0407 -0.0366"/>
         <!-- Instantiate wheels -->
-        <xacro:kelo_hub_wheel wheel_prefix="${wheel_prefix_right}" struct_prefix="${robot_prefix}${struct_prefix}" wheel_origin_xyz="${wheel_origin_xyz_right}" wheel_orientation_rpy="${wheel_orientation_rpy_right}"/>
-        <xacro:kelo_hub_wheel wheel_prefix="${wheel_prefix_left}" struct_prefix="${robot_prefix}${struct_prefix}" wheel_origin_xyz="${wheel_origin_xyz_left}" wheel_orientation_rpy="${wheel_orientation_rpy_left}"/>
+        <xacro:kelo_hub_wheel wheel_prefix="${wheel_prefix_right}"
+        joint_state_gui="${joint_state_gui}"
+        struct_prefix="${robot_prefix}${struct_prefix}"
+        wheel_origin_xyz="${wheel_origin_xyz_right}"
+        wheel_orientation_rpy="${wheel_orientation_rpy_right}"/>
+        <xacro:kelo_hub_wheel wheel_prefix="${wheel_prefix_left}"
+        joint_state_gui="${joint_state_gui}"
+        struct_prefix="${robot_prefix}${struct_prefix}"
+        wheel_origin_xyz="${wheel_origin_xyz_left}"
+        wheel_orientation_rpy="${wheel_orientation_rpy_left}"/>
         <!-- Links -->
         <link name="${robot_prefix}${struct_prefix}attachment_link">
@@ -72,4 +80,35 @@
             <axis xyz="0 0 1"/>
         </joint>
+        <!-- ros2 control tags -->
+        <xacro:if value="${joint_state_gui}">
+            <ros2_control name="${robot_prefix}${struct_prefix}ctr" type="system">
+                <hardware>
+                    <plugin>gz_ros2_control/GazeboSimSystem</plugin>
+                </hardware>
+                <joint name="${robot_prefix}${struct_prefix}struct_joint">
+                    <command_interface name="position">
+                    <param name="min">-1e+100</param>
+                    <param name="max">1e+100</param>
+                    </command_interface>
+                    <command_interface name="velocity">
+                    <param name="min">-1e+100</param>
+                    <param name="max">1e+100</param>
+                    </command_interface>
+                    <command_interface name="effort">
+                    <param name="min">-1e+100</param>
+                    <param name="max">1e+100</param>
+                    </command_interface>
+                    <state_interface name="position">
+                    <param name="initial_value">0.0</param>
+                    </state_interface>
+                    <state_interface name="velocity"/>
+                    <state_interface name="effort"/>
+                </joint>
+                <transmission name="${robot_prefix}${struct_prefix}struct_joint_transmission">
+                    <plugin>transmission_interface/SimpleTansmission</plugin>
+                    <param name="joint_to_actuator">1</param>
+                </transmission>
+            </ros2_control>
+        </xacro:if>
     </xacro:macro>
 </robot>

File: urdf/kelo_hub_wheel.macro.xacro (robot description, xacro)
@@ -1,5 +1,5 @@
 <?xml version="1.0"?>
 <robot xmlns:xacro="http://www.ros.org/wiki/xacro" name="kelo_hub_wheel">
-    <xacro:macro name="kelo_hub_wheel" params="wheel_prefix struct_prefix wheel_origin_xyz wheel_orientation_rpy">
+    <xacro:macro name="kelo_hub_wheel" params="wheel_prefix struct_prefix wheel_origin_xyz wheel_orientation_rpy joint_state_gui">
         <!-- Properties -->
         <xacro:property name="mesh_package" value="eddie_description"/>
@@ -34,4 +34,35 @@
             <axis xyz="0 0 1"/>
         </joint>
+        <!-- ros2 control tags -->
+        <xacro:if value="${joint_state_gui}">
+            <ros2_control name="${struct_prefix}${wheel_prefix}ctr" type="system">
+                <hardware>
+                    <plugin>gz_ros2_control/GazeboSimSystem</plugin>
+                </hardware>
+                <joint name="${struct_prefix}${wheel_prefix}joint">
+                    <command_interface name="position">
+                    <param name="min">-1e+100</param>
+                    <param name="max">1e+100</param>
+                    </command_interface>
+                    <command_interface name="velocity">
+                    <param name="min">-1e+100</param>
+                    <param name="max">1e+100</param>
+                    </command_interface>
+                    <command_interface name="effort">
+                    <param name="min">-1e+100</param>
+                    <param name="max">1e+100</param>
+                    </command_interface>
+                    <state_interface name="position">
+                    <param name="initial_value">0.0</param>
+                    </state_interface>
+                    <state_interface name="velocity"/>
+                    <state_interface name="effort"/>
+                </joint>
+                <transmission name="${struct_prefix}${wheel_prefix}joint_transmission">
+                    <plugin>transmission_interface/SimpleTansmission</plugin>
+                    <param name="joint_to_actuator">1</param>
+                </transmission>
+            </ros2_control>
+        </xacro:if>
     </xacro:macro>
 </robot>
