Commit message: add state intf to wheel, rename jnt_state_gui

File: urdf/eddie_base.macro.xacro (robot description, xacro)
@@ -3,5 +3,5 @@
     <!-- Include macro files -->
     <xacro:include filename="$(find eddie_description)/urdf/kelo_drive_unit.macro.xacro"/>
-    <xacro:macro name="eddie_base" params="robot_prefix joint_state_gui">
+    <xacro:macro name="eddie_base" params="robot_prefix use_ros2_control">
         <!-- Properties -->
         <xacro:property name="mesh_package" value="eddie_description"/>
@@ -27,5 +27,5 @@
         <xacro:kelo_drive_unit
         robot_prefix="${robot_prefix}"
-        joint_state_gui="${joint_state_gui}"
+        use_ros2_control="${use_ros2_control}"
         struct_prefix="front_left_drive_"
         struct_origin_xyz="${front_left_origin_xyz}"
@@ -33,5 +33,5 @@
         struct_wrt_attachment_orientation_rpy="${front_left_struct_wrt_attachment_orientation_rpy}"/>
         <xacro:kelo_drive_unit robot_prefix="${robot_prefix}"
-        joint_state_gui="${joint_state_gui}"
+        use_ros2_control="${use_ros2_control}"
         struct_prefix="rear_left_drive_"
         struct_origin_xyz="${rear_left_origin_xyz}"
@@ -39,5 +39,5 @@
         struct_wrt_attachment_orientation_rpy="${rear_left_struct_wrt_attachment_orientation_rpy}"/>
         <xacro:kelo_drive_unit robot_prefix="${robot_prefix}"
-        joint_state_gui="${joint_state_gui}"
+        use_ros2_control="${use_ros2_control}"
         struct_prefix="rear_right_drive_"
         struct_origin_xyz="${rear_right_origin_xyz}"
@@ -45,5 +45,5 @@
         struct_wrt_attachment_orientation_rpy="${front_right_struct_wrt_attachment_orientation_rpy}"/>
         <xacro:kelo_drive_unit robot_prefix="${robot_prefix}"
-        joint_state_gui="${joint_state_gui}"
+        use_ros2_control="${use_ros2_control}"
         struct_prefix="front_right_drive_"
         struct_origin_xyz="${front_right_origin_xyz}"

File: urdf/eddie_robot.urdf.xacro (robot description, xacro)
@@ -2,5 +2,5 @@
 <robot xmlns:xacro="http://www.ros.org/wiki/xacro" name="eddie_base_with_wheels">
     <xacro:arg name="robot_name" default="eddie_" />
-    <xacro:arg name="joint_state_gui" default="true" />
+    <xacro:arg name="use_ros2_control" default="true" />
     <xacro:arg name="robot_ip_left" default="192.168.1.10" />
     <xacro:arg name="robot_ip_right" default="192.168.1.11" />
@@ -34,5 +34,5 @@
     <xacro:include filename="$(find eddie_description)/urdf/kinova_gen3.macro.xacro"/>
     <xacro:include filename="$(find eddie_description)/urdf/kortex.ros2_gz_control.macro.xacro" />
-    <xacro:eddie_base robot_prefix="$(arg robot_name)" joint_state_gui="$(arg joint_state_gui)"/>
+    <xacro:eddie_base robot_prefix="$(arg robot_name)" use_ros2_control="$(arg use_ros2_control)"/>
     <xacro:kinova_gen3
         parent="$(arg robot_name)left_arm_attachment_link"

File: urdf/kelo_drive_unit.macro.xacro (robot description, xacro)
@@ -3,5 +3,5 @@
     <!-- Include macro files -->
     <xacro:include filename="$(find eddie_description)/urdf/kelo_hub_wheel.macro.xacro"/>
-    <xacro:macro name="kelo_drive_unit" params="robot_prefix joint_state_gui struct_prefix struct_origin_xyz struct_orientation_rpy struct_wrt_attachment_orientation_rpy">
+    <xacro:macro name="kelo_drive_unit" params="robot_prefix use_ros2_control struct_prefix struct_origin_xyz struct_orientation_rpy struct_wrt_attachment_orientation_rpy">
         <!-- Properties -->
         <xacro:property name="mesh_package" value="eddie_description"/>
@@ -17,10 +17,10 @@
         <!-- Instantiate wheels -->
         <xacro:kelo_hub_wheel wheel_prefix="${wheel_prefix_right}"
-        joint_state_gui="${joint_state_gui}"
+        use_ros2_control="${use_ros2_control}"
         struct_prefix="${robot_prefix}${struct_prefix}"
         wheel_origin_xyz="${wheel_origin_xyz_right}"
         wheel_orientation_rpy="${wheel_orientation_rpy_right}"/>
         <xacro:kelo_hub_wheel wheel_prefix="${wheel_prefix_left}"
-        joint_state_gui="${joint_state_gui}"
+        use_ros2_control="${use_ros2_control}"
         struct_prefix="${robot_prefix}${struct_prefix}"
         wheel_origin_xyz="${wheel_origin_xyz_left}"
@@ -80,4 +80,18 @@
             <axis xyz="0 0 1"/>
         </joint>
+        <!-- ros2 control tags -->
+        <xacro:if value="${use_ros2_control}">
+            <ros2_control name="${robot_prefix}${struct_prefix}ctr" type="system">
+                <hardware>
+                    <plugin>gz_ros2_control/GazeboSimSystem</plugin>
+                </hardware>
+                <joint name="${robot_prefix}${struct_prefix}struct_joint">
+                    <state_interface name="position">
+                    <param name="initial_value">0.0</param>
+                    </state_interface>
+                    <state_interface name="velocity"/>
+                </joint>
+            </ros2_control>
+        </xacro:if>
     </xacro:macro>
 </robot>

File: urdf/kelo_hub_wheel.macro.xacro (robot description, xacro)
@@ -2,5 +2,5 @@
 <robot xmlns:xacro="http://www.ros.org/wiki/xacro" name="kelo_hub_wheel">
     <xacro:macro name="kelo_hub_wheel"
-        params="wheel_prefix struct_prefix wheel_origin_xyz wheel_orientation_rpy joint_state_gui">
+        params="wheel_prefix struct_prefix wheel_origin_xyz wheel_orientation_rpy use_ros2_control">
         <!-- Properties -->
         <xacro:property name="mesh_package" value="eddie_description" />
@@ -37,5 +37,5 @@
         </joint>
         <!-- ros2 control tags -->
-        <xacro:if value="${joint_state_gui}">
+        <xacro:if value="${use_ros2_control}">
             <ros2_control name="${struct_prefix}${wheel_prefix}ctr" type="system">
                 <hardware>
@@ -61,8 +61,4 @@
                     <state_interface name="effort" />
                 </joint>
-                <!-- <transmission name="${struct_prefix}${wheel_prefix}joint_transmission">
-                    <plugin>transmission_interface/SimpleTansmission</plugin>
-                    <param name="joint_to_actuator">1</param>
-                </transmission> -->
             </ros2_control>
         </xacro:if>

Commit message: update base inertia

File: urdf/eddie_base.macro.xacro (robot description, xacro)
@@ -87,6 +87,6 @@
             <inertial>
                 <mass value="76.4377"/>
-                <origin xyz="-0.05172 -0.0045 0.2378" rpy="0 0 0"/>
-                <inertia ixx="4.128795216" ixy="0.126348211" ixz="0.746707686" iyy="4.117596854" iyz="0.038071359" izz="3.364397364"/>
+                <origin xyz="0 0 0.0833" rpy="0 0 0"/>
+                <inertia ixx="4.128795216" ixy="0" ixz="0" iyy="4.117596854" iyz="0" izz="3.364397364"/>
             </inertial>
         </link>
