Commit message: decluttered and removed redundandant params

File: urdf/eddie_base.macro.xacro (robot description, xacro)
@@ -2,114 +2,137 @@
 <robot xmlns:xacro="http://www.ros.org/wiki/xacro" name="eddie_base">
     <!-- Include macro files -->
-    <xacro:include filename="$(find eddie_description)/urdf/kelo_drive_unit.macro.xacro"/>
-    <xacro:macro name="eddie_base" params="robot_prefix use_ros2_control">
+    <xacro:include filename="$(find eddie_description)/urdf/kelo_drive_unit.macro.xacro" />
+    <xacro:macro name="eddie_base" params="robot_prefix use_ros2_control use_gz_sim">
         <!-- Properties -->
-        <xacro:property name="mesh_package" value="eddie_description"/>
-        <xacro:property name="eddie_base_file" value="kelo_base.stl"/>
-        <xacro:property name="eddie_torso_file" value="kelo_torso.stl"/>
-        <xacro:property name="front_left_origin_xyz" value="0.2078 0.1880 -0.0632"/>
-        <xacro:property name="rear_left_origin_xyz" value="-0.2078 0.1880 -0.0632"/>
-        <xacro:property name="rear_right_origin_xyz" value="-0.2078 -0.1880 -0.0632"/>
-        <xacro:property name="front_right_origin_xyz" value="0.2078 -0.1880 -0.0632"/>
-        <xacro:property name="front_left_orientation_rpy" value="0 0 1.5708"/>
-        <xacro:property name="rear_left_orientation_rpy" value="0 0 1.5708"/>
-        <xacro:property name="rear_right_orientation_rpy" value="0 0 -1.5708"/>
-        <xacro:property name="front_right_orientation_rpy" value="0 0 -1.5708"/>
-        <xacro:property name="front_right_struct_wrt_attachment_orientation_rpy" value="0 0 -1.5708"/>
-        <xacro:property name="front_left_struct_wrt_attachment_orientation_rpy" value="0 0 1.5708"/>
-        <xacro:property name="rear_right_struct_wrt_attachment_orientation_rpy" value="0 0 -1.5708"/>
-        <xacro:property name="rear_left_struct_wrt_attachment_orientation_rpy" value="0 0 1.5708"/>
-        <xacro:property name="torso_origin_wrt_base_link_xyz" value="-0.1738 0.0003 0.4184"/>
-        <xacro:property name="torso_orientation_wrt_base_link_rpy" value="0 0 1.5708"/>
-        <xacro:property name="base_link_origin_xyz" value="0 0 0.2164"/>
-        <xacro:property name="base_link_orientation_rpy" value="0 0 0"/>
-        <!-- Instantiate wheel units -->
-        <xacro:kelo_drive_unit
-        robot_prefix="${robot_prefix}"
-        use_ros2_control="${use_ros2_control}"
-        struct_prefix="front_left_drive_"
-        struct_origin_xyz="${front_left_origin_xyz}"
-        struct_orientation_rpy="${front_left_orientation_rpy}"
-        struct_wrt_attachment_orientation_rpy="${front_left_struct_wrt_attachment_orientation_rpy}"/>
-        <xacro:kelo_drive_unit robot_prefix="${robot_prefix}"
-        use_ros2_control="${use_ros2_control}"
-        struct_prefix="rear_left_drive_"
-        struct_origin_xyz="${rear_left_origin_xyz}"
-        struct_orientation_rpy="${rear_left_orientation_rpy}"
-        struct_wrt_attachment_orientation_rpy="${rear_left_struct_wrt_attachment_orientation_rpy}"/>
-        <xacro:kelo_drive_unit robot_prefix="${robot_prefix}"
-        use_ros2_control="${use_ros2_control}"
-        struct_prefix="rear_right_drive_"
-        struct_origin_xyz="${rear_right_origin_xyz}"
-        struct_orientation_rpy="${rear_right_orientation_rpy}"
-        struct_wrt_attachment_orientation_rpy="${front_right_struct_wrt_attachment_orientation_rpy}"/>
-        <xacro:kelo_drive_unit robot_prefix="${robot_prefix}"
-        use_ros2_control="${use_ros2_control}"
-        struct_prefix="front_right_drive_"
-        struct_origin_xyz="${front_right_origin_xyz}"
-        struct_orientation_rpy="${front_right_orientation_rpy}"
-        struct_wrt_attachment_orientation_rpy="${rear_right_struct_wrt_attachment_orientation_rpy}"/>
+        <xacro:property name="mesh_package" value="eddie_description" />
+        <xacro:property name="eddie_base_file" value="kelo_base.stl" />
+        <xacro:property name="eddie_torso_file" value="kelo_torso.stl" />
+        <!-- wheel unit attachments -->
+        <xacro:property name="front_left_attachment_origin">
+            <origin xyz="0.2078 0.1880 -0.0632" rpy="0 0 1.5708" />
+        </xacro:property>
+        <xacro:property name="rear_left_attachment_origin">
+            <origin xyz="-0.2078 0.1880 -0.0632" rpy="0 0 1.5708" />
+        </xacro:property>
+        <xacro:property name="rear_right_attachment_origin">
+            <origin xyz="-0.2078 -0.1880 -0.0632" rpy="0 0 -1.5708" />
+        </xacro:property>
+        <xacro:property name="front_right_attachment_origin">
+            <origin xyz="0.2078 -0.1880 -0.0632" rpy="0 0 -1.5708" />
+        </xacro:property>
+        <xacro:property name="front_right_struct_wrt_attachment_rpy" value="0 0 -1.5708" />
+        <xacro:property name="front_left_struct_wrt_attachment_rpy" value="0 0 1.5708" />
+        <xacro:property name="rear_right_struct_wrt_attachment_rpy" value="0 0 -1.5708" />
+        <xacro:property name="rear_left_struct_wrt_attachment_rpy" value="0 0 1.5708" />
+        <!-- base link origin -->
+        <xacro:property name="base_link_origin">
+            <origin xyz="0 0 0.2164" rpy="0 0 0" />
+        </xacro:property>
+        <!-- torso origin -->
+        <xacro:property name="torso_origin_wrt_base_link">
+            <origin xyz="-0.1738 0.0003 0.4184" rpy="0 0 1.5708" />
+        </xacro:property>
+        <!-- arm attachment origins -->
+        <xacro:property name="left_arm_attachment_origin">
+            <origin xyz="${-0.1738 + 0.0236} ${0.0003 + 0.0676} ${0.4184 + 0.1160}"
+                rpy="${0} ${0 + 0.09} ${1.5708 - 0.7783}" />
+        </xacro:property>
+        <xacro:property name="right_arm_attachment_origin">
+            <origin xyz="${-0.1738 + 0.0236} ${0.0003 - 0.0676} ${0.4184 + 0.1160}"
+                rpy="${0} ${0 + 0.09} ${1.5708 - 2.3632}" />
+        </xacro:property>
         <!-- Links -->
-        <link name="${robot_prefix}base_footprint"/>
+        <link name="${robot_prefix}base_footprint" />
         <link name="${robot_prefix}left_arm_attachment_link" />
         <link name="${robot_prefix}right_arm_attachment_link" />
-        <link name="${robot_prefix}torso_link" />
         <link name="${robot_prefix}base_link">
+            <!-- base -->
             <visual>
-                <origin rpy="0 0 0" xyz="0 0 0"/>
+                <origin rpy="0 0 0" xyz="0 0 0" />
                 <geometry>
-                    <mesh filename="package://${mesh_package}/meshes/${eddie_base_file}"/>
+                    <mesh filename="package://${mesh_package}/meshes/${eddie_base_file}" />
                 </geometry>
-                <material name="light_gray">
-                    <color rgba="0.5 0.5 0.5 1.0"/>
-                </material>
+                <material name="light_gray" />
             </visual>
             <collision>
                 <geometry>
-                    <mesh filename="package://${mesh_package}/meshes/${eddie_base_file}"/>
+                    <mesh filename="package://${mesh_package}/meshes/${eddie_base_file}" />
                 </geometry>
             </collision>
+            <!-- torso -->
             <visual>
-                <origin rpy="${torso_orientation_wrt_base_link_rpy}" xyz="${torso_origin_wrt_base_link_xyz}"/>
+                <xacro:insert_block name="torso_origin_wrt_base_link" />
                 <geometry>
                     <mesh filename="package://${mesh_package}/meshes/${eddie_torso_file}" />
                 </geometry>
-                <material name="metallic_silver">
-                    <color rgba="0.7 0.7 0.7 1.0"/>
-                </material>
+                <material name="metallic_silver" />
             </visual>
             <collision>
+                <xacro:insert_block name="torso_origin_wrt_base_link" />
                 <geometry>
-                    <mesh filename="package://${mesh_package}/meshes/${eddie_torso_file}"/>
+                    <mesh filename="package://${mesh_package}/meshes/${eddie_torso_file}" />
                 </geometry>
-                <origin rpy="${torso_orientation_wrt_base_link_rpy}" xyz="${torso_origin_wrt_base_link_xyz}"/>
             </collision>
+            <!-- base + torso -->
             <inertial>
-                <mass value="76.4377"/>
-                <origin xyz="0 0 0.0833" rpy="0 0 0"/>
-                <inertia ixx="4.128795216" ixy="0" ixz="0" iyy="4.117596854" iyz="0" izz="3.364397364"/>
+                <mass value="76.4377" />
+                <origin xyz="0 0 0.0833" rpy="0 0 0" />
+                <inertia ixx="4.128795216" ixy="0" ixz="0" iyy="4.117596854" iyz="0"
+                    izz="3.364397364" />
             </inertial>
         </link>
         <!-- Joints -->
-        <joint name="${robot_prefix}base_footprint_joint" type="fixed">
-            <parent link="${robot_prefix}base_footprint"/>
-            <child link="${robot_prefix}base_link"/>
-            <origin xyz="${base_link_origin_xyz}" rpy="${base_link_orientation_rpy}"/>
-        </joint>
-        <joint name="${robot_prefix}base_torso_joint" type="fixed">
-            <parent link="${robot_prefix}base_link"/>
-            <child link="${robot_prefix}torso_link"/>
-            <origin xyz="${torso_origin_wrt_base_link_xyz}" rpy="${torso_orientation_wrt_base_link_rpy}"/>
+        <joint name="${robot_prefix}base_link_joint" type="fixed">
+            <parent link="${robot_prefix}base_footprint" />
+            <child link="${robot_prefix}base_link" />
+            <xacro:insert_block name="base_link_origin" />
         </joint>
         <joint name="${robot_prefix}left_arm_attachment_joint" type="fixed">
-            <parent link="${robot_prefix}torso_link"/>
-            <child link="${robot_prefix}left_arm_attachment_link"/>
-            <origin xyz="0.0676 -0.0236 0.1160" rpy="0 0.09 -0.7783"/>
+            <parent link="${robot_prefix}base_link" />
+            <child link="${robot_prefix}left_arm_attachment_link" />
+            <xacro:insert_block name="left_arm_attachment_origin" />
         </joint>
         <joint name="${robot_prefix}right_arm_attachment_joint" type="fixed">
-            <parent link="${robot_prefix}torso_link"/>
-            <child link="${robot_prefix}right_arm_attachment_link"/>
-            <origin xyz="-0.0676 -0.0236 0.1160" rpy="0 0.09 -2.3632"/>
+            <parent link="${robot_prefix}base_link" />
+            <child link="${robot_prefix}right_arm_attachment_link" />
+            <xacro:insert_block name="right_arm_attachment_origin" />
         </joint>
+        <!-- Instantiate wheel units -->
+        <!-- front left -->
+        <xacro:kelo_drive_unit
+            parent="${robot_prefix}base_link"
+            use_ros2_control="${use_ros2_control}"
+            use_gz_sim="${use_gz_sim}"
+            struct_prefix="${robot_prefix}front_left_drive_"
+            struct_wrt_attachment_rpy="${front_left_struct_wrt_attachment_rpy}">
+            <xacro:insert_block name="front_left_attachment_origin" />
+        </xacro:kelo_drive_unit>
+        <!-- rear left -->
+        <xacro:kelo_drive_unit
+            parent="${robot_prefix}base_link"
+            use_ros2_control="${use_ros2_control}"
+            use_gz_sim="${use_gz_sim}"
+            struct_prefix="${robot_prefix}rear_left_drive_"
+            struct_wrt_attachment_rpy="${rear_left_struct_wrt_attachment_rpy}">
+            <xacro:insert_block name="rear_left_attachment_origin" />
+        </xacro:kelo_drive_unit>
+        <!-- rear right -->
+        <xacro:kelo_drive_unit
+            parent="${robot_prefix}base_link"
+            use_ros2_control="${use_ros2_control}"
+            use_gz_sim="${use_gz_sim}"
+            struct_prefix="${robot_prefix}rear_right_drive_"
+            struct_wrt_attachment_rpy="${front_right_struct_wrt_attachment_rpy}">
+            <xacro:insert_block name="rear_right_attachment_origin" />
+        </xacro:kelo_drive_unit>
+        <!-- front right -->
+        <xacro:kelo_drive_unit
+            parent="${robot_prefix}base_link"
+            use_ros2_control="${use_ros2_control}"
+            use_gz_sim="${use_gz_sim}"
+            struct_prefix="${robot_prefix}front_right_drive_"
+            struct_wrt_attachment_rpy="${rear_right_struct_wrt_attachment_rpy}">
+            <xacro:insert_block name="front_right_attachment_origin" />
+        </xacro:kelo_drive_unit>
     </xacro:macro>
 </robot>

File: urdf/eddie_robot.urdf.xacro (robot description, xacro)
@@ -2,5 +2,9 @@
 <robot xmlns:xacro="http://www.ros.org/wiki/xacro" name="eddie_base_with_wheels">
     <xacro:arg name="robot_name" default="eddie_" />
-    <xacro:arg name="use_ros2_control" default="true" />
+    <xacro:arg name="use_ros2_control" default="false" />
+    <xacro:arg name="use_gz_sim" default="false" />
+    <xacro:arg name="use_sim_isaac" default="false" />
+    <xacro:arg name="use_fake_hardware" default="false" />
+    <xacro:arg name="use_fake_sensor_commands" default="false" />
     <xacro:arg name="robot_ip_left" default="192.168.1.10" />
     <xacro:arg name="robot_ip_right" default="192.168.1.11" />
@@ -14,12 +18,8 @@
     <xacro:arg name="gripper" default="" />
     <xacro:arg name="gripper_joint_name" default="grasp_joint" />
-    <xacro:arg name="use_fake_hardware" default="false" />
-    <xacro:arg name="fake_sensor_commands" default="false" />
-    <xacro:arg name="sim_gz" default="true" />
-    <xacro:arg name="sim_isaac" default="false" />
     <xacro:arg name="use_internal_bus_gripper_comm" default="false" />
     <xacro:arg name="simulation_controllers"
         default="$(find eddie_gazebo)/config/eddie_controllers.yaml" />
-    <!-- initial position for simulations (Mock Hardware, Gazebo, Ignition) -->
+    <!-- initial position for simulations (Mock Hardware, Gazebo) -->
     <xacro:arg name="initial_positions_file_left"
         default="$(find eddie_description)/config/initial_positions_arm_left.yaml" />
@@ -31,8 +31,12 @@
         default="$(arg initial_positions_file_right)" />
     <!-- Include macro files -->
-    <xacro:include filename="$(find eddie_description)/urdf/eddie_base.macro.xacro"/>
-    <xacro:include filename="$(find eddie_description)/urdf/kinova_gen3.macro.xacro"/>
+    <xacro:include filename="$(find eddie_description)/urdf/materials.xacro" />
+    <xacro:include filename="$(find eddie_description)/urdf/eddie_base.macro.xacro" />
+    <xacro:include filename="$(find eddie_description)/urdf/kinova_gen3.macro.xacro" />
     <xacro:include filename="$(find eddie_description)/urdf/kortex.ros2_gz_control.macro.xacro" />
-    <xacro:eddie_base robot_prefix="$(arg robot_name)" use_ros2_control="$(arg use_ros2_control)"/>
+    <!-- Eddie base with KELO hub wheels -->
+    <xacro:eddie_base robot_prefix="$(arg robot_name)" use_ros2_control="$(arg use_ros2_control)"
+        use_gz_sim="$(arg use_gz_sim)" />
+    <!-- Left Kinova Gen3 7 DoF arm -->
     <xacro:kinova_gen3
         parent="$(arg robot_name)left_arm_attachment_link"
@@ -47,25 +51,28 @@
         connection_inactivity_timeout_ms="$(arg connection_inactivity_timeout_ms)"
         use_fake_hardware="$(arg use_fake_hardware)"
-        fake_sensor_commands="$(arg fake_sensor_commands)"
+        fake_sensor_commands="$(arg use_fake_sensor_commands)"
         initial_positions="${xacro.load_yaml(initial_positions_file_left)}">
         <origin xyz="0.01549 0 0" rpy="1.5708 -1.5708 1.5708" />
     </xacro:kinova_gen3>
-    <xacro:kortex_ros2_control
-        name="$(arg robot_name)left_arm_KortexMultiInterfaceHardware"
-        prefix="$(arg robot_name)left_arm_"
-        use_fake_hardware="$(arg use_fake_hardware)"
-        fake_sensor_commands="$(arg fake_sensor_commands)"
-        sim_gz="$(arg sim_gz)"
-        tf_prefix=""
-        initial_positions="${xacro.load_yaml(initial_positions_file_left)}"
-        robot_ip="$(arg robot_ip_left)"
-        username="$(arg username)"
-        password="$(arg password)"
-        port="$(arg port)"
-        port_realtime="$(arg port_realtime)"
-        session_inactivity_timeout_ms="$(arg session_inactivity_timeout_ms)"
-        connection_inactivity_timeout_ms="$(arg connection_inactivity_timeout_ms)"
-        use_internal_bus_gripper_comm="$(arg use_internal_bus_gripper_comm)"
-        gripper_joint_name="$(arg gripper_joint_name)"/>
+    <xacro:if value="$(arg use_ros2_control)">
+        <xacro:kortex_ros2_control
+            name="$(arg robot_name)left_arm_KortexMultiInterfaceHardware"
+            prefix="$(arg robot_name)left_arm_"
+            use_fake_hardware="$(arg use_fake_hardware)"
+            fake_sensor_commands="$(arg use_fake_sensor_commands)"
+            sim_gz="$(arg use_gz_sim)"
+            tf_prefix=""
+            initial_positions="${xacro.load_yaml(initial_positions_file_left)}"
+            robot_ip="$(arg robot_ip_left)"
+            username="$(arg username)"
+            password="$(arg password)"
+            port="$(arg port)"
+            port_realtime="$(arg port_realtime)"
+            session_inactivity_timeout_ms="$(arg session_inactivity_timeout_ms)"
+            connection_inactivity_timeout_ms="$(arg connection_inactivity_timeout_ms)"
+            use_internal_bus_gripper_comm="$(arg use_internal_bus_gripper_comm)"
+            gripper_joint_name="$(arg gripper_joint_name)" />
+    </xacro:if>
+    <!-- Right Kinova Gen3 7 DoF arm -->
     <xacro:kinova_gen3
         parent="$(arg robot_name)right_arm_attachment_link"
@@ -80,55 +87,63 @@
         connection_inactivity_timeout_ms="$(arg connection_inactivity_timeout_ms)"
         use_fake_hardware="$(arg use_fake_hardware)"
-        fake_sensor_commands="$(arg fake_sensor_commands)"
+        fake_sensor_commands="$(arg use_fake_sensor_commands)"
         initial_positions="${xacro.load_yaml(initial_positions_file_right)}">
         <origin xyz="0.01549 0 0" rpy="1.5708 -1.5708 1.5708" />
     </xacro:kinova_gen3>
-    <xacro:kortex_ros2_control
-        name="$(arg robot_name)right_arm_KortexMultiInterfaceHardware"
-        prefix="$(arg robot_name)right_arm_"
-        use_fake_hardware="$(arg use_fake_hardware)"
-        fake_sensor_commands="$(arg fake_sensor_commands)"
-        sim_gz="$(arg sim_gz)"
-        tf_prefix=""
-        initial_positions="${xacro.load_yaml(initial_positions_file_right)}"
-        robot_ip="$(arg robot_ip_right)"
-        username="$(arg username)"
-        password="$(arg password)"
-        port="$(arg port)"
-        port_realtime="$(arg port_realtime)"
-        session_inactivity_timeout_ms="$(arg session_inactivity_timeout_ms)"
-        connection_inactivity_timeout_ms="$(arg connection_inactivity_timeout_ms)"
-        use_internal_bus_gripper_comm="$(arg use_internal_bus_gripper_comm)"
-        gripper_joint_name="$(arg gripper_joint_name)"/>
-    <!-- gazebo tag for ros2 control -->
-    <gazebo>
-        <plugin filename="libgz_ros2_control-system.so"
-            name="gz_ros2_control::GazeboSimROS2ControlPlugin">
-            <robot_param>robot_description</robot_param>
-            <robot_param_node>robot_state_publisher</robot_param_node>
-            <parameters>$(arg simulation_controllers)</parameters>
-            <ros>
-                <remapping>~/odom:=odom</remapping>
-                <remapping>/tf:=tf</remapping>
-                <remapping>/tf_static:=tf_static</remapping>
-              </ros>
-        </plugin>
-        <self_collide>1</self_collide>
-    </gazebo>
-    <gazebo reference="base_link">
-        <gravity>true</gravity>
-        <self_collide>false</self_collide>
-    </gazebo>
-    <gazebo>
-        <plugin
-            filename="gz-sim-odometry-publisher-system"
-            name="gz::sim::systems::OdometryPublisher">
-            <odom_frame>odom</odom_frame>
-            <robot_base_frame>eddie_base_link</robot_base_frame>
-        </plugin>
-        <plugin
-            filename="gz-sim-velocity-control-system"
-            name="gz::sim::systems::VelocityControl">
-        </plugin>
-    </gazebo>
+    <xacro:if value="$(arg use_ros2_control)">
+        <xacro:kortex_ros2_control
+            name="$(arg robot_name)right_arm_KortexMultiInterfaceHardware"
+            prefix="$(arg robot_name)right_arm_"
+            use_fake_hardware="$(arg use_fake_hardware)"
+            fake_sensor_commands="$(arg use_fake_sensor_commands)"
+            sim_gz="$(arg use_gz_sim)"
+            tf_prefix=""
+            initial_positions="${xacro.load_yaml(initial_positions_file_right)}"
+            robot_ip="$(arg robot_ip_right)"
+            username="$(arg username)"
+            password="$(arg password)"
+            port="$(arg port)"
+            port_realtime="$(arg port_realtime)"
+            session_inactivity_timeout_ms="$(arg session_inactivity_timeout_ms)"
+            connection_inactivity_timeout_ms="$(arg connection_inactivity_timeout_ms)"
+            use_internal_bus_gripper_comm="$(arg use_internal_bus_gripper_comm)"
+            gripper_joint_name="$(arg gripper_joint_name)" />
+    </xacro:if>
+    <!-- gazebo and ros2 control -->
+    <xacro:if value="$(arg use_ros2_control)">
+        <xacro:if value="$(arg use_gz_sim)">
+            <gazebo>
+                <plugin filename="libgz_ros2_control-system.so"
+                    name="gz_ros2_control::GazeboSimROS2ControlPlugin">
+                    <robot_param>robot_description</robot_param>
+                    <robot_param_node>robot_state_publisher</robot_param_node>
+                    <parameters>$(arg simulation_controllers)</parameters>
+                    <!-- <ros>
+                        <remapping>~/odom:=odom</remapping>
+                        <remapping>/tf:=tf</remapping>
+                        <remapping>/tf_static:=tf_static</remapping>
+                    </ros> -->
+                </plugin>
+            </gazebo>
+        </xacro:if>
+    </xacro:if>
+    <xacro:if value="$(arg use_gz_sim)">
+        <gazebo>
+            <self_collide>1</self_collide>
+            <plugin
+                filename="gz-sim-odometry-publisher-system"
+                name="gz::sim::systems::OdometryPublisher">
+                <odom_frame>odom</odom_frame>
+                <robot_base_frame>$(arg robot_name)base_footprint</robot_base_frame>
+            </plugin>
+            <plugin
+                filename="gz-sim-velocity-control-system"
+                name="gz::sim::systems::VelocityControl">
+            </plugin>
+        </gazebo>
+        <gazebo reference="$(arg robot_name)base_link">
+            <gravity>true</gravity>
+            <self_collide>false</self_collide>
+        </gazebo>
+    </xacro:if>
 </robot>
