Commit message: added laser scanenr

File: urdf/eddie_base.macro.xacro (robot description, xacro)
@@ -3,5 +3,5 @@
     <!-- Include macro files -->
     <xacro:include filename="$(find eddie_description)/urdf/kelo_drive_unit.macro.xacro" />
-    <xacro:macro name="eddie_base" params="robot_prefix use_ros2_control use_gz_sim">
+    <xacro:macro name="eddie_base" params="robot_prefix use_ros2_control use_gz_sim use_kelo_tulip">
         <!-- Properties -->
         <xacro:property name="mesh_package" value="eddie_description" />
@@ -98,4 +98,37 @@
             <xacro:insert_block name="right_arm_attachment_origin" />
         </joint>
+        <!-- laser scanners -->
+        <link name="${robot_prefix}front_right_laser_attachment_link" />
+        <link name="${robot_prefix}rear_left_laser_attachment_link" />
+        <joint name="${robot_prefix}front_right_laser_attachment_joint" type="fixed">
+            <parent link="${robot_prefix}base_link" />
+            <child link="${robot_prefix}front_right_laser_attachment_link" />
+            <origin xyz="0.2193 -0.2391 0.0682" rpy="0 0 0" />
+        </joint>
+        <joint name="${robot_prefix}rear_left_laser_attachment_joint" type="fixed">
+            <parent link="${robot_prefix}base_link" />
+            <child link="${robot_prefix}rear_left_laser_attachment_link" />
+            <origin xyz="-0.2193 0.2386 0.0682" rpy="0 0 0" />
+        </joint>
+        <!-- instantiate laser scanners -->
+        <xacro:include filename="$(find eddie_description)/urdf/sensors/hokuyo.urdf.xacro" />
+        <!-- front right -->
+        <xacro:hokuyo
+            name="${robot_prefix}front_right_laser_"
+            parent="${robot_prefix}front_right_laser_attachment_link"
+            topic="/${robot_prefix}front_right_laser"
+            use_gz_sim="${use_gz_sim}"
+            min_angle="-1.5" >
+            <origin xyz="0 0 0" rpy="${pi} 0 0" />
+        </xacro:hokuyo>
+        <!-- rear left -->
+        <xacro:hokuyo
+            name="${robot_prefix}rear_left_laser_"
+            parent="${robot_prefix}rear_left_laser_attachment_link"
+            topic="/${robot_prefix}rear_left_laser"
+            use_gz_sim="${use_gz_sim}"
+            min_angle="-1.3" >
+            <origin xyz="0 0 0" rpy="${pi} 0 ${pi}" />
+        </xacro:hokuyo>
         <!-- Instantiate wheel units -->
         <!-- front left -->
@@ -104,4 +137,5 @@
             use_ros2_control="${use_ros2_control}"
             use_gz_sim="${use_gz_sim}"
+            use_kelo_tulip="${use_kelo_tulip}"
             struct_prefix="${robot_prefix}front_left_drive_"
             struct_wrt_attachment_rpy="${front_left_struct_wrt_attachment_rpy}">
@@ -113,4 +147,5 @@
             use_ros2_control="${use_ros2_control}"
             use_gz_sim="${use_gz_sim}"
+            use_kelo_tulip="${use_kelo_tulip}"
             struct_prefix="${robot_prefix}rear_left_drive_"
             struct_wrt_attachment_rpy="${rear_left_struct_wrt_attachment_rpy}">
@@ -122,4 +157,5 @@
             use_ros2_control="${use_ros2_control}"
             use_gz_sim="${use_gz_sim}"
+            use_kelo_tulip="${use_kelo_tulip}"
             struct_prefix="${robot_prefix}rear_right_drive_"
             struct_wrt_attachment_rpy="${front_right_struct_wrt_attachment_rpy}">
@@ -131,4 +167,5 @@
             use_ros2_control="${use_ros2_control}"
             use_gz_sim="${use_gz_sim}"
+            use_kelo_tulip="${use_kelo_tulip}"
             struct_prefix="${robot_prefix}front_right_drive_"
             struct_wrt_attachment_rpy="${rear_right_struct_wrt_attachment_rpy}">

File: urdf/eddie_robot.urdf.xacro (robot description, xacro)
@@ -37,6 +37,8 @@
     <xacro:include filename="$(find eddie_description)/urdf/kortex.ros2_gz_control.macro.xacro" />
     <!-- Eddie base with KELO hub wheels -->
-    <xacro:eddie_base robot_prefix="$(arg robot_name)" use_ros2_control="$(arg use_ros2_control)"
-        use_gz_sim="$(arg use_gz_sim)" />
+    <xacro:eddie_base robot_prefix="$(arg robot_name)"
+        use_ros2_control="$(arg use_ros2_control)"
+        use_gz_sim="$(arg use_gz_sim)"
+        use_kelo_tulip="$(arg use_kelo_tulip)" />
     <!-- Left Kinova Gen3 7 DoF arm -->
     <xacro:kinova_gen3

File: urdf/kelo_drive_unit.macro.xacro (robot description, xacro)
@@ -4,5 +4,13 @@
     <xacro:include filename="$(find eddie_description)/urdf/kelo_hub_wheel.macro.xacro" />
     <xacro:macro name="kelo_drive_unit"
-        params="parent use_ros2_control use_gz_sim struct_prefix *attachment_origin struct_wrt_attachment_rpy">
+        params="parent use_ros2_control use_gz_sim use_kelo_tulip struct_prefix *attachment_origin
+    struct_wrt_attachment_rpy">
+        <!-- pivot joint type based on use_kelo_tulip -->
+        <xacro:if value="${use_kelo_tulip}">
+            <xacro:property name="pivot_joint_type" value="continuous" />
+        </xacro:if>
+        <xacro:unless value="${use_kelo_tulip}">
+            <xacro:property name="pivot_joint_type" value="fixed" />
+        </xacro:unless>
         <!-- Properties -->
         <xacro:property name="mesh_package" value="eddie_description" />
@@ -59,5 +67,5 @@
         </link>
         <!-- pivot joint -->
-        <joint name="${struct_prefix}pivot_joint" type="continuous">
+        <joint name="${struct_prefix}pivot_joint" type="${pivot_joint_type}">
             <parent link="${struct_prefix}attachment_link" />
             <child link="${struct_prefix}struct_link" />
@@ -65,19 +73,21 @@
             <axis xyz="0 0 1" />
         </joint>
-        <!-- ros2 control tags -->
-        <xacro:if value="${use_ros2_control}">
-            <ros2_control name="${struct_prefix}ctr" type="system">
-                <xacro:if value="${use_gz_sim}">
-                    <hardware>
-                        <plugin>gz_ros2_control/GazeboSimSystem</plugin>
-                    </hardware>
-                </xacro:if>
-                <joint name="${struct_prefix}pivot_joint">
-                    <state_interface name="position">
-                        <param name="initial_value">0.0</param>
-                    </state_interface>
-                    <state_interface name="velocity" />
-                </joint>
-            </ros2_control>
+        <xacro:if value="${use_kelo_tulip}">
+            <!-- ros2 control tags -->
+            <xacro:if value="${use_ros2_control}">
+                <ros2_control name="${struct_prefix}ctr" type="system">
+                    <xacro:if value="${use_gz_sim}">
+                        <hardware>
+                            <plugin>gz_ros2_control/GazeboSimSystem</plugin>
+                        </hardware>
+                    </xacro:if>
+                    <joint name="${struct_prefix}pivot_joint">
+                        <state_interface name="position">
+                            <param name="initial_value">0.0</param>
+                        </state_interface>
+                        <state_interface name="velocity" />
+                    </joint>
+                </ros2_control>
+            </xacro:if>
         </xacro:if>
         <!-- wheels -->
@@ -90,5 +100,6 @@
             parent="${struct_prefix}struct_link"
             use_ros2_control="${use_ros2_control}"
-            use_gz_sim="${use_gz_sim}">
+            use_gz_sim="${use_gz_sim}"
+            use_kelo_tulip="${use_kelo_tulip}">
             <xacro:insert_block name="right_wheel_origin" />
         </xacro:kelo_hub_wheel>
@@ -101,5 +112,6 @@
             parent="${struct_prefix}struct_link"
             use_ros2_control="${use_ros2_control}"
-            use_gz_sim="${use_gz_sim}">
+            use_gz_sim="${use_gz_sim}"
+            use_kelo_tulip="${use_kelo_tulip}">
             <xacro:insert_block name="left_wheel_origin" />
         </xacro:kelo_hub_wheel>

File: urdf/kelo_hub_wheel.macro.xacro (robot description, xacro)
@@ -2,8 +2,15 @@
 <robot xmlns:xacro="http://www.ros.org/wiki/xacro" name="kelo_hub_wheel">
     <xacro:macro name="kelo_hub_wheel"
-        params="wheel_prefix parent *wheel_origin use_ros2_control use_gz_sim">
+        params="wheel_prefix parent *wheel_origin use_ros2_control use_gz_sim use_kelo_tulip">
         <!-- Properties -->
         <xacro:property name="mesh_package" value="eddie_description" />
         <xacro:property name="wheel_mesh_file" value="hub_wheel.stl" />
+        <!-- wheel joint type based on use_kelo_tulip -->
+        <xacro:if value="${use_kelo_tulip}">
+            <xacro:property name="wheel_joint_type" value="continuous" />
+        </xacro:if>
+        <xacro:unless value="${use_kelo_tulip}">
+            <xacro:property name="wheel_joint_type" value="fixed" />
+        </xacro:unless>
         <!-- Links -->
         <link name="${wheel_prefix}link">
@@ -23,6 +30,6 @@
                 <friction>
                     <ode>
-                    <mu>1.0</mu>
-                    <mu2>1.0</mu2>
+                        <mu>1.0</mu>
+                        <mu2>1.0</mu2>
                     </ode>
                 </friction>
@@ -36,5 +43,5 @@
         </link>
         <!-- Joints -->
-        <joint name="${wheel_prefix}joint" type="continuous">
+        <joint name="${wheel_prefix}joint" type="${wheel_joint_type}">
             <parent link="${parent}" />
             <child link="${wheel_prefix}link" />
@@ -42,32 +49,34 @@
             <axis xyz="0 0 1" />
         </joint>
-        <!-- ros2 control tags -->
-        <xacro:if value="${use_ros2_control}">
-            <ros2_control name="${wheel_prefix}ctr" type="system">
-                <xacro:if value="${use_gz_sim}">
-                    <hardware>
-                        <plugin>gz_ros2_control/GazeboSimSystem</plugin>
-                    </hardware>
-                </xacro:if>
-                <joint name="${wheel_prefix}joint">
-                    <command_interface name="position">
-                        <param name="min">-1e+100</param>
-                        <param name="max">1e+100</param>
-                    </command_interface>
-                    <command_interface name="velocity">
-                        <param name="min">-1e+100</param>
-                        <param name="max">1e+100</param>
-                    </command_interface>
-                    <command_interface name="effort">
-                        <param name="min">-1e+100</param>
-                        <param name="max">1e+100</param>
-                    </command_interface>
-                    <state_interface name="position">
-                        <param name="initial_value">0.0</param>
-                    </state_interface>
-                    <state_interface name="velocity" />
-                    <state_interface name="effort" />
-                </joint>
-            </ros2_control>
+        <xacro:if value="${use_kelo_tulip}">
+            <!-- ros2 control tags -->
+            <xacro:if value="${use_ros2_control}">
+                <ros2_control name="${wheel_prefix}ctr" type="system">
+                    <xacro:if value="${use_gz_sim}">
+                        <hardware>
+                            <plugin>gz_ros2_control/GazeboSimSystem</plugin>
+                        </hardware>
+                    </xacro:if>
+                    <joint name="${wheel_prefix}joint">
+                        <command_interface name="position">
+                            <param name="min">-1e+100</param>
+                            <param name="max">1e+100</param>
+                        </command_interface>
+                        <command_interface name="velocity">
+                            <param name="min">-1e+100</param>
+                            <param name="max">1e+100</param>
+                        </command_interface>
+                        <command_interface name="effort">
+                            <param name="min">-1e+100</param>
+                            <param name="max">1e+100</param>
+                        </command_interface>
+                        <state_interface name="position">
+                            <param name="initial_value">0.0</param>
+                        </state_interface>
+                        <state_interface name="velocity" />
+                        <state_interface name="effort" />
+                    </joint>
+                </ros2_control>
+            </xacro:if>
         </xacro:if>
     </xacro:macro>

File: urdf/sensors/hokuyo.urdf.xacro (robot description, xacro)
@@ -1,39 +1,20 @@
 <?xml version="1.0"?>
-<!--
-Copyright (c) 2013, Goncalo Cabrita, ISR University of Coimbra
-Copyright (c) 2014, 2015 Clearpath Robotics
-All rights reserved.
-Redistribution and use in source and binary forms, with or without
-modification, are permitted provided that the following conditions are met:
-    * Redistributions of source code must retain the above copyright
-      notice, this list of conditions and the following disclaimer.
-    * Redistributions in binary form must reproduce the above copyright
-      notice, this list of conditions and the following disclaimer in the
-      documentation and/or other materials provided with the distribution.
-    * Neither the name of Clearpath Robotics nor the
-      names of its contributors may be used to endorse or promote products
-      derived from this software without specific prior written permission.
-THIS SOFTWARE IS PROVIDED BY THE COPYRIGHT HOLDERS AND CONTRIBUTORS "AS IS" AND
-ANY EXPRESS OR IMPLIED WARRANTIES, INCLUDING, BUT NOT LIMITED TO, THE IMPLIED
-WARRANTIES OF MERCHANTABILITY AND FITNESS FOR A PARTICULAR PURPOSE ARE
-DISCLAIMED. IN NO EVENT SHALL THE COPYRIGHT HOLDERS BE LIABLE FOR ANY
-DIRECT, INDIRECT, INCIDENTAL, SPECIAL, EXEMPLARY, OR CONSEQUENTIAL DAMAGES
-(INCLUDING, BUT NOT LIMITED TO, PROCUREMENT OF SUBSTITUTE GOODS OR SERVICES;
-LOSS OF USE, DATA, OR PROFITS; OR BUSINESS INTERRUPTION) HOWEVER CAUSED AND
-ON ANY THEORY OF LIABILITY, WHETHER IN CONTRACT, STRICT LIABILITY, OR TORT
-(INCLUDING NEGLIGENCE OR OTHERWISE) ARISING IN ANY WAY OUT OF THE USE OF THIS
-SOFTWARE, EVEN IF ADVISED OF THE POSSIBILITY OF SUCH DAMAGE.
--->
 <robot xmlns:xacro="http://www.ros.org/wiki/xacro">
-    <xacro:include filename="$(find freddy_base_description)/urdf/sensors/common.xacro" />
-    <xacro:macro name="hokuyo" params="*origin name:=base_laser_front topic:=base_scan parent:=base_link sample_size:=1080 update_rate:=40
-    min_angle:=-2.35619 max_angle:=2.35619 min_range:=0.06 max_range:=10.0 robot_namespace:=/ use_gpu:=true visualize:=false" >
-        <joint name="${name}_joint" type="fixed">
-            <axis xyz="0 1 0" />
-            <xacro:insert_block name="origin"/>
-            <parent link="${parent}"/>
-            <child link="${name}_link"/>
+    <xacro:macro name="hokuyo"
+        params="*origin name topic parent
+                use_gz_sim:=false
+                sample_size:=1080
+                update_rate:=40
+                min_angle:=-2.35619
+                max_angle:=2.35619
+                min_range:=0.06
+                max_range:=10.0
+                visualize:=true">
+        <joint name="${name}joint" type="fixed">
+            <xacro:insert_block name="origin" />
+            <parent link="${parent}" />
+            <child link="${name}link" />
         </joint>
-        <link name="${name}_link">
+        <link name="${name}link">
             <inertial>
                 <mass value="0.16" />
@@ -42,30 +23,49 @@
             </inertial>
             <visual>
-                <origin xyz="0 0 0" rpy="0 0 0" />
+                <origin xyz="0 0 0.015" rpy="0 0 0"/>
                 <geometry>
-                    <mesh filename="package://freddy_base_description/meshes/sensors/hokuyo.dae" />
+                    <mesh filename="package://eddie_description/meshes/sensors/hokuyo.dae" />
                 </geometry>
             </visual>
             <collision>
-                <origin xyz="0 0 0" rpy="0 0 0" />
+                <origin xyz="0 0 0.015" rpy="0 0 0"/>
                 <geometry>
-                    <mesh filename="package://freddy_base_description/meshes/sensors/hokuyo_convex.dae" />
+                    <mesh
+                        filename="package://eddie_description/meshes/sensors/hokuyo_convex.dae" />
                 </geometry>
             </collision>
         </link>
-        <xacro:if value="${use_gpu}">
-            <xacro:gazebo_laser_plugin name="${name}" topic="${topic}" sample_size="${sample_size}"
-                                       update_rate="${update_rate}" min_angle="${min_angle}"
-                                       max_angle="${max_angle}" min_range="${min_range}" max_range="${max_range}"
-                                       robot_namespace="${robot_namespace}" visualize="${visualize}"
-                                       sensor_type="gpu_ray" plugin_filename="libgazebo_ros_gpu_laser"/>
+        <xacro:if value="${use_gz_sim}">
+            <gazebo reference="${name}link">
+                <sensor name='${name}gpu_lidar' type='gpu_lidar'>
+                    <pose relative_to='${name}link'>0 0 0.035 0 0 0</pose>
+                    <topic>${topic}</topic>
+                    <update_rate>${update_rate}</update_rate>
+                    <ray>
+                        <scan>
+                            <horizontal>
+                                <samples>${sample_size}</samples>
+                                <resolution>1</resolution>
+                                <min_angle>${min_angle}</min_angle>
+                                <max_angle>${max_angle}</max_angle>
+                            </horizontal>
+                            <vertical>
+                                <samples>1</samples>
+                                <resolution>0.01</resolution>
+                                <min_angle>0</min_angle>
+                                <max_angle>0</max_angle>
+                            </vertical>
+                        </scan>
+                        <range>
+                            <min>${min_range}</min>
+                            <max>${max_range}</max>
+                            <resolution>0.01</resolution>
+                        </range>
+                    </ray>
+                    <always_on>1</always_on>
+                    <visualize>${visualize}</visualize>
+                </sensor>
+            </gazebo>
         </xacro:if>
-        <xacro:unless value="${use_gpu}">
-            <xacro:gazebo_laser_plugin name="${name}" topic="${topic}" sample_size="${sample_size}"
-                                       update_rate="${update_rate}" min_angle="${min_angle}"
-                                       max_angle="${max_angle}" min_range="${min_range}" max_range="${max_range}"
-                                       robot_namespace="${robot_namespace}" visualize="${visualize}"
-                                       sensor_type="ray" plugin_filename="libgazebo_ros_laser"/>
-        </xacro:unless>
     </xacro:macro>
 </robot>

Commit message: add odom and imu links with joints to the URDF model

File: urdf/eddie_base.macro.xacro (robot description, xacro)
@@ -42,4 +42,11 @@
                 rpy="${0} ${0 + 0.09} ${1.5708 - 2.3632}" />
         </xacro:property>
+        <!-- odom -->
+        <link name="odom" />
+        <joint name="odom_joint" type="fixed">
+            <parent link="odom" />
+            <child link="${robot_prefix}base_footprint" />
+            <origin xyz="0 0 0" rpy="0 0 0" />
+        </joint>
         <!-- Links -->
         <link name="${robot_prefix}base_footprint" />
@@ -119,5 +126,5 @@
             topic="/${robot_prefix}front_right_laser"
             use_gz_sim="${use_gz_sim}"
-            min_angle="-1.5" >
+            min_angle="-1.5">
             <origin xyz="0 0 0" rpy="${pi} 0 0" />
         </xacro:hokuyo>
@@ -128,7 +135,24 @@
             topic="/${robot_prefix}rear_left_laser"
             use_gz_sim="${use_gz_sim}"
-            min_angle="-1.3" >
+            min_angle="-1.3">
             <origin xyz="0 0 0" rpy="${pi} 0 ${pi}" />
         </xacro:hokuyo>
+        <!-- imu -->
+        <link name="${robot_prefix}imu_link" />
+        <joint name="${robot_prefix}imu_joint" type="fixed">
+            <parent link="${robot_prefix}base_link" />
+            <child link="${robot_prefix}imu_link" />
+            <origin xyz="0 0 0" rpy="0 0 0" />
+        </joint>
+        <xacro:if value="${use_gz_sim}">
+            <gazebo reference="${robot_prefix}imu_link">
+                <sensor name="${robot_prefix}imu_sensor" type="imu">
+                    <always_on>1</always_on>
+                    <update_rate>1</update_rate>
+                    <visualize>true</visualize>
+                    <topic>${robot_prefix}imu</topic>
+                </sensor>
+            </gazebo>
+        </xacro:if>
         <!-- Instantiate wheel units -->
         <!-- front left -->

Commit message: remove odom link and joint from the URDF model; add gz_frame_id to hokuyo sensor

File: urdf/eddie_base.macro.xacro (robot description, xacro)
@@ -42,11 +42,4 @@
                 rpy="${0} ${0 + 0.09} ${1.5708 - 2.3632}" />
         </xacro:property>
-        <!-- odom -->
-        <link name="odom" />
-        <joint name="odom_joint" type="fixed">
-            <parent link="odom" />
-            <child link="${robot_prefix}base_footprint" />
-            <origin xyz="0 0 0" rpy="0 0 0" />
-        </joint>
         <!-- Links -->
         <link name="${robot_prefix}base_footprint" />

File: urdf/sensors/hokuyo.urdf.xacro (robot description, xacro)
@@ -42,4 +42,5 @@
                     <topic>${topic}</topic>
                     <update_rate>${update_rate}</update_rate>
+                    <gz_frame_id>${name}link</gz_frame_id>
                     <ray>
                         <scan>

Commit message: update laser link transforms and limits

File: urdf/eddie_base.macro.xacro (robot description, xacro)
@@ -119,6 +119,7 @@
             topic="/${robot_prefix}front_right_laser"
             use_gz_sim="${use_gz_sim}"
-            min_angle="-1.5">
-            <origin xyz="0 0 0" rpy="${pi} 0 0" />
+            max_angle="1.7"
+            min_angle="-1.7">
+            <origin xyz="0 0 0" rpy="${pi} 0 -0.7854" />
         </xacro:hokuyo>
         <!-- rear left -->
@@ -128,6 +129,7 @@
             topic="/${robot_prefix}rear_left_laser"
             use_gz_sim="${use_gz_sim}"
-            min_angle="-1.3">
-            <origin xyz="0 0 0" rpy="${pi} 0 ${pi}" />
+            max_angle="1.7"
+            min_angle="-1.7">
+            <origin xyz="0 0 0" rpy="${pi} 0 2.3562" />
         </xacro:hokuyo>
         <!-- imu -->
