Commit message: update friction values and add dynamics to kelo_hub_wheel and kelo_drive_unit macros

File: urdf/kelo_drive_unit.macro.xacro (robot description, xacro)
@@ -72,4 +72,5 @@
             <xacro:insert_block name="struct_wrt_attachment_origin" />
             <axis xyz="0 0 1" />
+            <dynamics damping="0.1" friction="0.1" />
         </joint>
         <xacro:if value="${use_kelo_tulip}">

File: urdf/kelo_hub_wheel.macro.xacro (robot description, xacro)
@@ -30,6 +30,6 @@
                 <friction>
                     <ode>
-                        <mu>1.0</mu>
-                        <mu2>1.0</mu2>
+                        <mu>0.2</mu>
+                        <mu2>0.1</mu2>
                     </ode>
                 </friction>
@@ -48,4 +48,5 @@
             <xacro:insert_block name="wheel_origin" />
             <axis xyz="0 0 1" />
+            <dynamics damping="0.1" friction="0.1" />
         </joint>
         <xacro:if value="${use_kelo_tulip}">
