Commit message: added kinova gen3 arms

File: urdf/eddie_robot.urdf.xacro (robot description, xacro)
@@ -1,6 +1,66 @@
 <?xml version="1.0"?>
 <robot xmlns:xacro="http://www.ros.org/wiki/xacro" name="eddie_base_with_wheels">
+    <xacro:arg name="robot_name" default="eddie_" />
+    <xacro:arg name="robot_ip_left" default="192.168.1.10" />
+    <xacro:arg name="robot_ip_right" default="192.168.1.11" />
+    <xacro:arg name="username" default="admin" />
+    <xacro:arg name="password" default="admin" />
+    <xacro:arg name="port" default="10000" />
+    <xacro:arg name="port_realtime" default="10001" />
+    <xacro:arg name="session_inactivity_timeout_ms" default="60000" />
+    <xacro:arg name="connection_inactivity_timeout_ms" default="2000" />
+    <!-- <xacro:arg name="gripper" default="robotiq_2f_85" /> -->
+    <xacro:arg name="gripper" default="" />
+    <xacro:arg name="gripper_joint_name" default="grasp_joint" />
+    <xacro:arg name="use_fake_hardware" default="false" />
+    <xacro:arg name="fake_sensor_commands" default="false" />
+    <xacro:arg name="sim_gz" default="true" />
+    <xacro:arg name="sim_isaac" default="false" />
+    <xacro:arg name="use_internal_bus_gripper_comm" default="false" />
+    <!-- initial position for simulations (Mock Hardware, Gazebo, Ignition) -->
+    <xacro:arg name="initial_positions_file_left"
+        default="$(find eddie_description)/config/initial_positions_arm_left.yaml" />
+    <xacro:arg name="initial_positions_file_right"
+        default="$(find eddie_description)/config/initial_positions_arm_right.yaml" />
     <!-- Include the Eddie Base -->
     <xacro:include filename="$(find eddie_description)/urdf/eddie_base.macro.xacro"/>
-    <xacro:eddie_base prefix="eddie_"/>
+    <!-- Include Gen3 Arm -->
+    <xacro:include filename="$(find kortex_description)/urdf/kinova_gen3.macro.xacro"/>
+    <xacro:eddie_base prefix="${xacro:arg robot_name}" />
+    <xacro:kinova_gen3
+        parent="${xacro:arg robot_name}left_arm_attachment_link"
+        prefix="${xacro:arg robot_name}left_arm_"
+        gripper="robotiq_2f_85"
+        robot_ip="$(arg robot_ip_left)"
+        username="$(arg username)"
+        password="$(arg password)"
+        port="$(arg port)"
+        port_realtime="$(arg port_realtime)"
+        session_inactivity_timeout_ms="$(arg session_inactivity_timeout_ms)"
+        connection_inactivity_timeout_ms="$(arg connection_inactivity_timeout_ms)"
+        use_fake_hardware="$(arg use_fake_hardware)"
+        fake_sensor_commands="$(arg fake_sensor_commands)"
+        initial_positions="${xacro.load_yaml(initial_positions_file_left)}"
+        >
+        <!-- TODO: Update origin -->
+        <origin xyz="0 0 0" rpy="0 0 0" />
+    </xacro:kinova_gen3>
+    <xacro:kinova_gen3
+        parent="${xacro:arg robot_name}right_arm_attachment_link"
+        prefix="${xacro:arg robot_name}right_arm_"
+        gripper="robotiq_2f_85"
+        robot_ip="$(arg robot_ip_right)"
+        username="$(arg username)"
+        password="$(arg password)"
+        port="$(arg port)"
+        port_realtime="$(arg port_realtime)"
+        session_inactivity_timeout_ms="$(arg session_inactivity_timeout_ms)"
+        connection_inactivity_timeout_ms="$(arg connection_inactivity_timeout_ms)"
+        use_fake_hardware="$(arg use_fake_hardware)"
+        fake_sensor_commands="$(arg fake_sensor_commands)"
+        initial_positions="${xacro.load_yaml(initial_positions_file_right)}"
+        >
+        <!-- TODO: Update origin -->
+        <origin xyz="0 0 0" rpy="0 0 0" />
+    </xacro:kinova_gen3>
 </robot>

Commit message: add gazebo and control plugins

File: urdf/eddie_robot.urdf.xacro (robot description, xacro)
@@ -19,4 +19,6 @@
     <xacro:arg name="sim_isaac" default="false" />
     <xacro:arg name="use_internal_bus_gripper_comm" default="false" />
+    <xacro:arg name="simulation_controllers"
+        default="$(find eddie_gazebo)/config/eddie_controller.yaml" />
     <!-- initial position for simulations (Mock Hardware, Gazebo, Ignition) -->
     <xacro:arg name="initial_positions_file_left"
@@ -28,8 +30,8 @@
     <xacro:property name="initial_positions_file_right"
         default="$(arg initial_positions_file_right)" />
-    <!-- Include the Eddie Base -->
+    <!-- Include macro files -->
     <xacro:include filename="$(find eddie_description)/urdf/eddie_base.macro.xacro"/>
-    <!-- Include Gen3 Arm -->
     <xacro:include filename="$(find eddie_description)/urdf/kinova_gen3.macro.xacro"/>
+    <xacro:include filename="$(find eddie_description)/urdf/kortex.ros2_gz_control.macro.xacro" />
     <xacro:eddie_base robot_prefix="$(arg robot_name)" joint_state_gui="$(arg joint_state_gui)"/>
     <xacro:kinova_gen3
@@ -49,4 +51,21 @@
         <origin xyz="0.01549 0 0" rpy="1.5708 -1.5708 1.5708" />
     </xacro:kinova_gen3>
+    <xacro:kortex_ros2_control
+        name="$(arg robot_name)left_arm_KortexMultiInterfaceHardware"
+        prefix="$(arg robot_name)left_arm_"
+        use_fake_hardware="$(arg use_fake_hardware)"
+        fake_sensor_commands="$(arg fake_sensor_commands)"
+        sim_gz="$(arg sim_gz)"
+        tf_prefix=""
+        initial_positions="${xacro.load_yaml(initial_positions_file_left)}"
+        robot_ip="$(arg robot_ip_left)"
+        username="$(arg username)"
+        password="$(arg password)"
+        port="$(arg port)"
+        port_realtime="$(arg port_realtime)"
+        session_inactivity_timeout_ms="$(arg session_inactivity_timeout_ms)"
+        connection_inactivity_timeout_ms="$(arg connection_inactivity_timeout_ms)"
+        use_internal_bus_gripper_comm="$(arg use_internal_bus_gripper_comm)"
+        gripper_joint_name="$(arg gripper_joint_name)"/>
     <xacro:kinova_gen3
         parent="$(arg robot_name)right_arm_attachment_link"
@@ -65,3 +84,46 @@
         <origin xyz="0.01549 0 0" rpy="1.5708 -1.5708 1.5708" />
     </xacro:kinova_gen3>
+    <xacro:kortex_ros2_control
+        name="$(arg robot_name)right_arm_KortexMultiInterfaceHardware"
+        prefix="$(arg robot_name)right_arm_"
+        use_fake_hardware="$(arg use_fake_hardware)"
+        fake_sensor_commands="$(arg fake_sensor_commands)"
+        sim_gz="$(arg sim_gz)"
+        tf_prefix=""
+        initial_positions="${xacro.load_yaml(initial_positions_file_right)}"
+        robot_ip="$(arg robot_ip_right)"
+        username="$(arg username)"
+        password="$(arg password)"
+        port="$(arg port)"
+        port_realtime="$(arg port_realtime)"
+        session_inactivity_timeout_ms="$(arg session_inactivity_timeout_ms)"
+        connection_inactivity_timeout_ms="$(arg connection_inactivity_timeout_ms)"
+        use_internal_bus_gripper_comm="$(arg use_internal_bus_gripper_comm)"
+        gripper_joint_name="$(arg gripper_joint_name)"/>
+    <!-- gazebo tag for ros2 control -->
+    <gazebo>
+        <plugin filename="libgz_ros2_control-system.so"
+            name="gz_ros2_control::GazeboSimROS2ControlPlugin">
+            <robot_param>robot_description</robot_param>
+            <robot_param_node>robot_state_publisher</robot_param_node>
+            <parameters>$(arg simulation_controllers)</parameters>
+        </plugin>
+        <self_collide>1</self_collide>
+    </gazebo>
+    <gazebo reference="base_link">
+        <gravity>true</gravity>
+        <self_collide>false</self_collide>
+    </gazebo>
+    <gazebo>
+        <plugin
+            filename="gz-sim-odometry-publisher-system"
+            name="gz::sim::systems::OdometryPublisher">
+            <odom_frame>odom</odom_frame>
+            <robot_base_frame>eddie_base_link</robot_base_frame>
+        </plugin>
+        <plugin
+            filename="gz-sim-velocity-control-system"
+            name="gz::sim::systems::VelocityControl">
+        </plugin>
+    </gazebo>
 </robot>

File: urdf/kelo_drive_unit.macro.xacro (robot description, xacro)
@@ -80,35 +80,4 @@
             <axis xyz="0 0 1"/>
         </joint>
-        <!-- ros2 control tags -->
-        <xacro:if value="${joint_state_gui}">
-            <ros2_control name="${robot_prefix}${struct_prefix}ctr" type="system">
-                <hardware>
-                    <plugin>gz_ros2_control/GazeboSimSystem</plugin>
-                </hardware>
-                <joint name="${robot_prefix}${struct_prefix}struct_joint">
-                    <command_interface name="position">
-                    <param name="min">-1e+100</param>
-                    <param name="max">1e+100</param>
-                    </command_interface>
-                    <command_interface name="velocity">
-                    <param name="min">-1e+100</param>
-                    <param name="max">1e+100</param>
-                    </command_interface>
-                    <command_interface name="effort">
-                    <param name="min">-1e+100</param>
-                    <param name="max">1e+100</param>
-                    </command_interface>
-                    <state_interface name="position">
-                    <param name="initial_value">0.0</param>
-                    </state_interface>
-                    <state_interface name="velocity"/>
-                    <state_interface name="effort"/>
-                </joint>
-                <transmission name="${robot_prefix}${struct_prefix}struct_joint_transmission">
-                    <plugin>transmission_interface/SimpleTansmission</plugin>
-                    <param name="joint_to_actuator">1</param>
-                </transmission>
-            </ros2_control>
-        </xacro:if>
     </xacro:macro>
 </robot>

Commit message: removed redundant gazebo params

File: urdf/eddie_robot.urdf.xacro (robot description, xacro)
@@ -20,5 +20,5 @@
     <xacro:arg name="use_internal_bus_gripper_comm" default="false" />
     <xacro:arg name="simulation_controllers"
-        default="$(find eddie_gazebo)/config/eddie_controller.yaml" />
+        default="$(find eddie_gazebo)/config/eddie_controllers.yaml" />
     <!-- initial position for simulations (Mock Hardware, Gazebo, Ignition) -->
     <xacro:arg name="initial_positions_file_left"
@@ -105,9 +105,13 @@
         <plugin filename="libgz_ros2_control-system.so"
             name="gz_ros2_control::GazeboSimROS2ControlPlugin">
-            <robot_param>robot_description</robot_param>
-            <robot_param_node>robot_state_publisher</robot_param_node>
+            <!-- <robot_param>robot_description</robot_param>
+            <robot_param_node>robot_state_publisher</robot_param_node> -->
             <parameters>$(arg simulation_controllers)</parameters>
+            <ros>
+                <remapping>~/odom:=odom</remapping>
+                <remapping>/tf:=tf</remapping>
+                <remapping>/tf_static:=tf_static</remapping>
+              </ros>
         </plugin>
-        <self_collide>1</self_collide>
     </gazebo>
     <gazebo reference="base_link">

File: urdf/kelo_hub_wheel.macro.xacro (robot description, xacro)
@@ -1,36 +1,38 @@
 <?xml version="1.0"?>
 <robot xmlns:xacro="http://www.ros.org/wiki/xacro" name="kelo_hub_wheel">
-    <xacro:macro name="kelo_hub_wheel" params="wheel_prefix struct_prefix wheel_origin_xyz wheel_orientation_rpy joint_state_gui">
+    <xacro:macro name="kelo_hub_wheel"
+        params="wheel_prefix struct_prefix wheel_origin_xyz wheel_orientation_rpy joint_state_gui">
         <!-- Properties -->
-        <xacro:property name="mesh_package" value="eddie_description"/>
-        <xacro:property name="wheel_mesh_file" value="hub_wheel.stl"/>
+        <xacro:property name="mesh_package" value="eddie_description" />
+        <xacro:property name="wheel_mesh_file" value="hub_wheel.stl" />
         <!-- Links -->
         <link name="${struct_prefix}${wheel_prefix}link">
             <visual>
-                <origin rpy="0 0 0" xyz="0 0 0"/>
+                <origin rpy="0 0 0" xyz="0 0 0" />
                 <geometry>
                     <mesh filename="package://${mesh_package}/meshes/${wheel_mesh_file}" />
                 </geometry>
                 <material name="black">
-                    <color rgba="0 0 0 1.0"/>
+                    <color rgba="0 0 0 1.0" />
                 </material>
             </visual>
             <collision>
                 <geometry>
-                    <mesh filename="package://${mesh_package}/meshes/${wheel_mesh_file}"/>
+                    <mesh filename="package://${mesh_package}/meshes/${wheel_mesh_file}" />
                 </geometry>
             </collision>
             <inertial>
-                <mass value="1.563"/>
+                <mass value="1.563" />
                 <origin rpy="0 0 0" xyz="0 0.00003 -0.00044" />
-                <inertia ixx="0.001012837" ixy="0" ixz="0" iyy="0.001013130" iyz="0" izz="0.001579986"/>
+                <inertia ixx="0.001012837" ixy="0" ixz="0" iyy="0.001013130" iyz="0"
+                    izz="0.001579986" />
             </inertial>
         </link>
         <!-- Joints -->
         <joint name="${struct_prefix}${wheel_prefix}joint" type="continuous">
-            <parent link="${struct_prefix}struct_link"/>
-            <child link="${struct_prefix}${wheel_prefix}link"/>
-            <origin xyz="${wheel_origin_xyz}" rpy="${wheel_orientation_rpy}"/>
-            <axis xyz="0 0 1"/>
+            <parent link="${struct_prefix}struct_link" />
+            <child link="${struct_prefix}${wheel_prefix}link" />
+            <origin xyz="${wheel_origin_xyz}" rpy="${wheel_orientation_rpy}" />
+            <axis xyz="0 0 1" />
         </joint>
         <!-- ros2 control tags -->
@@ -42,25 +44,25 @@
                 <joint name="${struct_prefix}${wheel_prefix}joint">
                     <command_interface name="position">
-                    <param name="min">-1e+100</param>
-                    <param name="max">1e+100</param>
+                        <param name="min">-1e+100</param>
+                        <param name="max">1e+100</param>
                     </command_interface>
                     <command_interface name="velocity">
-                    <param name="min">-1e+100</param>
-                    <param name="max">1e+100</param>
+                        <param name="min">-1e+100</param>
+                        <param name="max">1e+100</param>
                     </command_interface>
                     <command_interface name="effort">
-                    <param name="min">-1e+100</param>
-                    <param name="max">1e+100</param>
+                        <param name="min">-1e+100</param>
+                        <param name="max">1e+100</param>
                     </command_interface>
                     <state_interface name="position">
-                    <param name="initial_value">0.0</param>
+                        <param name="initial_value">0.0</param>
                     </state_interface>
-                    <state_interface name="velocity"/>
-                    <state_interface name="effort"/>
+                    <state_interface name="velocity" />
+                    <state_interface name="effort" />
                 </joint>
-                <transmission name="${struct_prefix}${wheel_prefix}joint_transmission">
+                <!-- <transmission name="${struct_prefix}${wheel_prefix}joint_transmission">
                     <plugin>transmission_interface/SimpleTansmission</plugin>
                     <param name="joint_to_actuator">1</param>
-                </transmission>
+                </transmission> -->
             </ros2_control>
         </xacro:if>

Commit message: add robotiq gripper configuration

File: urdf/eddie_robot.urdf.xacro (robot description, xacro)
@@ -16,6 +16,6 @@
     <xacro:arg name="session_inactivity_timeout_ms" default="60000" />
     <xacro:arg name="connection_inactivity_timeout_ms" default="2000" />
-    <!-- <xacro:arg name="gripper" default="robotiq_2f_85" /> -->
-    <xacro:arg name="gripper" default="" />
+    <xacro:arg name="gripper" default="robotiq_2f_85" />
+    <!-- <xacro:arg name="gripper" default="" /> -->
     <xacro:arg name="gripper_joint_name" default="grasp_joint" />
     <xacro:arg name="use_internal_bus_gripper_comm" default="false" />

File: urdf/kinova_gen3.macro.xacro (robot description, xacro)
@@ -94,4 +94,14 @@
         <origin xyz="0 0 0" rpy="0 0 0" />
       </xacro:robotiq_gripper>
+      <!-- robotiq 2f-85 length parameters -->
+      <xacro:property name="robotiq_85_base_tip_open_length" value="0.1489" />
+      <xacro:property name="robotiq_85_base_tip_closed_length" value="0.1628" />
+      <!-- robotiq 2f-85 grasp link -->
+      <link name="${prefix}robotiq_85_grasp_link" />
+      <joint name="${prefix}robotiq_85_grasp_joint" type="fixed">
+        <parent link="${prefix}robotiq_85_base_link"/>
+        <child link="${prefix}robotiq_85_grasp_link"/>
+        <origin rpy="0 0 0" xyz="0 0 ${robotiq_85_base_tip_open_length}"/>
+      </joint>
     </xacro:unless>
   </xacro:macro>

Commit message: add ft sensor with gripper coupling

File: urdf/eddie_robot.urdf.xacro (robot description, xacro)
@@ -82,4 +82,7 @@
         prefix="$(arg robot_name)right_arm_"
         gripper="$(arg gripper)"
+        insert_ft_sensor="true"
+        ft_sensor_height="0.064"
+        ft_sensor_diameter="0.075"
         robot_ip="$(arg robot_ip_right)"
         username="$(arg username)"

File: urdf/kinova_gen3.macro.xacro (robot description, xacro)
@@ -26,4 +26,7 @@
     isaac_joint_states:=/isaac_joint_states
     use_external_cable:=false
+    insert_ft_sensor:=false
+    ft_sensor_height:=0.064
+    ft_sensor_diameter:=0.075
     initial_positions:=${dict(joint_1=0.0,joint_2=0.0,joint_3=0.0,joint_4=0.0,joint_5=0.0,joint_6=0.0,joint_7=0.0)}
     gripper_max_velocity:=100.0
@@ -81,8 +84,41 @@
         <xacro:property name="include_ros2_control" value="true" />
       </xacro:if>
+      <xacro:property name="gripper_parent_link" value="${prefix}${last_arm_link}" />
+      <xacro:property name="gripper_mount_z" value="0.0" />
+      <xacro:if value="${insert_ft_sensor}">
+        <link name="${prefix}ft_sensor_link">
+          <visual>
+            <origin xyz="0 0 ${ft_sensor_height / 2.0 + 0.0029}" rpy="0 0 0" />
+            <geometry>
+              <cylinder radius="${ft_sensor_diameter / 2.0}" length="${ft_sensor_height}" />
+            </geometry>
+            <material name="${prefix}ft_sensor_material">
+              <color rgba="0.2 0.2 0.2 1" />
+            </material>
+          </visual>
+          <collision>
+            <origin xyz="0 0 ${ft_sensor_height / 2.0}" rpy="0 0 0" />
+            <geometry>
+              <cylinder radius="${ft_sensor_diameter / 2.0}" length="${ft_sensor_height}" />
+            </geometry>
+          </collision>
+          <inertial>
+            <origin xyz="0 0 ${ft_sensor_height / 2.0}" rpy="0 0 0" />
+            <mass value="0.6" />
+            <inertia ixx="1e-4" ixy="0" ixz="0" iyy="1e-4" iyz="0" izz="1e-4" />
+          </inertial>
+        </link>
+        <joint name="${prefix}ft_sensor_joint" type="fixed">
+          <parent link="${prefix}${last_arm_link}" />
+          <child link="${prefix}ft_sensor_link" />
+          <origin xyz="0 0 0" rpy="0 0 0" />
+        </joint>
+        <xacro:property name="gripper_parent_link" value="${prefix}ft_sensor_link" />
+        <xacro:property name="gripper_mount_z" value="${ft_sensor_height}" />
+      </xacro:if>
       <xacro:robotiq_gripper
         name="RobotiqGripperHardwareInterface"
         prefix="${prefix}"
-        parent="${prefix}${last_arm_link}"
+        parent="${gripper_parent_link}"
         include_ros2_control="false"
         com_port="${gripper_com_port}"
@@ -92,5 +128,5 @@
         isaac_joint_commands="${isaac_joint_commands}"
         isaac_joint_states="${isaac_joint_states}">
-        <origin xyz="0 0 0" rpy="0 0 0" />
+        <origin xyz="0 0 ${gripper_mount_z}" rpy="0 0 0" />
       </xacro:robotiq_gripper>
       <!-- robotiq 2f-85 length parameters -->
