Commit message: changed table size

File: urdf/table.macro.xacro (robot description, xacro)
@@ -7,5 +7,5 @@
         <origin xyz="-0.305 0 0.682" rpy="0 0 0" />
         <geometry>
-          <box size="0.8 0.8 0.05" />
+          <box size="0.8 1.6 0.05" />
         </geometry>
         <material name="Grey">
@@ -15,5 +15,5 @@
       <visual>
         <!-- Leg 1 -->
-        <origin xyz="0.045 0.35 0.3285" rpy="0 0 0" />
+        <origin xyz="0.045 0.70 0.3285" rpy="0 0 0" />
         <geometry>
           <box size="0.05 0.05 0.657" />
@@ -25,5 +25,5 @@
       <visual>
         <!-- Leg 2 -->
-        <origin xyz="0.045 -0.35 0.3285" rpy="0 0 0" />
+        <origin xyz="0.045 -0.70 0.3285" rpy="0 0 0" />
         <geometry>
           <box size="0.05 0.05 0.657" />
@@ -35,5 +35,5 @@
       <visual>
         <!-- Leg 3 -->
-        <origin xyz="-0.655 0.35 0.3285" rpy="0 0 0" />
+        <origin xyz="-0.655 0.70 0.3285" rpy="0 0 0" />
         <geometry>
           <box size="0.05 0.05 0.657" />
@@ -45,5 +45,5 @@
       <visual>
         <!-- Leg 4 -->
-        <origin xyz="-0.655 -0.35 0.3285" rpy="0 0 0" />
+        <origin xyz="-0.655 -0.70 0.3285" rpy="0 0 0" />
         <geometry>
           <box size="0.05 0.05 0.657" />
@@ -57,10 +57,10 @@
         <origin xyz="-0.305 0 0.682" rpy="0 0 0" />
         <geometry>
-          <box size="0.8 0.8 0.05" />
+          <box size="0.8 1.6 0.05" />
         </geometry>
       </collision>
       <collision>
         <!-- Leg 1 -->
-        <origin xyz="0.045 0.35 0.3285" rpy="0 0 0" />
+        <origin xyz="0.045 0.70 0.3285" rpy="0 0 0" />
         <geometry>
           <box size="0.05 0.05 0.657" />
@@ -69,5 +69,5 @@
       <collision>
         <!-- Leg 2 -->
-        <origin xyz="0.045 -0.35 0.3285" rpy="0 0 0" />
+        <origin xyz="0.045 -0.70 0.3285" rpy="0 0 0" />
         <geometry>
           <box size="0.05 0.05 0.657" />
@@ -76,5 +76,5 @@
       <collision>
         <!-- Leg 3 -->
-        <origin xyz="-0.655 0.35 0.3285" rpy="0 0 0" />
+        <origin xyz="-0.655 0.70 0.3285" rpy="0 0 0" />
         <geometry>
           <box size="0.05 0.05 0.657" />
@@ -83,5 +83,5 @@
       <collision>
         <!-- Leg 4 -->
-        <origin xyz="-0.655 -0.35 0.3285" rpy="0 0 0" />
+        <origin xyz="-0.655 -0.70 0.3285" rpy="0 0 0" />
         <geometry>
           <box size="0.05 0.05 0.657" />
