Commit message: increase weight of force torque sensor

File: urdf/kinova_gen3.macro.xacro (robot description, xacro)
@@ -105,5 +105,5 @@
           <inertial>
             <origin xyz="0 0 ${ft_sensor_height / 2.0}" rpy="0 0 0" />
-            <mass value="0.6" />
+            <mass value="1.2" />
             <inertia ixx="1e-4" ixy="0" ixz="0" iyy="1e-4" iyz="0" izz="1e-4" />
           </inertial>
